Commit message: hand-eye calibration completed.

File: urdf/common/camera.urdf.xacro (robot description, xacro)
@@ -33,5 +33,11 @@
             <child link="${frame_id}"/>
         </joint>
-        <link name="${frame_id}"/>
+        <link name="${frame_id}">
+            <inertial>
+                <mass value="0.001"/>
+                <origin xyz="0.0 0.0 0.0"/>
+                <inertia ixx="2.129e-9" ixy="7.329e-9" ixz="-1.11e-9" iyy="2.198e-9" iyz="-8.04e-9" izz="2.197e-9"/>
+            </inertial>
+        </link>
         <xacro:if value="${camera_sim}">
             <gazebo reference="camera_link">

File: urdf/standard3/gimbal.transmission.urdf.xacro (robot description, xacro)
@@ -7,5 +7,5 @@
         </actuator>
         <joint name="yaw_joint">
-            <offset>-3.678</offset>
+            <offset>-3.689</offset>
             <hardwareInterface>hardware_interface/EffortJointInterface</hardwareInterface>
         </joint>
@@ -17,5 +17,5 @@
         </actuator>
         <joint name="pitch_joint">
-            <offset>-2.208</offset>
+            <offset>-2.268</offset>
             <hardwareInterface>hardware_interface/EffortJointInterface</hardwareInterface>
         </joint>

File: urdf/standard3/standard3.urdf.xacro (robot description, xacro)
@@ -15,4 +15,13 @@
             <xacro:include filename="$(find rm_description)/urdf/common/camera.urdf.xacro"/>
             <xacro:include filename="$(find rm_description)/urdf/common/imu.urdf.xacro"/>
+            <xacro:camera_sensor xyz="0.01 0.05 0.06" rpy="0 0 0" frame_id="$(arg camera_link)" parent="pitch"
+                                 camera_sim="$(arg use_simulation)"/>
+            <xacro:camera_optical_frame xyz="0.03630540 0.02695002 0.07130801" rpy="1.5997419 0.1162527 1.5697408"
+                                        frame_id="$(arg camera_optical_frame)"
+                                        parent="pitch"
+                                        camera_sim="$(arg use_simulation)"/>
+            <xacro:IMU connected_to="$(arg camera_optical_frame)" imu_name="gimbal_imu"
+                       xyz="-0.05766461 -0.00498878 -0.02889381"
+                       rpy="1.44537832 0.01314763 0.09321356"/>
             <xacro:if value="$(arg load_shooter)">
                 <xacro:include filename="$(find rm_description)/urdf/standard/shooter.urdf.xacro"/>
