Commit message: Update balance by adding reaction_wheel and updating swerve drive.

File: urdf/common/swerve_drive.urdf.xacro (robot description, xacro)
@@ -1,5 +1,5 @@
 <robot xmlns:xacro="http://www.ros.org/wiki/xacro">
     <xacro:macro name="swerve_drive"
-                 params="prefix wheel_x_offset wheel_y_offset wheel_z_offset  connected_to">
+                 params="prefix x_offset y_offset z_offset  connected_to">
         <link name="${prefix}_pivot">
             <visual>
@@ -11,28 +11,21 @@
             </visual>
             <inertial>
-                    <mass value="0.854"/>
-                    <origin xyz="0.000054 0.008 0.00548" rpy="0 0 0"/>
-                    <inertia ixx="6.711e-4" ixy="1.958e-9" ixz="-1.109e-6" iyy="6.703e-4" iyz="-1.095e-7"
-                             izz="7.091e-4"/>
+                <mass value="0.114131"/>
+                <origin xyz="-0.00005 0.017079 -0.041536" rpy="0 0 0"/>
+                <inertia ixx="1.335e-4" ixy="26.001e-9" ixz="65.031e-9" iyy="1.372e-4" iyz="20051.742e-9"
+                         izz="66866.081e-9"/>
             </inertial>
-            <collision>
-                <origin xyz="0 0 0" rpy="0 0 0"/>
-                <geometry>
-                    <mesh filename="package://rm_description/meshes/common/swerve_pivot.stl"
-                          scale="0.001 0.001 0.001"/>
-                </geometry>
-            </collision>
         </link>
         <joint name="${prefix}_pivot_joint" type="revolute">
             <axis xyz="0 0 1"/>
-            <origin xyz="${wheel_x_offset} ${wheel_y_offset} ${wheel_z_offset}" rpy="0 0 0"/>
+            <origin xyz="${x_offset} ${y_offset} ${z_offset}" rpy="0 0 0"/>
             <parent link="${connected_to}"/>
             <child link="${prefix}_pivot"/>
             <dynamics damping="0.0" friction="0.1"/>
-            <limit effort="1.2" velocity="31" lower="-1e10" upper="1e10"/>
+            <limit effort="1.2" velocity="50" lower="-1e10" upper="1e10"/>
         </joint>
         <link name="${prefix}_wheel">
             <visual>
-                <origin xyz="0 0.0265 0" rpy="0 0 0"/>
+                <origin xyz="0 0 0" rpy="0 0 0"/>
                 <geometry>
                     <mesh filename="package://rm_description/meshes/common/swerve_wheel.stl"
@@ -41,12 +34,13 @@
             </visual>
             <inertial>
-                <mass value="0.543"/>
-                <origin xyz="0.000024 0.024 0.000129" rpy="0 0 0"/>
-                <inertia ixx="4.895e-4" ixy="-3.948e-7" ixz="1.726e-7" iyy="2.894e-4" iyz="1.133e-6" izz="4.887e-4"/>
+                <mass value="0.267401"/>
+                <origin xyz="-0.000004 0.000125 0.000001" rpy="0 0 0"/>
+                <inertia ixx="3.585e-4" ixy="0" ixz="13.459e-9" iyy="6.846e-4" iyz="0"
+                         izz="3.584e-4"/>
             </inertial>
             <collision>
                 <origin xyz="0 0 0" rpy="${pi/2.} 0 0"/>
                 <geometry>
-                    <cylinder radius="0.05" length="0.053"/>
+                    <cylinder length="0.02" radius="0.055"/>
                 </geometry>
             </collision>
@@ -54,8 +48,8 @@
         <joint name="${prefix}_wheel_joint" type="revolute">
             <axis xyz="0 1 0"/>
-            <origin xyz="0 0 -0.112" rpy="0 0 0"/>
+            <origin xyz="0 0 -0.06635" rpy="0 0 0"/>
             <parent link="${prefix}_pivot"/>
             <child link="${prefix}_wheel"/>
-            <limit effort="2.2" velocity="68" lower="-1e10" upper="1e10"/>
+            <limit effort="3" velocity="76" lower="-1e10" upper="1e10"/>
             <dynamics damping="0.0" friction="0.05"/>
         </joint>
@@ -79,13 +73,13 @@
             </joint>
         </transmission>
-        <transmission name="${prefix}_wheel_trans">
-            <type>transmission_interface/SimpleTransmission</type>
-            <actuator name="${prefix}_wheel_motor">
-                <mechanicalReduction>${wheel_reduction}</mechanicalReduction>
-            </actuator>
-            <joint name="${prefix}_wheel_joint">
-                <hardwareInterface>hardware_interface/EffortJointInterface</hardwareInterface>
-            </joint>
-        </transmission>
+        <!--        <transmission name="${prefix}_wheel_trans">-->
+        <!--            <type>transmission_interface/SimpleTransmission</type>-->
+        <!--            <actuator name="${prefix}_wheel_motor">-->
+        <!--                <mechanicalReduction>${wheel_reduction}</mechanicalReduction>-->
+        <!--            </actuator>-->
+        <!--            <joint name="${prefix}_wheel_joint">-->
+        <!--                <hardwareInterface>hardware_interface/EffortJointInterface</hardwareInterface>-->
+        <!--            </joint>-->
+        <!--        </transmission>-->
     </xacro:macro>
 </robot>

Commit message: Update the swerve_drive.urdf.xacro by uncommenting and correcting the gazebo label.

File: urdf/common/swerve_drive.urdf.xacro (robot description, xacro)
@@ -55,6 +55,6 @@
         </joint>
         <gazebo reference="${prefix}_wheel">
-            <mu1 value="20"/>
-            <mu2 value="20"/>
+            <mu1 value="1.0"/>
+            <mu2 value="1.0"/>
             <kp value="1000000.0"/>
             <kd value="100.0"/>
@@ -73,13 +73,13 @@
             </joint>
         </transmission>
-        <!--        <transmission name="${prefix}_wheel_trans">-->
-        <!--            <type>transmission_interface/SimpleTransmission</type>-->
-        <!--            <actuator name="${prefix}_wheel_motor">-->
-        <!--                <mechanicalReduction>${wheel_reduction}</mechanicalReduction>-->
-        <!--            </actuator>-->
-        <!--            <joint name="${prefix}_wheel_joint">-->
-        <!--                <hardwareInterface>hardware_interface/EffortJointInterface</hardwareInterface>-->
-        <!--            </joint>-->
-        <!--        </transmission>-->
+        <transmission name="${prefix}_wheel_trans">
+            <type>transmission_interface/SimpleTransmission</type>
+            <actuator name="${prefix}_wheel_motor">
+                <mechanicalReduction>${wheel_reduction}</mechanicalReduction>
+            </actuator>
+            <joint name="${prefix}_wheel_joint">
+                <hardwareInterface>hardware_interface/EffortJointInterface</hardwareInterface>
+            </joint>
+        </transmission>
     </xacro:macro>
 </robot>
