Commit message: Update the hero description files

File: urdf/hero/gimbal.urdf.xacro (robot description, xacro)
@@ -6,8 +6,8 @@
     <link name="yaw">
         <inertial>
-            <mass value="3.941"/>
-            <origin xyz="-0.052 -0.057 0.152"/>
-            <inertia ixx="1.250e-1" ixy="-1.357e-2" ixz="3.487e-2" iyy="1.218e-1"
-                     iyz="3.775e-2" izz="3.242e-2"/>
+            <mass value="2.171"/>
+            <origin xyz="-0.0423 0.0528 0.0324"/>
+            <inertia ixx="1.926e-2" ixy="4.754e-3" ixz="7.073e-3" iyy="1.801e-2"
+                     iyz="-3.208e-3" izz="1.945e-2"/>
         </inertial>
         <visual>
@@ -25,5 +25,5 @@
     </link>
     <joint name="yaw_joint" type="revolute">
-        <origin xyz="0 0 0.129"
+        <origin xyz="0 0 0.205"
                 rpy="0 0 0"/>
         <dynamics damping="0.0" friction="0.1"/>
@@ -35,8 +35,8 @@
     <link name="pitch">
         <inertial>
-            <mass value="1.125"/>
-            <origin xyz="0.104 0.0 0.024"/>
-            <inertia ixx="2.658e-3" ixy="4.995e-6" ixz="-3.326e-3" iyy="2.084e-2"
-                     iyz="6.020e-6" izz="1.948e-2"/>
+            <mass value="1.43"/>
+            <origin xyz="0.0480 0.00133 0.0501"/>
+            <inertia ixx="1.087e-2" ixy="1.543e-3" ixz="-1.474e-3" iyy="1.820e-2"
+                     iyz="3.219e-3" izz="1.614e-2"/>
         </inertial>
         <visual>
@@ -54,5 +54,5 @@
     </link>
     <joint name="pitch_joint" type="revolute">
-        <origin xyz="-0.06  0 0.191 " rpy="0 0 0"/>
+        <origin xyz="-0.05 0 0.151 " rpy="0 0 0"/>
         <dynamics damping="0.0" friction="0.1"/>
         <limit effort="1.2" velocity="13.82" lower="${pitch_lower_limit}" upper="${pitch_upper_limit}"/>

File: urdf/hero/hero.urdf.xacro (robot description, xacro)
@@ -16,10 +16,10 @@
             <xacro:include filename="$(find rm_description)/urdf/common/imu.urdf.xacro"/>
             <xacro:include filename="$(find rm_description)/urdf/common/camera.urdf.xacro"/>
-            <xacro:camera_sensor xyz="0.05 0 -0.07" rpy="${pi} 0 -0.02" frame_id="$(arg camera_link)" parent="pitch"
+            <xacro:camera_sensor xyz="0.0445 0 0.109" rpy="${pi} 0 -0.02" frame_id="$(arg camera_link)" parent="pitch"
                                  camera_sim="$(arg use_simulation)"/>
             <xacro:camera_optical_frame xyz="0.2527 0.0071 -0.0984" rpy="1.5486 -0.0025 1.600"
                                         frame_id="$(arg camera_optical_frame)" parent="pitch"
                                         camera_sim="$(arg use_simulation)"/>
-            <xacro:IMU connected_to="pitch" imu_name="gimbal_imu" xyz="0.08 0. 0.08" rpy="0 0 -${pi/2}"/>
+            <xacro:IMU connected_to="pitch" imu_name="gimbal_imu" xyz="0.08 0. 0.08" rpy="${pi} ${pi} ${pi}"/>
             <xacro:if value="$(arg load_shooter)">
                 <xacro:include filename="$(find rm_description)/urdf/hero/shooter.urdf.xacro"/>
