Commit message: Update hero gimbal offset and trigger_joint limit.

File: urdf/hero/gimbal.transmission.urdf.xacro (robot description, xacro)
@@ -7,5 +7,5 @@
         </actuator>
         <joint name="yaw_joint">
-            <offset>-3.607</offset>
+            <offset>-6.245</offset>
             <hardwareInterface>hardware_interface/EffortJointInterface</hardwareInterface>
         </joint>
@@ -17,5 +17,5 @@
         </actuator>
         <joint name="pitch_joint">
-            <offset>0.876</offset>
+            <offset>1.738</offset>
             <hardwareInterface>hardware_interface/EffortJointInterface</hardwareInterface>
         </joint>

File: urdf/hero/hero.urdf.xacro (robot description, xacro)
@@ -18,8 +18,11 @@
             <xacro:camera_sensor xyz="0.0445 0 0.109" rpy="${pi} 0 -0.02" frame_id="$(arg camera_link)" parent="pitch"
                                  camera_sim="$(arg use_simulation)"/>
-            <xacro:camera_optical_frame xyz="0.2527 0.0071 -0.0984" rpy="1.5486 -0.0025 1.600"
+            <xacro:camera_optical_frame xyz="0.053996383919419064 0.011426263468641337 0.12687034281800838"
+                                        rpy="-1.565194 -0.0032789 -1.5085619"
                                         frame_id="$(arg camera_optical_frame)" parent="pitch"
                                         camera_sim="$(arg use_simulation)"/>
-            <xacro:IMU connected_to="pitch" imu_name="gimbal_imu" xyz="0.08 0. 0.08" rpy="${pi} ${pi} ${pi}"/>
+            <xacro:IMU connected_to="$(arg camera_optical_frame)" imu_name="gimbal_imu"
+                       xyz="-0.00242945 0.0499815 -0.06200325"
+                       rpy="1.5680182 -0.0089037 3.1351505"/>
             <xacro:if value="$(arg load_shooter)">
                 <xacro:include filename="$(find rm_description)/urdf/hero/shooter.urdf.xacro"/>

File: urdf/hero/shooter.urdf.xacro (robot description, xacro)
@@ -30,8 +30,8 @@
         </collision>
     </link>
-    <joint name="trigger_joint" type="continuous">
+    <joint name="trigger_joint" type="revolute">
         <origin xyz="0 0 0.063" rpy="0 0 0"/>
         <dynamics damping="0.0" friction="0.01"/>
-        <limit effort="6.99" velocity="35.758" lower="-1e16" upper="1e16"/>
+        <limit effort="12" velocity="12.5" lower="-1e16" upper="1e16"/>
         <parent link="base_link"/>
         <child link="trigger"/>
