Commit message: Update hero urdf and yaml.

File: urdf/hero/chassis.urdf.xacro (robot description, xacro)
@@ -2,14 +2,14 @@
     <xacro:include filename="$(find rm_description)/urdf/common/mecanum_wheel.urdf.xacro"/>
     <!-- https://upload.wikimedia.org/wikipedia/commons/5/52/Wheelbase_and_Track.png -->
-    <xacro:property name="wheel_track" value="0.392"/>
-    <xacro:property name="wheel_base" value="0.404"/>
-    <xacro:property name="wheel_offset_z" value="0.000031"/>
+    <xacro:property name="wheel_track" value="0.4"/>
+    <xacro:property name="wheel_base" value="0.4"/>
+    <xacro:property name="wheel_offset_z" value="-0.068374"/>
     <xacro:macro name="chassis" params="roller_type">
         <link name="base_link">
             <inertial>
-                <mass value="8.44"/>
-                <origin xyz="-0.000578 0.00437 0.0620"/>
-                <inertia ixx="2.081e-1" ixy="5.195e-3" ixz="2.242e-3" iyy="2.784e-1"
-                         iyz="2.494e-3" izz="3.521e-1"/>
+                <mass value="10.34269"/>
+                <origin xyz="-0.003691 -0.001885 0.024404"/>
+                <inertia ixx="1.952E-01" ixy="-1.504E-03" ixz="5.871E-03" iyy="3.011E-01"
+                         iyz="-1.077E-03" izz="4.074E-01"/>
             </inertial>
             <visual>
@@ -29,17 +29,17 @@
                              wheel_x_offset="${wheel_track/2}" wheel_y_offset="${wheel_base/2}"
                              wheel_z_offset="${wheel_offset_z}"
-                             reflect="1" roller_type="${roller_type}" max_effort="5" max_velocity="50"/>
+                             reflect="1" roller_type="${roller_type}"/>
         <xacro:mecanum_wheel prefix="right_front" connected_to="base_link"
                              wheel_x_offset="${wheel_track/2}" wheel_y_offset="${-wheel_base/2}"
                              wheel_z_offset="${wheel_offset_z}"
-                             reflect="-1" roller_type="${roller_type}" max_effort="5" max_velocity="50"/>
+                             reflect="-1" roller_type="${roller_type}"/>
         <xacro:mecanum_wheel prefix="left_back" connected_to="base_link"
                              wheel_x_offset="${-wheel_track/2}" wheel_y_offset="${wheel_base/2}"
                              wheel_z_offset="${wheel_offset_z}"
-                             reflect="-1" roller_type="${roller_type}" max_effort="5" max_velocity="50"/>
+                             reflect="-1" roller_type="${roller_type}"/>
         <xacro:mecanum_wheel prefix="right_back" connected_to="base_link"
                              wheel_x_offset="${-wheel_track/2}" wheel_y_offset="${-wheel_base/2}"
                              wheel_z_offset="${wheel_offset_z}"
-                             reflect="1" roller_type="${roller_type}" max_effort="5" max_velocity="50"/>
+                             reflect="1" roller_type="${roller_type}"/>
         <xacro:wheel_transmission prefix="left_front" mechanical_reduction="19.2032"/>
         <xacro:wheel_transmission prefix="right_front" mechanical_reduction="-19.2032"/>

File: urdf/hero/gimbal.transmission.urdf.xacro (robot description, xacro)
@@ -4,8 +4,8 @@
         <type>transmission_interface/SimpleTransmission</type>
         <actuator name="yaw_joint_motor">
-            <mechanicalReduction>1</mechanicalReduction>
+            <mechanicalReduction>-1</mechanicalReduction>
         </actuator>
         <joint name="yaw_joint">
-            <offset>-0.6102930359999998</offset>
+            <offset>1.763526116</offset>
             <hardwareInterface>hardware_interface/EffortJointInterface</hardwareInterface>
         </joint>
@@ -17,5 +17,5 @@
         </actuator>
         <joint name="pitch_joint">
-            <offset>1.738</offset>
+            <offset>2.180819812</offset>
             <hardwareInterface>hardware_interface/EffortJointInterface</hardwareInterface>
         </joint>

File: urdf/hero/gimbal.urdf.xacro (robot description, xacro)
@@ -6,8 +6,8 @@
     <link name="yaw">
         <inertial>
-            <mass value="2.171"/>
-            <origin xyz="-0.0423 0.0528 0.0324"/>
-            <inertia ixx="1.926e-2" ixy="4.754e-3" ixz="7.073e-3" iyy="1.801e-2"
-                     iyz="-3.208e-3" izz="1.945e-2"/>
+            <mass value="3.362534"/>
+            <origin xyz="-0.048138 0.035027 0.064443"/>
+            <inertia ixx="5.361E-02" ixy="-1.810E-03" ixz="1.319E-02" iyy="4.651E-02"
+                     iyz="1.298E-02" izz="2.967E-02"/>
         </inertial>
         <visual>
@@ -25,8 +25,8 @@
     </link>
     <joint name="yaw_joint" type="revolute">
-        <origin xyz="0 0 0.205"
+        <origin xyz="0 0 0.184"
                 rpy="0 0 0"/>
         <dynamics damping="0.0" friction="0.1"/>
-        <limit effort="1.2" velocity="13.82" lower="-1e10" upper="1e10"/>
+        <limit effort="1.2" velocity="13.82" lower="-1E10" upper="1E10"/>
         <parent link="base_link"/>
         <child link="yaw"/>
@@ -35,8 +35,8 @@
     <link name="pitch">
         <inertial>
-            <mass value="1.43"/>
-            <origin xyz="0.0480 0.00133 0.0501"/>
-            <inertia ixx="1.087e-2" ixy="1.543e-3" ixz="-1.474e-3" iyy="1.820e-2"
-                     iyz="3.219e-3" izz="1.614e-2"/>
+            <mass value="1.183148"/>
+            <origin xyz="0.085638 0.00023 0.047017"/>
+            <inertia ixx="2.934E-03" ixy="3.462E-05" ixz="1.834E-03" iyy="9.223E-03"
+                     iyz="-0.422E-05" izz="8.072E-03"/>
         </inertial>
         <visual>
@@ -54,5 +54,5 @@
     </link>
     <joint name="pitch_joint" type="revolute">
-        <origin xyz="-0.05 0 0.151 " rpy="0 0 0"/>
+        <origin xyz="-0.05 0 0.151" rpy="0 0 0"/>
         <dynamics damping="0.0" friction="0.1"/>
         <limit effort="1.2" velocity="13.82" lower="${pitch_lower_limit}" upper="${pitch_upper_limit}"/>

File: urdf/hero/hero.urdf.xacro (robot description, xacro)
@@ -18,11 +18,8 @@
             <xacro:camera_sensor xyz="0.0445 0 0.109" rpy="${pi} 0 -0.02" frame_id="$(arg camera_link)" parent="pitch"
                                  camera_sim="$(arg use_simulation)"/>
-            <xacro:camera_optical_frame xyz="0.053996383919419064 0.011426263468641337 0.12687034281800838"
-                                        rpy="-1.565194 -0.0032789 -1.5085619"
+            <xacro:camera_optical_frame xyz="0.2527 0.0071 -0.0984" rpy="1.5486 -0.0025 1.600"
                                         frame_id="$(arg camera_optical_frame)" parent="pitch"
                                         camera_sim="$(arg use_simulation)"/>
-            <xacro:IMU connected_to="$(arg camera_optical_frame)" imu_name="gimbal_imu"
-                       xyz="-0.00242945 0.0499815 -0.06200325"
-                       rpy="1.5680182 -0.0089037 3.1351505"/>
+            <xacro:IMU connected_to="pitch" imu_name="gimbal_imu" xyz="0.08 0. 0.08" rpy="${pi} 0 ${pi/2}"/>
             <xacro:if value="$(arg load_shooter)">
                 <xacro:include filename="$(find rm_description)/urdf/hero/shooter.urdf.xacro"/>

File: urdf/hero/shooter.urdf.xacro (robot description, xacro)
@@ -12,8 +12,8 @@
     <link name="trigger">
         <inertial>
-            <mass value="1.4"/>
-            <origin xyz="-0.0146 -0.00736 -0.00154"/>
-            <inertia ixx="4.443e-3" ixy="-1.694e-3" ixz="-1.776e-3" iyy="1.122e-2"
-                     iyz="-3.693e-4" izz="1.347e-2"/>
+            <mass value="0.956931"/>
+            <origin xyz="0.053245 0.000335 -0.031478"/>
+            <inertia ixx="1.367E-03" ixy="0.879E-04" ixz="4.058E-04" iyy="4.812E-03"
+                     iyz="0.221E-04" izz="4.823E-03"/>
         </inertial>
         <visual>
@@ -30,8 +30,8 @@
         </collision>
     </link>
-    <joint name="trigger_joint" type="revolute">
-        <origin xyz="0 0 0.063" rpy="0 0 0"/>
+    <joint name="trigger_joint" type="continuous">
+        <origin xyz="0 0 0.0223" rpy="0 0 0"/>
         <dynamics damping="0.0" friction="0.01"/>
-        <limit effort="7.77" velocity="19.305019" lower="-1e16" upper="1e16"/>
+        <limit effort="6.99" velocity="35.758" lower="-1e16" upper="1e16"/>
         <parent link="base_link"/>
         <child link="trigger"/>

File: urdf/standard4/gimbal.transmission.urdf.xacro (robot description, xacro)
@@ -7,5 +7,5 @@
         </actuator>
         <joint name="yaw_joint">
-            <offset>-6.7771871400000006</offset>
+            <offset>0.519315868</offset>
             <hardwareInterface>hardware_interface/EffortJointInterface</hardwareInterface>
         </joint>
