Commit message: Update hero trigger mechanical reductio, max effort and max velocity.

File: urdf/hero/shooter.transmission.urdf.xacro (robot description, xacro)
@@ -4,5 +4,5 @@
         <type>transmission_interface/SimpleTransmission</type>
         <actuator name="trigger_joint_motor">
-            <mechanicalReduction>76.8128</mechanicalReduction>
+            <mechanicalReduction>49.8083</mechanicalReduction>
         </actuator>
         <joint name="trigger_joint">

File: urdf/hero/shooter.urdf.xacro (robot description, xacro)
@@ -33,5 +33,5 @@
         <origin xyz="0 0 0.063" rpy="0 0 0"/>
         <dynamics damping="0.0" friction="0.01"/>
-        <limit effort="12" velocity="12.5" lower="-1e16" upper="1e16"/>
+        <limit effort="7.77" velocity="19.305019" lower="-1e16" upper="1e16"/>
         <parent link="base_link"/>
         <child link="trigger"/>

Commit message: Update hero trigger transmission and block params.

File: urdf/hero/shooter.transmission.urdf.xacro (robot description, xacro)
@@ -4,5 +4,5 @@
         <type>transmission_interface/SimpleTransmission</type>
         <actuator name="trigger_joint_motor">
-            <mechanicalReduction>49.8083</mechanicalReduction>
+            <mechanicalReduction>69.544</mechanicalReduction>
         </actuator>
         <joint name="trigger_joint">

File: urdf/hero/shooter.urdf.xacro (robot description, xacro)
@@ -33,5 +33,5 @@
         <origin xyz="0 0 0.0223" rpy="0 0 0"/>
         <dynamics damping="0.0" friction="0.01"/>
-        <limit effort="6.99" velocity="35.758" lower="-1e16" upper="1e16"/>
+        <limit effort="18" velocity="13.5327" lower="-1e16" upper="1e16"/>
         <parent link="base_link"/>
         <child link="trigger"/>
