Commit message: Update standard3 urdf.

File: urdf/rmua/rmua.urdf.xacro (robot description, xacro)
@@ -13,4 +13,8 @@
         <xacro:include filename="$(find rm_description)/urdf/rmua/gimbal.urdf.xacro"/>
         <xacro:include filename="$(find rm_description)/urdf/rmua/gimbal.transmission.urdf.xacro"/>
+        <xacro:include filename="$(find rm_description)/urdf/common/imu.urdf.xacro"/>
+        <xacro:IMU connected_to="$(arg camera_optical_frame)" imu_name="gimbal_imu"
+                   xyz="0 -0.0255 -0.0348"
+                   rpy="1.57 0 0"/>
     </xacro:if>
     <xacro:if value="$(arg load_shooter)">

File: urdf/standard/gimbal.urdf.xacro (robot description, xacro)
@@ -35,8 +35,8 @@
     <link name="pitch">
         <inertial>
-            <mass value="0.652"/>
-            <origin xyz="0.033 0.000032 0.0384"/>
-            <inertia ixx="3.867378e-3" ixy="13867e-9" ixz="-395626e-9" iyy="8280849e-9"
-                     iyz="-36575e-9" izz="5849504e-9"/>
+            <mass value="0.644"/>
+            <origin xyz="0.029 0.000617 0.0376"/>
+            <inertia ixx="1.8216e-3" ixy="5.514e-6" ixz="1.58e-4" iyy="5.68e-3"
+                     iyz="-6.628e-6" izz="4.396e-3"/>
         </inertial>
         <visual>

File: urdf/standard3/standard3.urdf.xacro (robot description, xacro)
@@ -24,6 +24,6 @@
                                         camera_sim="false"/>
             <xacro:IMU connected_to="$(arg camera_optical_frame)" imu_name="gimbal_imu"
-                       xyz="0 -0.0255 -0.0348"
-                       rpy="1.57 0 0"/>
+                       xyz="0.04139555 0.06043143 -0.09599202"
+                       rpy="1.5064926 -0.0371791 -3.1361393"/>
             <xacro:if value="$(arg load_shooter)">
                 <xacro:include filename="$(find rm_description)/urdf/standard/shooter.urdf.xacro"/>
