Commit message: Add cover.stl and change base.stl.

File: urdf/standard/chassis.urdf.xacro (robot description, xacro)
@@ -2,6 +2,6 @@
     <xacro:include filename="$(find rm_description)/urdf/common/omni_wheel.urdf.xacro"/>
     <!-- https://upload.wikimedia.org/wikipedia/commons/5/52/Wheelbase_and_Track.png -->
-    <xacro:property name="chassis_radius" value="0.208"/>
-    <xacro:property name="wheel_offset_z" value="0.0"/>
+    <xacro:property name="chassis_radius" value="0.196"/>
+    <xacro:property name="wheel_offset_z" value="-0.04373"/>
     <xacro:macro name="chassis">
         <link name="base_link">

Commit message: Update standard3 urdf.

File: urdf/standard/chassis.urdf.xacro (robot description, xacro)
@@ -4,5 +4,5 @@
     <xacro:property name="chassis_radius" value="0.196"/>
     <xacro:property name="wheel_offset_z" value="-0.04373"/>
-    <xacro:macro name="chassis">
+    <xacro:macro name="chassis" params="roller_type">
         <link name="base_link">
             <inertial>
@@ -21,5 +21,5 @@
                 <origin xyz="0 0 0" rpy="0 0 0"/>
                 <geometry>
-                    <box size="0.580 0.500 0.050"/>
+                    <box size="0.392 0.392 0.2"/>
                 </geometry>
             </collision>
@@ -27,17 +27,17 @@
         <xacro:omni_wheel prefix="left_front" connected_to="base_link"
                           wheel_x_offset="${chassis_radius/sqrt(2)}" wheel_y_offset="${chassis_radius/sqrt(2)}"
-                          wheel_z_offset="${wheel_offset_z}" rotation_degree="${3*pi/4}"
+                          wheel_z_offset="${wheel_offset_z}" rotation_degree="${3*pi/4}" roller_type="${roller_type}"
         />
         <xacro:omni_wheel prefix="right_front" connected_to="base_link"
                           wheel_x_offset="${chassis_radius/sqrt(2)}" wheel_y_offset="${-chassis_radius/sqrt(2)}"
-                          wheel_z_offset="${wheel_offset_z}" rotation_degree="${pi/4}"
+                          wheel_z_offset="${wheel_offset_z}" rotation_degree="${pi/4}" roller_type="${roller_type}"
         />
         <xacro:omni_wheel prefix="left_back" connected_to="base_link"
                           wheel_x_offset="${-chassis_radius/sqrt(2)}" wheel_y_offset="${chassis_radius/sqrt(2)}"
-                          wheel_z_offset="${wheel_offset_z}" rotation_degree="${-3*pi/4}"
+                          wheel_z_offset="${wheel_offset_z}" rotation_degree="${-3*pi/4}" roller_type="${roller_type}"
         />
         <xacro:omni_wheel prefix="right_back" connected_to="base_link"
                           wheel_x_offset="${-chassis_radius/sqrt(2)}" wheel_y_offset="${-chassis_radius/sqrt(2)}"
-                          wheel_z_offset="${wheel_offset_z}" rotation_degree="${-pi/4}"
+                          wheel_z_offset="${wheel_offset_z}" rotation_degree="${-pi/4}" roller_type="${roller_type}"
         />
         <xacro:wheel_transmission prefix="left_front" mechanical_reduction="-19.2032"/>

File: urdf/standard/gimbal.urdf.xacro (robot description, xacro)
@@ -2,12 +2,12 @@
 <robot xmlns:xacro="http://www.ros.org/wiki/xacro">
     <xacro:property name="threshold" value="0.1"/>
-    <xacro:property name="pitch_lower_limit" value="-0.644"/>
-    <xacro:property name="pitch_upper_limit" value="0.467"/>
+    <xacro:property name="pitch_lower_limit" value="-0.627"/>
+    <xacro:property name="pitch_upper_limit" value="0.406"/>
     <link name="yaw">
         <inertial>
-            <mass value="2.497"/>
-            <origin xyz="0.014616 -0.007729 -0.004103"/>
-            <inertia ixx="1.039e-2" ixy="1.575e-3" ixz="-2.149e-3" iyy="1.181e-2"
-                     iyz="1.267e-3" izz="6.380e-3"/>
+            <mass value="0.2"/>
+            <origin xyz="-0.034 0.002 0.036"/>
+            <inertia ixx="4.878e-4" ixy="1.941e-5" ixz="2.44e-4" iyy="8.322e-4"
+                     iyz="-1.812e-5" izz="4.513e-4"/>
         </inertial>
         <visual>
@@ -23,44 +23,44 @@
             </geometry>
         </collision>
-        </link>
-        <joint name="yaw_joint" type="revolute">
-            <origin xyz="0 0 0.162"
-                    rpy="0 0 0"/>
-            <dynamics damping="0.0" friction="0.1"/>
-            <limit effort="1.2" velocity="31" lower="-1e10" upper="1e10"/>
-            <parent link="base_link"/>
-            <child link="yaw"/>
-            <axis xyz="0 0 1"/>
-        </joint>
-        <link name="pitch">
-            <inertial>
-                <mass value="2.244065"/>
-                <origin xyz="0.00115 -0.0128 0.0253"/>
-                <inertia ixx="9.63e-3" ixy="-4.829e-3" ixz="-1.382e-3" iyy="1.723e-2"
-                         iyz="-1.088e-3" izz="1.867e-2"/>
-            </inertial>
-            <visual>
-                <origin xyz="0 0 0" rpy="0 0 0"/>
-                <geometry>
-                    <mesh filename="package://rm_description/meshes/standard/pitch.stl" scale="0.001 0.001 0.001"/>
-                </geometry>
-            </visual>
-            <collision>
-                <origin xyz="0 0 0" rpy="0 0 0"/>
-                <geometry>
-                    <mesh filename="package://rm_description/meshes/standard/pitch.stl" scale="0.001 0.001 0.001"/>
-                </geometry>
-            </collision>
-        </link>
-        <joint name="pitch_joint" type="revolute">
-            <origin xyz="0 0 0.129897" rpy="0 0 0"/>
-            <dynamics damping="0.0" friction="0.1"/>
-            <limit effort="1.2" velocity="13.82" lower="${pitch_lower_limit}" upper="${pitch_upper_limit}"/>
-            <safety_controller k_position="100" k_velocity="0.1"
-                               soft_lower_limit="${pitch_lower_limit+threshold}"
-                               soft_upper_limit="${pitch_upper_limit-threshold}"/>
-            <parent link="yaw"/>
-            <child link="pitch"/>
-            <axis xyz="0 1 0 "/>
-        </joint>
+    </link>
+    <joint name="yaw_joint" type="revolute">
+        <origin xyz="0 0 0.162"
+                rpy="0 0 0"/>
+        <dynamics damping="0.0" friction="0.1"/>
+        <limit effort="1.2" velocity="31" lower="-1e10" upper="1e10"/>
+        <parent link="base_link"/>
+        <child link="yaw"/>
+        <axis xyz="0 0 1"/>
+    </joint>
+    <link name="pitch">
+        <inertial>
+            <mass value="1.145"/>
+            <origin xyz="0.033 0.000032 0.0384"/>
+            <inertia ixx="3.867378e-3" ixy="13867e-9" ixz="-395626e-9" iyy="8280849e-9"
+                     iyz="-36575e-9" izz="5849504e-9"/>
+        </inertial>
+        <visual>
+            <origin xyz="0 0 0" rpy="0 0 0"/>
+            <geometry>
+                <mesh filename="package://rm_description/meshes/standard/pitch.stl" scale="0.001 0.001 0.001"/>
+            </geometry>
+        </visual>
+        <collision>
+            <origin xyz="0 0 0" rpy="0 0 0"/>
+            <geometry>
+                <mesh filename="package://rm_description/meshes/standard/pitch.stl" scale="0.001 0.001 0.001"/>
+            </geometry>
+        </collision>
+    </link>
+    <joint name="pitch_joint" type="revolute">
+        <origin xyz="0 0 0.09" rpy="0 0 0"/>
+        <dynamics damping="0.0" friction="0.1"/>
+        <limit effort="3" velocity="13.82" lower="${pitch_lower_limit}" upper="${pitch_upper_limit}"/>
+        <safety_controller k_position="100" k_velocity="0.1"
+                           soft_lower_limit="${pitch_lower_limit+threshold}"
+                           soft_upper_limit="${pitch_upper_limit-threshold}"/>
+        <parent link="yaw"/>
+        <child link="pitch"/>
+        <axis xyz="0 1 0 "/>
+    </joint>
 </robot>

File: urdf/standard/shooter.urdf.xacro (robot description, xacro)
@@ -2,7 +2,7 @@
     <xacro:include filename="$(find rm_description)/urdf/common/friction.urdf.xacro"/>
     <!--    <xacro:include filename="$(find rm_description)/urdf/standard/gimbal.urdf.xacro"/>-->
-    <xacro:property name="wheel_offset_x" value="0.055"/>
+    <xacro:property name="wheel_offset_x" value="0.047"/>
     <xacro:property name="wheel_offset_y" value="0.0365"/>
-    <xacro:property name="wheel_offset_z" value="0.022375"/>
+    <xacro:property name="wheel_offset_z" value="0.02320"/>
     <xacro:friction_wheel prefixs="left" connected_to="pitch"
                           wheel_x_offset="${wheel_offset_x}" wheel_y_offset="${wheel_offset_y}"

File: urdf/standard3/gimbal.transmission.urdf.xacro (robot description, xacro)
@@ -7,5 +7,5 @@
         </actuator>
         <joint name="yaw_joint">
-            <offset>-3.644</offset>
+            <offset>-8.872</offset>
             <hardwareInterface>hardware_interface/EffortJointInterface</hardwareInterface>
         </joint>
@@ -14,8 +14,8 @@
         <type>transmission_interface/SimpleTransmission</type>
         <actuator name="pitch_joint_motor">
-            <mechanicalReduction>1</mechanicalReduction>
+            <mechanicalReduction>-11</mechanicalReduction>
         </actuator>
         <joint name="pitch_joint">
-            <offset>-2.268</offset>
+            <offset>0.483</offset>
             <hardwareInterface>hardware_interface/EffortJointInterface</hardwareInterface>
         </joint>

File: urdf/standard3/shooter.transmission.urdf.xacro (robot description, xacro)
@@ -8,4 +8,5 @@
         <joint name="trigger_joint">
             <hardwareInterface>hardware_interface/EffortJointInterface</hardwareInterface>
+            <offset>0.2</offset>
         </joint>
     </transmission>
@@ -13,5 +14,5 @@
         <type>transmission_interface/SimpleTransmission</type>
         <actuator name="left_friction_wheel_joint_motor">
-            <mechanicalReduction>1</mechanicalReduction>
+            <mechanicalReduction>-2.5</mechanicalReduction>
         </actuator>
         <joint name="left_friction_wheel_joint">

File: urdf/standard3/standard3.urdf.xacro (robot description, xacro)
@@ -6,8 +6,10 @@
     <xacro:arg name="camera_link" default="camera_link"/>
     <xacro:arg name="camera_optical_frame" default="camera_optical_frame"/>
+    <xacro:arg name="roller_type" default="simple"/>
     <xacro:arg name="use_simulation" default="true"/>
+    <xacro:arg name="roller_type" default="realistic"/>
     <xacro:if value="$(arg load_chassis)">
         <xacro:include filename="$(find rm_description)/urdf/standard/chassis.urdf.xacro"/>
-        <xacro:chassis/>
+        <xacro:chassis roller_type="$(arg roller_type)"/>
         <xacro:if value="$(arg load_gimbal)">
             <xacro:include filename="$(find rm_description)/urdf/standard/gimbal.urdf.xacro"/>
@@ -15,13 +17,13 @@
             <xacro:include filename="$(find rm_description)/urdf/common/camera.urdf.xacro"/>
             <xacro:include filename="$(find rm_description)/urdf/common/imu.urdf.xacro"/>
-            <xacro:camera_sensor xyz="0.01 0.05 0.06" rpy="0 0 0" frame_id="$(arg camera_link)" parent="pitch"
+            <xacro:camera_sensor xyz="0 0 0.0887" rpy="0 0 0" frame_id="$(arg camera_link)" parent="pitch"
                                  camera_sim="$(arg use_simulation)"/>
-            <xacro:camera_optical_frame xyz="0.03630540 0.02695002 0.07130801" rpy="1.5997419 0.1162527 1.5697408"
+            <xacro:camera_optical_frame xyz="0 0 0.0887" rpy="1.57 0 1.57"
                                         frame_id="$(arg camera_optical_frame)"
                                         parent="pitch"
-                                        camera_sim="$(arg use_simulation)"/>
+                                        camera_sim="false"/>
             <xacro:IMU connected_to="$(arg camera_optical_frame)" imu_name="gimbal_imu"
-                       xyz="-0.05766461 -0.00498878 -0.02889381"
-                       rpy="1.44537832 0.01314763 0.09321356"/>
+                       xyz="0 -0.0255 -0.0348"
+                       rpy="1.57 0 0"/>
             <xacro:if value="$(arg load_shooter)">
                 <xacro:include filename="$(find rm_description)/urdf/standard/shooter.urdf.xacro"/>

Commit message: Update standard3 urdf.

File: urdf/standard/chassis.urdf.xacro (robot description, xacro)
@@ -7,8 +7,8 @@
         <link name="base_link">
             <inertial>
-                <mass value="8.472226"/>
-                <origin xyz="0.009872  0.010973  0.001286"/>
-                <inertia ixx="1.131e-1" ixy="-4.480e-4" ixz="-9.581e-3" iyy="1.473e-1"
-                         iyz="3.352e-3" izz="2.048e-1"/>
+                <mass value="12.326"/>
+                <origin xyz="-0.000932  -0.000668  -0.01"/>
+                <inertia ixx="1.924e-1" ixy="-6.458e-4" ixz="5.951352e-3" iyy="2.473e-1"
+                         iyz="-7.22e-4" izz="3.187e-1"/>
             </inertial>
             <visual>

File: urdf/standard/gimbal.urdf.xacro (robot description, xacro)
@@ -56,5 +56,5 @@
         <origin xyz="0 0 0.09" rpy="0 0 0"/>
         <dynamics damping="0.0" friction="0.1"/>
-        <limit effort="3" velocity="13.82" lower="${pitch_lower_limit}" upper="${pitch_upper_limit}"/>
+        <limit effort="3." velocity="86" lower="${pitch_lower_limit}" upper="${pitch_upper_limit}"/>
         <safety_controller k_position="100" k_velocity="0.1"
                            soft_lower_limit="${pitch_lower_limit+threshold}"

File: urdf/standard3/gimbal.transmission.urdf.xacro (robot description, xacro)
@@ -7,5 +7,5 @@
         </actuator>
         <joint name="yaw_joint">
-            <offset>-8.872</offset>
+            <offset>-5.730</offset>
             <hardwareInterface>hardware_interface/EffortJointInterface</hardwareInterface>
         </joint>
