Commit message: Update standard3 urdf.

File: urdf/standard/gimbal.urdf.xacro (robot description, xacro)
@@ -2,6 +2,6 @@
 <robot xmlns:xacro="http://www.ros.org/wiki/xacro">
     <xacro:property name="threshold" value="0.1"/>
-    <xacro:property name="pitch_lower_limit" value="-0.583"/>
-    <xacro:property name="pitch_upper_limit" value="0.562"/>
+    <xacro:property name="pitch_lower_limit" value="-0.644"/>
+    <xacro:property name="pitch_upper_limit" value="0.467"/>
     <link name="yaw">
         <inertial>

File: urdf/standard3/gimbal.transmission.urdf.xacro (robot description, xacro)
@@ -7,5 +7,5 @@
         </actuator>
         <joint name="yaw_joint">
-            <offset>-3.689</offset>
+            <offset>-3.644</offset>
             <hardwareInterface>hardware_interface/EffortJointInterface</hardwareInterface>
         </joint>

Commit message: Correct the pitch's mass and shooter's reduction.

File: urdf/standard/gimbal.urdf.xacro (robot description, xacro)
@@ -35,5 +35,5 @@
     <link name="pitch">
         <inertial>
-            <mass value="1.145"/>
+            <mass value="0.652"/>
             <origin xyz="0.033 0.000032 0.0384"/>
             <inertia ixx="3.867378e-3" ixy="13867e-9" ixz="-395626e-9" iyy="8280849e-9"

File: urdf/standard3/shooter.transmission.urdf.xacro (robot description, xacro)
@@ -4,5 +4,5 @@
         <type>transmission_interface/SimpleTransmission</type>
         <actuator name="trigger_joint_motor">
-            <mechanicalReduction>-3</mechanicalReduction>
+            <mechanicalReduction>-2.5</mechanicalReduction>
         </actuator>
         <joint name="trigger_joint">
@@ -14,5 +14,5 @@
         <type>transmission_interface/SimpleTransmission</type>
         <actuator name="left_friction_wheel_joint_motor">
-            <mechanicalReduction>-2.5</mechanicalReduction>
+            <mechanicalReduction>1</mechanicalReduction>
         </actuator>
         <joint name="left_friction_wheel_joint">

Commit message: Update standard3 pitch limit.

File: urdf/standard/gimbal.urdf.xacro (robot description, xacro)
@@ -2,6 +2,6 @@
 <robot xmlns:xacro="http://www.ros.org/wiki/xacro">
     <xacro:property name="threshold" value="0.1"/>
-    <xacro:property name="pitch_lower_limit" value="-0.627"/>
-    <xacro:property name="pitch_upper_limit" value="0.406"/>
+    <xacro:property name="pitch_lower_limit" value="-0.6"/>
+    <xacro:property name="pitch_upper_limit" value="0.457"/>
     <link name="yaw">
         <inertial>

Commit message: Add supply_frame to standard3.

File: urdf/standard/gimbal.urdf.xacro (robot description, xacro)
@@ -33,4 +33,10 @@
         <axis xyz="0 0 1"/>
     </joint>
+    <link name="supply_frame"/>
+    <joint name="supply_joint" type="fixed">
+        <origin xyz="0 0 0" rpy="0 0 ${pi/2}"/>
+        <parent link="yaw"/>
+        <child link="supply_frame"/>
+    </joint>
     <link name="pitch">
         <inertial>

Commit message: Update standard urdf.

File: urdf/standard/gimbal.urdf.xacro (robot description, xacro)
@@ -1,5 +1,5 @@
 <?xml version="1.0" encoding="utf-8"?>
 <robot xmlns:xacro="http://www.ros.org/wiki/xacro">
-    <xacro:property name="threshold" value="0.1"/>
+    <xacro:property name="threshold" value="0.05"/>
     <xacro:property name="pitch_lower_limit" value="-0.6"/>
     <xacro:property name="pitch_upper_limit" value="0.457"/>
@@ -35,5 +35,5 @@
     <link name="supply_frame"/>
     <joint name="supply_joint" type="fixed">
-        <origin xyz="0 0 0" rpy="0 0 ${pi/2}"/>
+        <origin xyz="0 0 0" rpy="0 0 ${pi/3}"/>
         <parent link="yaw"/>
         <child link="supply_frame"/>

File: urdf/standard3/gimbal.transmission.urdf.xacro (robot description, xacro)
@@ -7,5 +7,5 @@
         </actuator>
         <joint name="yaw_joint">
-            <offset>-3.650552756</offset>
+            <offset>-0.502</offset>
             <hardwareInterface>hardware_interface/EffortJointInterface</hardwareInterface>
         </joint>

File: urdf/standard3/standard3.urdf.xacro (robot description, xacro)
@@ -25,6 +25,6 @@
                                         camera_sim="false"/>
             <xacro:IMU connected_to="$(arg camera_optical_frame)" imu_name="gimbal_imu"
-                       xyz="0 0.03 -0.1"
-                       rpy="1.575871 -0.0491724 3.1268903"/>
+                       xyz="0.00246956 0.04105199 -0.07160856"
+                       rpy="1.5487827 -0.0054278 -0.01"/>
             <xacro:if value="$(arg load_shooter)">
                 <xacro:include filename="$(find rm_description)/urdf/standard/shooter.urdf.xacro"/>

Commit message: Update standard urdf.

File: urdf/standard/gimbal.urdf.xacro (robot description, xacro)
@@ -1,6 +1,6 @@
 <?xml version="1.0" encoding="utf-8"?>
 <robot xmlns:xacro="http://www.ros.org/wiki/xacro">
-    <xacro:property name="threshold" value="0.05"/>
-    <xacro:property name="pitch_lower_limit" value="-0.6"/>
+    <xacro:property name="threshold" value="0.08"/>
+    <xacro:property name="pitch_lower_limit" value="-0.72"/>
     <xacro:property name="pitch_upper_limit" value="0.457"/>
     <link name="yaw">

File: urdf/standard3/standard3.urdf.xacro (robot description, xacro)
@@ -20,5 +20,5 @@
                                  camera_sim="$(arg use_simulation)"/>
             <xacro:camera_optical_frame xyz="0.06559775176285364 0.000187 0.08746327160978175"
-                                        rpy="-1.5729591 -0.0114965 -1.5698711"
+                                        rpy="-1.6547075 0.0527913 -1.5597212"
                                         frame_id="$(arg camera_optical_frame)"
                                         parent="pitch"
