Commit message: Update standard4 description.

File: urdf/standard4/chassis.urdf.xacro (robot description, xacro)
@@ -1,21 +1,19 @@
 <robot xmlns:xacro="http://www.ros.org/wiki/xacro">
-    <xacro:include filename="$(find rm_description)/urdf/common/swerve_drive.urdf.xacro"/>
+    <xacro:include filename="$(find rm_description)/urdf/common/omni_wheel.urdf.xacro"/>
     <!-- https://upload.wikimedia.org/wikipedia/commons/5/52/Wheelbase_and_Track.png -->
-    <xacro:property name="wheel_track" value="0.35"/>
-    <xacro:property name="wheel_base" value="0.35"/>
-    <xacro:property name="wheel_offset_z" value="0.06"/>
-    <xacro:macro name="chassis">
+    <xacro:property name="chassis_radius" value="0.196"/>
+    <xacro:property name="wheel_offset_z" value="-0.04373"/>
+    <xacro:macro name="chassis" params="roller_type">
         <link name="base_link">
             <inertial>
-                <mass value="1.737"/>
-                <origin xyz="0.000425  -0.000733  0.00762"/>
-                <inertia ixx="4.088e-2" ixy="9.103e-5" ixz="-1.697e-4" iyy="4.498e-2"
-                         iyz="6.472e-5" izz="8.107e-2"/>
+                <mass value="12.326"/>
+                <origin xyz="-0.000932  -0.000668  -0.01"/>
+                <inertia ixx="1.924e-1" ixy="-6.458e-4" ixz="5.951352e-3" iyy="2.473e-1"
+                         iyz="-7.22e-4" izz="3.187e-1"/>
             </inertial>
             <visual>
                 <origin xyz="0 0 0" rpy="0 0 0"/>
                 <geometry>
-                    <mesh filename="package://rm_description/meshes/standard/standard4_base.stl"
-                          scale="0.001 .001 0.001"/>
+                    <mesh filename="package://rm_description/meshes/standard/base.stl" scale="0.001 0.001 0.001"/>
                 </geometry>
             </visual>
@@ -23,25 +21,28 @@
                 <origin xyz="0 0 0" rpy="0 0 0"/>
                 <geometry>
-                    <mesh filename="package://rm_description/meshes/standard/standard4_base.stl"
-                          scale="0.001 0.001 0.001"/>
+                    <box size="0.392 0.392 0.2"/>
                 </geometry>
             </collision>
         </link>
-        <xacro:swerve_drive prefix="left_front" connected_to="base_link"
-                            wheel_x_offset="${wheel_track/2}" wheel_y_offset="${wheel_base/2}"
-                            wheel_z_offset="${wheel_offset_z}"/>
-        <xacro:swerve_drive prefix="right_front" connected_to="base_link"
-                            wheel_x_offset="${wheel_track/2}" wheel_y_offset="${-wheel_base/2}"
-                            wheel_z_offset="${wheel_offset_z}"/>
-        <xacro:swerve_drive prefix="left_back" connected_to="base_link"
-                            wheel_x_offset="${-wheel_track/2}" wheel_y_offset="${wheel_base/2}"
-                            wheel_z_offset="${wheel_offset_z}"/>
-        <xacro:swerve_drive prefix="right_back" connected_to="base_link"
-                            wheel_x_offset="${-wheel_track/2}" wheel_y_offset="${-wheel_base/2}"
-                            wheel_z_offset="${wheel_offset_z}"/>
-        <xacro:swerve_transmission prefix="left_front" wheel_reduction="13.733" pivot_offset="0"/>
-        <xacro:swerve_transmission prefix="right_front" wheel_reduction="-13.733" pivot_offset="1.861"/>
-        <xacro:swerve_transmission prefix="left_back" wheel_reduction="13.733" pivot_offset="1.585"/>
-        <xacro:swerve_transmission prefix="right_back" wheel_reduction="-13.733" pivot_offset="6.283"/>
+        <xacro:omni_wheel prefix="left_front" connected_to="base_link"
+                          wheel_x_offset="${chassis_radius/sqrt(2)}" wheel_y_offset="${chassis_radius/sqrt(2)}"
+                          wheel_z_offset="${wheel_offset_z}" rotation_degree="${3*pi/4}" roller_type="${roller_type}"
+        />
+        <xacro:omni_wheel prefix="right_front" connected_to="base_link"
+                          wheel_x_offset="${chassis_radius/sqrt(2)}" wheel_y_offset="${-chassis_radius/sqrt(2)}"
+                          wheel_z_offset="${wheel_offset_z}" rotation_degree="${pi/4}" roller_type="${roller_type}"
+        />
+        <xacro:omni_wheel prefix="left_back" connected_to="base_link"
+                          wheel_x_offset="${-chassis_radius/sqrt(2)}" wheel_y_offset="${chassis_radius/sqrt(2)}"
+                          wheel_z_offset="${wheel_offset_z}" rotation_degree="${-3*pi/4}" roller_type="${roller_type}"
+        />
+        <xacro:omni_wheel prefix="right_back" connected_to="base_link"
+                          wheel_x_offset="${-chassis_radius/sqrt(2)}" wheel_y_offset="${-chassis_radius/sqrt(2)}"
+                          wheel_z_offset="${wheel_offset_z}" rotation_degree="${-pi/4}" roller_type="${roller_type}"
+        />
+        <xacro:wheel_transmission prefix="left_front" mechanical_reduction="-13"/>
+        <xacro:wheel_transmission prefix="right_front" mechanical_reduction="-13"/>
+        <xacro:wheel_transmission prefix="left_back" mechanical_reduction="-13"/>
+        <xacro:wheel_transmission prefix="right_back" mechanical_reduction="-13"/>
     </xacro:macro>
 </robot>

File: urdf/standard4/gimbal.transmission.urdf.xacro (robot description, xacro)
@@ -7,5 +7,5 @@
         </actuator>
         <joint name="yaw_joint">
-            <offset>-3.829</offset>
+            <offset>-2.60425018</offset>
             <hardwareInterface>hardware_interface/EffortJointInterface</hardwareInterface>
         </joint>
@@ -14,8 +14,8 @@
         <type>transmission_interface/SimpleTransmission</type>
         <actuator name="pitch_joint_motor">
-            <mechanicalReduction>-1</mechanicalReduction>
+            <mechanicalReduction>-11</mechanicalReduction>
         </actuator>
         <joint name="pitch_joint">
-            <offset>1.737</offset>
+            <offset>0.483</offset>
             <hardwareInterface>hardware_interface/EffortJointInterface</hardwareInterface>
         </joint>
@@ -24,5 +24,5 @@
         <type>transmission_interface/SimpleTransmission</type>
         <actuator name="cover_joint_motor">
-            <mechanicalReduction>1</mechanicalReduction>
+            <mechanicalReduction>-1</mechanicalReduction>
         </actuator>
         <joint name="cover_joint">

File: urdf/standard4/standard4.urdf.xacro (robot description, xacro)
@@ -1,4 +1,4 @@
 <?xml version="1.0"?>
-<robot xmlns:xacro="http://www.ros.org/wiki/xacro" name="swerve">
+<robot xmlns:xacro="http://www.ros.org/wiki/xacro" name="standard3">
     <xacro:arg name="load_chassis" default="true"/>
     <xacro:arg name="load_gimbal" default="true"/>
@@ -6,22 +6,28 @@
     <xacro:arg name="camera_link" default="camera_link"/>
     <xacro:arg name="camera_optical_frame" default="camera_optical_frame"/>
+    <xacro:arg name="roller_type" default="simple"/>
     <xacro:arg name="use_simulation" default="true"/>
+    <xacro:arg name="roller_type" default="realistic"/>
     <xacro:if value="$(arg load_chassis)">
         <xacro:include filename="$(find rm_description)/urdf/standard4/chassis.urdf.xacro"/>
-        <xacro:chassis/>
+        <xacro:chassis roller_type="$(arg roller_type)"/>
         <xacro:if value="$(arg load_gimbal)">
             <xacro:include filename="$(find rm_description)/urdf/standard/gimbal.urdf.xacro"/>
             <xacro:include filename="$(find rm_description)/urdf/standard4/gimbal.transmission.urdf.xacro"/>
-            <!--            <xacro:include filename="$(find rm_description)/urdf/common/camera.urdf.xacro"/>-->
-            <!--            <xacro:camera_sensor xyz="0.127 0 -0.038" rpy="0 0 0" frame_id="$(arg camera_link)" parent="pitch"-->
-            <!--                                 camera_sim="$(arg use_simulation)"/>-->
-            <!--            <xacro:camera_optical_frame xyz="0.089 -0.004 -0.083" rpy="1.593 0.0 1.567"-->
-            <!--                                        frame_id="$(arg camera_optical_frame)" parent="pitch"-->
-            <!--                                        camera_sim="$(arg use_simulation)"/>-->
+            <xacro:include filename="$(find rm_description)/urdf/common/camera.urdf.xacro"/>
             <xacro:include filename="$(find rm_description)/urdf/common/imu.urdf.xacro"/>
-            <xacro:IMU connected_to="pitch" imu_name="gimbal_imu" xyz="0.08 0. 0.08" rpy="0 0 0"/>
+            <xacro:camera_sensor xyz="0 0 0.0887" rpy="0 0 0" frame_id="$(arg camera_link)" parent="pitch"
+                                 camera_sim="$(arg use_simulation)"/>
+            <xacro:camera_optical_frame xyz="0.05652213613351791 0.00334582754042001 0.08951459665737103"
+                                        rpy="-1.6276063 0.0179391 -1.5604531"
+                                        frame_id="$(arg camera_optical_frame)"
+                                        parent="pitch"
+                                        camera_sim="false"/>
+            <xacro:IMU connected_to="$(arg camera_optical_frame)" imu_name="gimbal_imu"
+                       xyz="0 0.03 -0.1"
+                       rpy="1.575871 -0.0491724 3.1268903"/>
             <xacro:if value="$(arg load_shooter)">
                 <xacro:include filename="$(find rm_description)/urdf/standard/shooter.urdf.xacro"/>
-                <xacro:include filename="$(find rm_description)/urdf/standard4/shooter.transmission.urdf.xacro"/>
+                <xacro:include filename="$(find rm_description)/urdf/standard3/shooter.transmission.urdf.xacro"/>
             </xacro:if>
         </xacro:if>
