Commit message: Update new engineer's urdf

File: urdf/engineer/arm.transmission.xacro (robot description, xacro)
@@ -4,11 +4,27 @@
         <!-- transmission -->
         <transmission name="trans_joint1">
-            <type>transmission_interface/SimpleTransmission</type>
-            <actuator name="joint1_motor">
-                <mechanicalReduction>71.75</mechanicalReduction>
+            <type>transmission_interface/MultiActuatorTransmission</type>
+            <actuator name="joint1_motor_left">
+                <role>main</role>
+                <mechanicalReduction>19.2032</mechanicalReduction>
+            </actuator>
+            <actuator name="joint1_motor_right">
+                <role>joint1_motor_right</role>
+                <mechanicalReduction>-19.2032</mechanicalReduction>
             </actuator>
             <joint name="joint1">
                 <hardwareInterface>hardware_interface/EffortJointInterface</hardwareInterface>
-                <offset>2.068</offset>
+                <offset>0</offset>
+                 <mechanicalReduction>-21.1677852</mechanicalReduction>
+            </joint>
+        </transmission>
+        <transmission name="trans_joint2">
+            <type>transmission_interface/SimpleTransmission</type>
+            <actuator name="joint2_motor">
+                <mechanicalReduction>3</mechanicalReduction>
+            </actuator>
+            <joint name="joint2">
+                <hardwareInterface>hardware_interface/EffortJointInterface</hardwareInterface>
+                <offset>-0.85</offset>
             </joint>
         </transmission>
@@ -43,34 +59,24 @@
             </joint>
         </transmission>
-        <xacro:unless value="${simulation}">
-            <transmission name="trans_joint2">
-                <type>transmission_interface/DoubleActuatorTransmission</type>
-                <actuator name="joint2_left_motor">
-                    <role>actuator1</role>
-                    <mechanicalReduction>3</mechanicalReduction>
-                </actuator>
-                <actuator name="joint2_right_motor">
-                    <role>actuator2</role>
-                    <mechanicalReduction>-3</mechanicalReduction>
-                </actuator>
-                <joint name="joint2">
-                    <hardwareInterface>hardware_interface/EffortJointInterface</hardwareInterface>
-                    <offset>-2.391650</offset>
-                    <mechanicalReduction>1</mechanicalReduction>
-                </joint>
-            </transmission>
-        </xacro:unless>
-        <xacro:if value="${simulation}">
-            <transmission name="trans_joint2">
-                <type>transmission_interface/SimpleTransmission</type>
-                <actuator name="joint2_motor">
-                    <mechanicalReduction>-3</mechanicalReduction>
-                </actuator>
-                <joint name="joint2">
-                    <hardwareInterface>hardware_interface/EffortJointInterface</hardwareInterface>
-                    <offset>-2.3764</offset>
-                </joint>
-            </transmission>
-        </xacro:if>
+        <transmission name="trans_joint6">
+            <type>transmission_interface/SimpleTransmission</type>
+            <actuator name="joint6_motor">
+                <mechanicalReduction>50.895</mechanicalReduction>
+            </actuator>
+            <joint name="joint6">
+                <hardwareInterface>hardware_interface/EffortJointInterface</hardwareInterface>
+                <offset>1.4378487</offset>
+            </joint>
+        </transmission>
+        <transmission name="trans_joint7">
+            <type>transmission_interface/SimpleTransmission</type>
+            <actuator name="joint7_motor">
+                <mechanicalReduction>50.895</mechanicalReduction>
+            </actuator>
+            <joint name="joint7">
+                <hardwareInterface>hardware_interface/EffortJointInterface</hardwareInterface>
+                <offset>1.4378487</offset>
+            </joint>
+        </transmission>
     </xacro:macro>
 </robot>

File: urdf/engineer/arm.urdf.xacro (robot description, xacro)
@@ -3,20 +3,24 @@
     <xacro:macro name="arm" params="connected_to">
         <xacro:property name="threshold" value="0.1"/>
-        <xacro:property name="joint1_lower_limit" value="-4.0246823"/>
-        <xacro:property name="joint1_upper_limit" value="2.05507607"/>
-        <xacro:property name="joint2_lower_limit" value="-2.378679831401"/>
-        <xacro:property name="joint2_upper_limit" value="-0.0989819625299"/>
-        <xacro:property name="joint3_lower_limit" value="-0.88921949"/>
-        <xacro:property name="joint3_upper_limit" value="2.535032168"/>
-        <xacro:property name="joint4_lower_limit" value="-0.2989008"/>
-        <xacro:property name="joint4_upper_limit" value="2.614725376878"/>
-        <xacro:property name="joint5_lower_limit" value="-4.27171178"/>
-        <xacro:property name="joint5_upper_limit" value="1.40800999"/>
+        <xacro:property name="joint1_lower_limit" value="0"/>
+        <xacro:property name="joint1_upper_limit" value="0.3"/>
+        <xacro:property name="joint2_lower_limit" value="-0.415"/>
+        <xacro:property name="joint2_upper_limit" value="0.42"/>
+        <xacro:property name="joint3_lower_limit" value="-0.22"/>
+        <xacro:property name="joint3_upper_limit" value="0.22"/>
+        <xacro:property name="joint4_lower_limit" value="-0.176"/>
+        <xacro:property name="joint4_upper_limit" value="0.176"/>
+        <xacro:property name="joint5_lower_limit" value="-3.132"/>
+        <xacro:property name="joint5_upper_limit" value="0.5916"/>
+        <xacro:property name="joint6_lower_limit" value="-4.785"/>
+        <xacro:property name="joint6_upper_limit" value="0.435"/>
+        <xacro:property name="joint7_lower_limit" value="-3.132"/>
+        <xacro:property name="joint7_upper_limit" value="3.132"/>
         <!--  link  -->
         <link name="link1">
             <inertial>
-                <mass value="1.768"/>
-                <origin xyz="-0.005 0.046 0.0"/>
-                <inertia ixx="9.816e-3" ixy="-2.523e-4" ixz="7.839e-6" iyy="9.203e-3" iyz="9.389e-5" izz="3.735e-3"/>
+                <mass value="2.933612"/>
+                <origin xyz="0.009153 -0.001831 0.028124"/>
+                <inertia ixx="1.232e-1" ixy="-5.053e-4" ixz="7.076e-4" iyy="6.280e-2" iyz="2.855e-4" izz="1.773e-1"/>
             </inertial>
             <visual>
@@ -27,38 +31,105 @@
             </visual>
             <collision>
-                <origin xyz="-0.022768 -0.000245 0.034512" rpy="0 0 0"/>
-                <geometry>
-                    <box size="0.088 0.142 0.106"/>
-                </geometry>
-            </collision>
-            <collision>
-                <origin xyz="0.001 -0.000245 0.04" rpy="1.57 0 0"/>
-                <geometry>
-                    <cylinder length="0.19" radius="0.047"/>
-                </geometry>
-            </collision>
-        </link>
-        <link name="link2">
-            <inertial>
-                <mass value="1.256"/>
-                <origin xyz="0.057 0.002 0"/>
-                <inertia ixx="1.678e-3" ixy="1.267e-5" ixz="-4.26e-7" iyy="3.761e-3" iyz="1.345e-6" izz="4.111e-3"/>
-            </inertial>
-            <visual>
-                <origin xyz="0 0 0" rpy="0 0 0"/>
-                <geometry>
-                    <mesh filename="package://rm_description/meshes/engineer/link2.stl" scale="0.001 0.001 0.001"/>
-                </geometry>
-            </visual>
-            <collision>
-                <origin xyz="0.072 0 0"/>
-                <geometry>
-                    <box size="0.215 0.096 0.075"/>
-                </geometry>
-            </collision>
-            <collision>
-                <origin xyz="0.165 0 0" rpy="1.5707963 0 0"/>
-                <geometry>
-                    <cylinder length="0.096" radius="0.047"/>
+                <origin xyz="0.004 0.1903 0.045" rpy="0 0 0"/>
+                <geometry>
+                    <box size="0.57 0.1356 0.045"/>
+                </geometry>
+            </collision>
+            <collision>
+                <origin xyz="0.004 -0.1903 0.045" rpy="0 0 0"/>
+                <geometry>
+                    <box size="0.57 0.1356 0.045"/>
+                </geometry>
+            </collision>
+            <collision>
+                <origin xyz="-0.185 0. 0.045" rpy="0 0 0"/>
+                <geometry>
+                    <box size="0.04 0.245 0.025"/>
+                </geometry>
+            </collision>
+            <collision>
+                <origin xyz="0. 0.237 -0.0175" rpy="0 0 0"/>
+                <geometry>
+                    <box size="0.29 0.042 0.08"/>
+                </geometry>
+            </collision>
+            <collision>
+                <origin xyz="0. -0.237 -0.0175" rpy="0 0 0"/>
+                <geometry>
+                    <box size="0.29 0.042 0.08"/>
+                </geometry>
+            </collision>
+            <collision>
+                <origin xyz="0.054 0.1815 0.003" rpy="0 0 0"/>
+                <geometry>
+                    <box size="0.086 0.069 0.039"/>
+                </geometry>
+            </collision>
+            <collision>
+                <origin xyz="0.054 -0.1815 0.003" rpy="0 0 0"/>
+                <geometry>
+                    <box size="0.086 0.069 0.039"/>
+                </geometry>
+            </collision>
+        </link>
+        <link name="link2_1">
+            <inertial>
+                <mass value="4.534716"/>
+                <origin xyz="-0.059835 -0.017665 -0.006662"/>
+                <inertia ixx="1.613e-1" ixy="4.286e-3" ixz="-3.019e-4" iyy="1.536e-1" iyz="-1.859e-3" izz="3.117e-1"/>
+            </inertial>
+            <visual>
+                <origin xyz="0 0 0" rpy="0 0 0"/>
+                <geometry>
+                    <mesh filename="package://rm_description/meshes/engineer/link2_1.stl" scale="0.001 0.001 0.001"/>
+                </geometry>
+            </visual>
+            <collision>
+                <origin xyz="0.01275 -0.1835 -0.011" rpy="0 0 0"/>
+                <geometry>
+                    <box size="0.5455 0.124 0.07"/>
+                </geometry>
+            </collision>
+            <collision>
+                <origin xyz="0.01275 0.1955 -0.011" rpy="0 0 0"/>
+                <geometry>
+                    <box size="0.5455 0.1 0.07"/>
+                </geometry>
+            </collision>
+            <collision>
+                <origin xyz="-0.283 -0.134 0.003" rpy="0 0 0"/>
+                <geometry>
+                    <box size="0.054 0.12 0.054"/>
+                </geometry>
+            </collision>
+            <collision>
+                <origin xyz="-0.283 0.134 0.003" rpy="0 0 0"/>
+                <geometry>
+                    <box size="0.054 0.12 0.054"/>
+                </geometry>
+            </collision>
+        </link>
+        <link name="link2_2">
+            <inertial>
+                <mass value="0.95156"/>
+                <origin xyz="-0.001706 -0.000534 0.016649"/>
+                <inertia ixx="1.271e-2" ixy="3.344217e-6" ixz="2.5531018e-5" iyy="8.153e-4" iyz="-3.333465e-6" izz="1.244e-2"/>
+            </inertial>
+            <visual>
+                <geometry>
+                    <mesh filename="package://rm_description/meshes/engineer/link2_2.stl" scale="0.001 0.001 0.001"/>
+                </geometry>
+                <origin xyz="0 0 0" rpy="0 0 0"/>
+            </visual>
+            <collision>
+                <origin xyz="-0.001 0 0.0015" rpy="0 0 0"/>
+                <geometry>
+                    <box size="0.114 0.475 0.031"/>
+                </geometry>
+            </collision>
+            <collision>
+                <origin xyz="0.015 0 0.044" rpy="0 0 0"/>
+                <geometry>
+                    <box size="0.082 0.122 0.054"/>
                 </geometry>
             </collision>
@@ -66,7 +137,7 @@
         <link name="link3">
             <inertial>
-                <mass value="1.139"/>
-                <origin xyz="0.081 -0.0 0.022"/>
-                <inertia ixx="9.633e-4" ixy="-2.836e-4" ixz="-5.244e-4" iyy="2.739e-3" iyz="-8.552e-5" izz="2.963e-3"/>
+                <mass value="0.739277"/>
+                <origin xyz="0.000853 -0.001219 0.003256"/>
+                <inertia ixx="9.950e-3" ixy="-1.181569e-6" ixz="1.1018936e-5" iyy="3.150e-4" iyz="3.7875649e-5" izz="9.892e-3"/>
             </inertial>
             <visual>
@@ -77,13 +148,13 @@
             </visual>
             <collision>
-                <origin xyz="0.006 0 0.007" rpy="0 0.8726 0"/>
-                <geometry>
-                    <box size="0.072 0.066 0.072"/>
-                </geometry>
-            </collision>
-            <collision>
-                <origin xyz="0.066 0 0.027"/>
-                <geometry>
-                    <box size="0.135 0.066 0.062"/>
+                <origin xyz="0. 0. 0.005" rpy="0 0 0"/>
+                <geometry>
+                    <box size="0.052 0.475 0.03"/>
+                </geometry>
+            </collision>
+            <collision>
+                <origin xyz="0. 0. 0.056" rpy="0 0 0"/>
+                <geometry>
+                    <box size="0.052 0.144 0.072"/>
                 </geometry>
             </collision>
@@ -91,7 +162,7 @@
         <link name="link4">
             <inertial>
-                <mass value="0.362"/>
-                <origin xyz="0.035 -0.027 0.06"/>
-                <inertia ixx="8.647e-4" ixy="-5.427e-5" ixz="-1.425e-4" iyy="8.477e-4" iyz="-2.555e-4" izz="5.668e-4"/>
+                <mass value="0.597915"/>
+                <origin xyz="0.0033 -0.051861 0.000004"/>
+                <inertia ixx="3.027e-3" ixy="-6.403167e-6" ixz="2.37196e-7" iyy="2.774e-4" iyz="-7.08963e-7" izz="3.084e-3"/>
             </inertial>
             <visual>
@@ -102,13 +173,7 @@
             </visual>
             <collision>
-                <origin xyz="0.02 -0.015 0.017" rpy="0 0.8028 0"/>
-                <geometry>
-                    <box size="0.0582 0.092 0.099"/>
-                </geometry>
-            </collision>
-            <collision>
-                <origin xyz="0.0347 -0.015 0.071"/>
-                <geometry>
-                    <box size="0.08 0.094 0.083"/>
+                <origin xyz="0.01475 -0.041 0." rpy="0 0 0"/>
+                <geometry>
+                    <box size="0.085 0.168 0.067"/>
                 </geometry>
             </collision>
@@ -116,7 +181,7 @@
         <link name="link5">
             <inertial>
-                <mass value="0.85"/>
-                <origin xyz="-0.061 0.0 0.0"/>
-                <inertia ixx="1.761e-4" ixy="6.99e-7" ixz="1.26e-7" iyy="5.874e-4" iyz="2.72e-7" izz="5.863e-4"/>
+                <mass value="0.705206"/>
+                <origin xyz="-0.030997 0.000129 0.038143"/>
+                <inertia ixx="4.444e-3" ixy="8.7593e-7" ixz="4.924e-4" iyy="5.629e-3" iyz="-7.662224e-6" izz="1.390e-3"/>
             </inertial>
             <visual>
@@ -126,61 +191,102 @@
                 </geometry>
             </visual>
-        </link>
-        <!--  joint  -->
-        <joint name="joint1" type="revolute">
-            <axis xyz="0 0 1"/>
-            <origin xyz="0.175 0 0.174" rpy="0 0 0"/>
-            <!--      limit not work while type="continuous"-->
-            <limit effort="20" velocity="13" lower="${joint1_lower_limit}" upper="${joint1_upper_limit}"/>
-            <safety_controller k_position="37.5" k_velocity="10"
-                               soft_lower_limit="${joint1_lower_limit+threshold}"
-                               soft_upper_limit="${joint1_upper_limit-threshold}"/>
-            <dynamics damping="0.0" friction="0.1"/>
+            <collision>
+                <origin xyz="-0.011 0. 0.103" rpy="0 0 0"/>
+                <geometry>
+                    <box size="0.056 0.054 0.26"/>
+                </geometry>
+            </collision>
+            <collision>
+                <origin xyz="-0.065 0. 0.2255" rpy="0 0 0"/>
+                <geometry>
+                    <box size="0.052 0.054 0.015"/>
+                </geometry>
+            </collision>
+            <collision>
+                <origin xyz="-0.0665 0. 0." rpy="0 0 0"/>
+                <geometry>
+                    <box size="0.055 0.054 0.054"/>
+                </geometry>
+            </collision>
+        </link>
+        <link name="link6">
+            <inertial>
+                <mass value="0.771338"/>
+                <origin xyz="0.04148 -0.000028 -0.028949"/>
+                <inertia ixx="2.206e-3" ixy="-3.0455e-8" ixz="-1.041e-4" iyy="4.988e-3" iyz="-4.58505e-7" izz="3.998e-3"/>
+            </inertial>
+            <visual>
+                <origin xyz="0 0 0" rpy="0 0 0"/>
+                <geometry>
+                    <mesh filename="package://rm_description/meshes/engineer/link6.stl" scale="0.001 0.001 0.001"/>
+                </geometry>
+            </visual>
+            <collision>
+                <origin xyz="0. 0. -0.04855" rpy="0 0 0"/>
+                <geometry>
+                    <box size="0.048 0.054 0.0971"/>
+                </geometry>
+            </collision>
+            <collision>
+                <origin xyz="0.0535 0. -0.0025" rpy="0 0 0"/>
+                <geometry>
+                    <box size="0.167 0.160 0.005"/>
+                </geometry>
+            </collision>
+            <collision>
+                <origin xyz="0.0995 0. 0.005" rpy="0 0 0"/>
+                <geometry>
+                    <box size="0.075 0.16 0.07"/>
+                </geometry>
+            </collision>
+        </link>
+        <joint name="joint1" type="prismatic">
             <parent link="${connected_to}"/>
             <child link="link1"/>
-        </joint>
-        <joint name="joint2" type="revolute">
+            <origin xyz="0 0 0.1375" rpy="0 0 0"/>
+            <axis xyz="0 0 1"/>
+            <limit lower="${joint1_lower_limit}" upper="${joint1_upper_limit}" velocity="0.1" effort="3000"/>
+        </joint>
+        <joint name="joint2" type="prismatic">
+            <parent link="link1"/>
+            <child link="link2_1"/>
+            <origin xyz="0. 0. 0.098707" rpy="0 0 0"/>
+            <axis xyz="1 0 0"/>
+            <limit lower="${joint2_lower_limit}" upper="${joint2_upper_limit}" velocity="0.1" effort="300"/>
+        </joint>
+        <joint name="joint3" type="prismatic">
+            <parent link="link2_1"/>
+            <child link="link2_2"/>
+            <origin xyz="0.022 0. 0.034" rpy="0 0 0"/>
+            <axis xyz="1 0 0"/>
+            <limit lower="${joint3_lower_limit}" upper="${joint3_upper_limit}" velocity="0.1" effort="300"/>
+        </joint>
+        <joint name="joint4" type="prismatic">
+            <parent link="link2_2"/>
+            <child link="link3"/>
+            <origin xyz="0. 0. 0.068" rpy="0 0 0"/>
             <axis xyz="0 1 0"/>
-            <origin xyz="0.005327 0 0.128" rpy="0 0 0"/>
-            <limit effort="60" velocity="10" lower="${joint2_lower_limit}" upper="${joint2_upper_limit}"/>
-            <safety_controller k_position="150" k_velocity="10"
-                               soft_lower_limit="${joint2_lower_limit+threshold}"
-                               soft_upper_limit="${joint2_upper_limit-threshold}"/>
-            <dynamics damping="0.0" friction="0.8"/>
-            <parent link="link1"/>
-            <child link="link2"/>
-        </joint>
-        <joint name="joint3" type="revolute">
-            <axis xyz="0 1 0"/>
-            <origin xyz="0.165 0 0" rpy="0 0 0"/>
-            <limit effort="30" velocity="10" lower="${joint3_lower_limit}" upper="${joint3_upper_limit}"/>
-            <safety_controller k_position="100" k_velocity="6"
-                               soft_lower_limit="${joint3_lower_limit+threshold}"
-                               soft_upper_limit="${joint3_upper_limit-threshold}"/>
-            <dynamics damping="0.0" friction="0.5"/>
-            <parent link="link2"/>
-            <child link="link3"/>
-        </joint>
-        <joint name="joint4" type="revolute">
-            <axis xyz="0 1 0"/>
-            <origin xyz="0.106 0 0.028"/>
-            <limit effort="18.53" velocity="13.5" lower="${joint4_lower_limit}" upper="${joint4_upper_limit}"/>
-            <safety_controller k_position="20" k_velocity="2.5"
-                               soft_lower_limit="${joint4_lower_limit+threshold}"
-                               soft_upper_limit="${joint4_upper_limit-threshold}"/>
-            <dynamics damping="0.0" friction="0.5"/>
+            <limit lower="${joint4_lower_limit}" upper="${joint4_upper_limit}" velocity="0.1" effort="300"/>
+        </joint>
+        <joint name="joint5" type="revolute">
             <parent link="link3"/>
             <child link="link4"/>
-        </joint>
-        <joint name="joint5" type="revolute">
+            <origin xyz="0. 0. 0.069" rpy="0 0 0"/>
+            <axis xyz="0 1 0"/>
+            <limit lower="${joint5_lower_limit}" upper="${joint5_upper_limit}" velocity="0.1" effort="300"/>
+        </joint>
+        <joint name="joint6" type="revolute">
+            <parent link="link4"/>
+            <child link="link5"/>
+            <origin xyz="0.06925 0. 0" rpy="0 0 0"/>
             <axis xyz="1 0 0"/>
-            <origin xyz="0.097 0 0.055"/>
-            <limit effort="13" velocity="18" lower="${joint5_lower_limit}" upper="${joint5_upper_limit}"/>
-            <safety_controller k_position="20" k_velocity="5"
-                               soft_lower_limit="${joint5_lower_limit+threshold}"
-                               soft_upper_limit="${joint5_upper_limit-threshold}"/>
-            <dynamics damping="0.0" friction="0.5"/>
-            <parent link="link4"/>z
-            <child link="link5"/>
+            <limit lower="${joint6_lower_limit}" upper="${joint6_upper_limit}" velocity="0.1" effort="300"/>
+        </joint>
+        <joint name="joint7" type="revolute">
+            <parent link="link5"/>
+            <child link="link6"/>
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