Commit message: Update new engineer's urdf

File: urdf/engineer/chassis.urdf.xacro (robot description, xacro)
@@ -1,176 +1,71 @@
 <robot xmlns:xacro="http://www.ros.org/wiki/xacro" name="chassis">
-    <xacro:include filename="$(find rm_description)/urdf/common/mecanum_wheel.urdf.xacro"/>
-    <!-- https://upload.wikimedia.org/wikipedia/commons/5/52/Wheelbase_and_Track.png -->
-    <xacro:property name="wheel_front" value="0.134874"/>
-    <xacro:property name="wheel_back" value="-0.134874"/>
-    <xacro:property name="wheel_right" value="-0.2448"/>
-    <xacro:property name="wheel_left" value="0.2448"/>
-    <xacro:property name="wheel_offset_z" value="-0.029928"/>
-    <xacro:property name="wheel_joint_damping" value="1.0"/>
-    <xacro:property name="wheel_joint_friction" value="1.0"/>
     <xacro:macro name="chassis" params="roller_type">
         <link name="base_link">
             <inertial>
-                <mass value="13"/>
-                <origin xyz="-0.063 -0.010 -0.027"/>
-                <inertia ixx="4.302e-2" ixy="7.618e-4" ixz="6.881e-3" iyy="3.95e-2"
-                         iyz="-1.841e-4" izz="7.25e-2"/>
+                <mass value="6.78192"/>
+                <origin xyz="-0.010204 -0.005935 0.071865"/>
+                <inertia ixx="4.319e-1" ixy="-3.679e-4" ixz="9.099e-3" iyy="2.759e-1" iyz="-2.652e-3" izz="3.458e-1"/>
             </inertial>
             <visual>
                 <origin xyz="0 0 0" rpy="0 0 0"/>
                 <geometry>
-                    <mesh filename="package://rm_description/meshes/engineer/base.stl" scale="0.001 .001 0.001"/>
+                    <mesh filename="package://rm_description/meshes/engineer/base_link.stl" scale="0.001 0.001 0.001"/>
                 </geometry>
             </visual>
             <collision>
-                <origin xyz="-0.125 0. 0.06" rpy="0 0 0"/>
+                <origin xyz="0. 0. 0.04" rpy="0 0 0"/>
                 <geometry>
-                    <box size="0.25 0.596 0.169"/>
+                    <box size="0.43 0.602 0.08"/>
                 </geometry>
             </collision>
             <collision>
-                <origin xyz="0.15 -0.15 0.015" rpy="0 0 0"/>
+                <origin xyz="0.125 0.2645 0.3" rpy="0 0 0"/>
                 <geometry>
-                    <box size="0.255 0.29 0.06"/>
+                    <box size="0.04 0.043 0.44"/>
                 </geometry>
             </collision>
             <collision>
-                <origin xyz="0.15 0.144 0.015" rpy="0 0 0"/>
+                <origin xyz="0.125 -0.2645 0.3" rpy="0 0 0"/>
                 <geometry>
-                    <box size="0.255 0.29 0.06"/>
+                    <box size="0.04 0.043 0.44"/>
                 </geometry>
             </collision>
             <collision>
-                <origin xyz="0.16 0. 0.1" rpy="0 0 0"/>
+                <origin xyz="-0.0965 0.272 0.3" rpy="0 0 0"/>
                 <geometry>
-                    <box size="0.12 0.2 0.1"/>
+                    <box size="0.097 0.058 0.44"/>
                 </geometry>
             </collision>
             <collision>
-                <origin xyz="-0.038526 0.245965 0.224" rpy="0 0 -0.507"/>
+                <origin xyz="-0.0965 -0.272 0.3" rpy="0 0 0"/>
                 <geometry>
-                    <box size="0.08 0.024213 0.448"/>
+                    <box size="0.097 0.058 0.44"/>
                 </geometry>
             </collision>
             <collision>
-                <origin xyz="-0.160269 0.184128 0.284" rpy="0 0 1.0646508"/>
+                <origin xyz="-0.013 0.274 0.1055" rpy="0 0 0"/>
                 <geometry>
-                    <box size="0.08 0.0217 0.3033"/>
+                    <box size="0.07 0.054 0.051"/>
                 </geometry>
             </collision>
             <collision>
-                <origin xyz="-0.148196 0.0485 0.224" rpy="0 0 -0.507"/>
+                <origin xyz="-0.013 -0.274 0.1055" rpy="0 0 0"/>
                 <geometry>
-                    <box size="0.08 0.03 0.448"/>
+                    <box size="0.07 0.054 0.051"/>
                 </geometry>
             </collision>
             <collision>
-                <origin xyz="0.019028 0.084742 0.269" rpy="0 0 1.0646508"/>
+                <origin xyz="0.0285 0.2685 0.5" rpy="0 0 0"/>
                 <geometry>
-                    <box size="0.080 0.003 0.250"/>
+                    <box size="0.153 0.035 0.040"/>
+                </geometry>
+            </collision>
+            <collision>
+                <origin xyz="0.0285 -0.2685 0.5" rpy="0 0 0"/>
+                <geometry>
+                    <box size="0.153 0.035 0.040"/>
                 </geometry>
             </collision>
         </link>
-        <link name="stone_platform">
-            <inertial>
-                <mass value="0.073"/>
-                <origin xyz="-0.037 -0.005 0.009"/>
-                <inertia ixx="5.874e-4" ixy="-2.845e-4" ixz="1.882e-5" iyy="2.133e-4" iyz="2.682e-5" izz="7.780e-4"/>
-            </inertial>
-            <visual>
-                <origin xyz="0 0 0" rpy="0 0 0"/>
-                <geometry>
-                    <mesh filename="package://rm_description/meshes/engineer/stone_platform.stl"
-                          scale="0.001 0.001 0.001"/>
-                </geometry>
-            </visual>
-            <collision>
-                <origin xyz="0.0 0.0 0.0" rpy="0 0.0 0"/>
-                <geometry>
-                    <box size="0.106 0.105 0.002"/>
-                </geometry>
-            </collision>
-            <collision>
-                <origin xyz="-0.08 -0.09 0.02" rpy="0 0 1.0646508"/>
-                <geometry>
-                    <box size="0.03 0.06 0.05"/>
-                </geometry>
-            </collision>
-        </link>
-        <link name="card">
-            <inertial>
-                <mass value="0.26"/>
-                <origin xyz="-0.071 -0.006 0.003"/>
-                <inertia ixx="1.078e-3" ixy="6.486e-5" ixz="1.454e-5" iyy="1.142e-4" iyz="5.143e-6" izz="2.215e-3"/>
-            </inertial>
-            <visual>
-                <origin xyz="0 0 0" rpy="0 0 0"/>
-                <geometry>
-                    <mesh filename="package://rm_description/meshes/engineer/card.stl" scale="0.001 0.001 0.001"/>
-                </geometry>
-            </visual>
-            <collision>
-                <origin xyz="-0.08 0 0" rpy="0 0.0 0"/>
-                <geometry>
-                    <box size="0.253 0.151 0.011"/>
-                </geometry>
-            </collision>
-        </link>
-        <joint name="card_joint" type="prismatic">
-            <axis xyz="1 0 0"/>
-            <origin xyz="0.15205 0. -0.07"/>
-            <limit effort="20.0" velocity="1.0" lower="0" upper="0.281"/>
-            <dynamics damping="0.0" friction="0.1"/>
-            <parent link="base_link"/>
-            <child link="card"/>
-        </joint>
-        <joint name="stone_platform_joint" type="prismatic">
-            <axis xyz="0 0 1"/>
-            <origin xyz="-0.0706 0.134 0.114"/>
-            <limit effort="20.0" velocity="1.0" lower="0" upper="0.19"/>
-            <dynamics damping="0.0" friction="0.1"/>
-            <parent link="base_link"/>
-            <child link="stone_platform"/>
-        </joint>
-        <transmission name="trans_stone_platform_joint">
-            <type>transmission_interface/SimpleTransmission</type>
-            <actuator name="stone_platform_joint_motor">
-                <mechanicalReduction>49.97</mechanicalReduction>
-            </actuator>
-            <joint name="stone_platform_joint">
-                <hardwareInterface>hardware_interface/EffortJointInterface</hardwareInterface>
-                <offset>0</offset>
-            </joint>
-        </transmission>
-        <transmission name="trans_card_joint">
-            <type>transmission_interface/SimpleTransmission</type>
-            <actuator name="card_joint_motor">
-                <mechanicalReduction>49.97</mechanicalReduction>
-            </actuator>
-            <joint name="card_joint">
-                <hardwareInterface>hardware_interface/EffortJointInterface</hardwareInterface>
-                <offset>0</offset>
-            </joint>
-        </transmission>
-        <xacro:mecanum_wheel prefix="left_front" connected_to="base_link"
-                             wheel_x_offset="${wheel_front}" wheel_y_offset="${wheel_left}"
-                             wheel_z_offset="${wheel_offset_z}"
-                             reflect="1" roller_type="${roller_type}"/>
-        <xacro:mecanum_wheel prefix="right_front" connected_to="base_link"
-                             wheel_x_offset="${wheel_front}" wheel_y_offset="${wheel_right}"
-                             wheel_z_offset="${wheel_offset_z}"
-                             reflect="-1" roller_type="${roller_type}"/>
-        <xacro:mecanum_wheel prefix="left_back" connected_to="base_link"
-                             wheel_x_offset="${wheel_back}" wheel_y_offset="${wheel_left}"
-                             wheel_z_offset="${wheel_offset_z}"
-                             reflect="-1" roller_type="${roller_type}"/>
-        <xacro:mecanum_wheel prefix="right_back" connected_to="base_link"
-                             wheel_x_offset="${wheel_back}" wheel_y_offset="${wheel_right}"
-                             wheel_z_offset="${wheel_offset_z}"
-                             reflect="1" roller_type="${roller_type}"/>
-        <xacro:wheel_transmission prefix="left_front" mechanical_reduction="19.2032"/>
-        <xacro:wheel_transmission prefix="right_front" mechanical_reduction="-19.2032"/>
-        <xacro:wheel_transmission prefix="left_back" mechanical_reduction="19.2032"/>
-        <xacro:wheel_transmission prefix="right_back" mechanical_reduction="-19.2032"/>
     </xacro:macro>
 </robot>

Commit message: # This is a combination of 11 commits. # This is the 1st commit message:
Update new engineer's urdf

# This is the commit message #2:

Apply MultiActuatorTransmission on joint123

# This is the commit message #3:

Update the stl and limits of link456

# This is the commit message #4:

Update joint's pid and modify transmission

# This is the commit message #5:

Modify the arm's pid and vel effort limits

# This is the commit message #6:

Update offset and mechicalreduction

# This is the commit message #7:

Update the joint's limit

# This is the commit message #8:

Update the joint's limit and max vel effort

# This is the commit message #9:

Add mini link and the controllers of mini jooint

# This is the commit message #10:

Add hold card and chassis's urdf

# This is the commit message #11:

Add card and drag's link , add the params "simulation"

File: urdf/engineer/arm.transmission.xacro (robot description, xacro)
@@ -6,9 +6,19 @@
             <type>transmission_interface/SimpleTransmission</type>
             <actuator name="joint1_motor">
-                <mechanicalReduction>71.75</mechanicalReduction>
+                <mechanicalReduction>406.489213</mechanicalReduction>
             </actuator>
             <joint name="joint1">
                 <hardwareInterface>hardware_interface/EffortJointInterface</hardwareInterface>
-                <offset>2.068</offset>
+                <offset>0</offset>
+            </joint>
+        </transmission>
+        <transmission name="trans_joint2">
+            <type>transmission_interface/SimpleTransmission</type>
+            <actuator name="joint2_motor">
+                <mechanicalReduction>476.977368</mechanicalReduction>
+            </actuator>
+            <joint name="joint2">
+                <hardwareInterface>hardware_interface/EffortJointInterface</hardwareInterface>
+                <offset>0</offset>
             </joint>
         </transmission>
@@ -16,9 +26,9 @@
             <type>transmission_interface/SimpleTransmission</type>
             <actuator name="joint3_motor">
-                <mechanicalReduction>3</mechanicalReduction>
+                <mechanicalReduction>1036.0854</mechanicalReduction>
             </actuator>
             <joint name="joint3">
                 <hardwareInterface>hardware_interface/EffortJointInterface</hardwareInterface>
-                <offset>-0.85</offset>
+                <offset>0</offset>
             </joint>
         </transmission>
@@ -26,9 +36,9 @@
             <type>transmission_interface/SimpleTransmission</type>
             <actuator name="joint4_motor">
-                <mechanicalReduction>-71.165</mechanicalReduction>
+                <mechanicalReduction>328.29</mechanicalReduction>
             </actuator>
             <joint name="joint4">
                 <hardwareInterface>hardware_interface/EffortJointInterface</hardwareInterface>
-                <offset>-0.334978036</offset>
+                <offset>0.3415371896670</offset>
             </joint>
         </transmission>
@@ -40,37 +50,59 @@
             <joint name="joint5">
                 <hardwareInterface>hardware_interface/EffortJointInterface</hardwareInterface>
-                <offset>1.4378487</offset>
+                <offset>0</offset>
+            </joint>
+        </transmission>
+        <transmission name="trans_joint6">
+            <type>transmission_interface/SimpleTransmission</type>
+            <actuator name="joint6_motor">
+                <mechanicalReduction>50.895</mechanicalReduction>
+            </actuator>
+            <joint name="joint6">
+                <hardwareInterface>hardware_interface/EffortJointInterface</hardwareInterface>
+                <offset>0</offset>
+            </joint>
+        </transmission>
+        <transmission name="trans_joint7">
+            <type>transmission_interface/SimpleTransmission</type>
+            <actuator name="joint7_motor">
+                <mechanicalReduction>19.2032</mechanicalReduction>
+            </actuator>
+            <joint name="joint7">
+                <hardwareInterface>hardware_interface/EffortJointInterface</hardwareInterface>
+                <offset>0</offset>
             </joint>
         </transmission>
         <xacro:unless value="${simulation}">
-            <transmission name="trans_joint2">
-                <type>transmission_interface/DoubleActuatorTransmission</type>
-                <actuator name="joint2_left_motor">
-                    <role>actuator1</role>
-                    <mechanicalReduction>3</mechanicalReduction>
+            <transmission name="trans_joint1_mime">
+                <type>transmission_interface/SimpleTransmission</type>
+                <actuator name="joint1_mime_motor">
+                    <mechanicalReduction>-406.489213</mechanicalReduction>
                 </actuator>
-                <actuator name="joint2_right_motor">
-                    <role>actuator2</role>
-                    <mechanicalReduction>-3</mechanicalReduction>
+                <joint name="joint1_mime">
+                    <hardwareInterface>hardware_interface/EffortJointInterface</hardwareInterface>
+                    <offset>0</offset>
+                </joint>
+            </transmission>
+            <transmission name="trans_joint2_mime">
+                <type>transmission_interface/SimpleTransmission</type>
+                <actuator name="joint2_mime_motor">
+                    <mechanicalReduction>-476.977368</mechanicalReduction>
                 </actuator>
-                <joint name="joint2">
+                <joint name="joint2_mime">
                     <hardwareInterface>hardware_interface/EffortJointInterface</hardwareInterface>
-                    <offset>-2.391650</offset>
-                    <mechanicalReduction>1</mechanicalReduction>
+                    <offset>0</offset>
+                </joint>
+            </transmission>
+            <transmission name="trans_joint3_mime">
+                <type>transmission_interface/SimpleTransmission</type>
+                <actuator name="joint3_mime_motor">
+                    <mechanicalReduction>-1036.0854</mechanicalReduction>
+                </actuator>
+                <joint name="joint3_mime">
+                    <hardwareInterface>hardware_interface/EffortJointInterface</hardwareInterface>
+                    <offset>0</offset>
                 </joint>
             </transmission>
         </xacro:unless>
-        <xacro:if value="${simulation}">
-            <transmission name="trans_joint2">
-                <type>transmission_interface/SimpleTransmission</type>
-                <actuator name="joint2_motor">
-                    <mechanicalReduction>-3</mechanicalReduction>
-                </actuator>
-                <joint name="joint2">
-                    <hardwareInterface>hardware_interface/EffortJointInterface</hardwareInterface>
-                    <offset>-2.3764</offset>
-                </joint>
-            </transmission>
-        </xacro:if>
     </xacro:macro>
 </robot>
