Commit message: Modify the arm's pid and vel effort limits

File: urdf/engineer/arm.transmission.xacro (robot description, xacro)
@@ -15,6 +15,6 @@
             <joint name="joint1">
                 <hardwareInterface>hardware_interface/EffortJointInterface</hardwareInterface>
-                <offset>0.</offset>
-                 <mechanicalReduction>21.1677852</mechanicalReduction>
+                <offset>-0.003720897933201</offset>
+                <mechanicalReduction>21.1677852</mechanicalReduction>
             </joint>
         </transmission>
@@ -31,8 +31,8 @@
             <joint name="joint2">
                 <hardwareInterface>hardware_interface/EffortJointInterface</hardwareInterface>
-                <offset>0.</offset>
-                <mechanicalReduction>21.739</mechanicalReduction>
+                <offset>-0.215818870427</offset>
+                <mechanicalReduction>24.8516</mechanicalReduction>
             </joint>
-        </transmission>`
+        </transmission>
         <transmission name="trans_joint3">
             <type>transmission_interface/MultiActuatorTransmission</type>
@@ -47,6 +47,6 @@
             <joint name="joint3">
                 <hardwareInterface>hardware_interface/EffortJointInterface</hardwareInterface>
-                <offset>0.</offset>
-                <mechanicalReduction>-56.920</mechanicalReduction>
+                <offset>-0.209661752078</offset>
+                <mechanicalReduction>-53.9811</mechanicalReduction>
             </joint>
         </transmission>
@@ -58,5 +58,5 @@
             <joint name="joint4">
                 <hardwareInterface>hardware_interface/EffortJointInterface</hardwareInterface>
-                <offset>0.</offset>
+                <offset>0.3373738684</offset>
             </joint>
         </transmission>
@@ -68,5 +68,5 @@
             <joint name="joint5">
                 <hardwareInterface>hardware_interface/EffortJointInterface</hardwareInterface>
-                <offset>0.</offset>
+                <offset>0.0087707703</offset>
             </joint>
         </transmission>
@@ -78,5 +78,5 @@
             <joint name="joint6">
                 <hardwareInterface>hardware_interface/EffortJointInterface</hardwareInterface>
-                <offset>0</offset>
+                <offset>0.53846803044</offset>
             </joint>
         </transmission>
@@ -88,5 +88,5 @@
             <joint name="joint7">
                 <hardwareInterface>hardware_interface/EffortJointInterface</hardwareInterface>
-                <offset>0</offset>
+                <offset>3.941673196467</offset>
             </joint>
         </transmission>

File: urdf/engineer/arm.urdf.xacro (robot description, xacro)
@@ -5,16 +5,16 @@
         <xacro:property name="joint1_lower_limit" value="0"/>
         <xacro:property name="joint1_upper_limit" value="0.3"/>
-        <xacro:property name="joint2_lower_limit" value="-0.415"/>
-        <xacro:property name="joint2_upper_limit" value="0.42"/>
-        <xacro:property name="joint3_lower_limit" value="-0.22"/>
-        <xacro:property name="joint3_upper_limit" value="0.22"/>
-        <xacro:property name="joint4_lower_limit" value="-0.176"/>
-        <xacro:property name="joint4_upper_limit" value="0.176"/>
-        <xacro:property name="joint5_lower_limit" value="-3.141"/>
-        <xacro:property name="joint5_upper_limit" value="0."/>
-        <xacro:property name="joint6_lower_limit" value="-4.176"/>
-        <xacro:property name="joint6_upper_limit" value="0.783"/>
-        <xacro:property name="joint7_lower_limit" value="-3.915"/>
-        <xacro:property name="joint7_upper_limit" value="0.783"/>
+        <xacro:property name="joint2_lower_limit" value="-0.253350256769"/>
+        <xacro:property name="joint2_upper_limit" value="0.385167154"/>
+        <xacro:property name="joint3_lower_limit" value="-0.229388728029366"/>
+        <xacro:property name="joint3_upper_limit" value="0.281850996668"/>
+        <xacro:property name="joint4_lower_limit" value="-0.40983099899072"/>
+        <xacro:property name="joint4_upper_limit" value="0.43667063"/>
+        <xacro:property name="joint5_lower_limit" value="-3.42203741234"/>
+        <xacro:property name="joint5_upper_limit" value="0.047983045788"/>
+        <xacro:property name="joint6_lower_limit" value="-4.327149605070"/>
+        <xacro:property name="joint6_upper_limit" value="0.593107173715"/>
+        <xacro:property name="joint7_lower_limit" value="-1.507979833"/>
+        <xacro:property name="joint7_upper_limit" value="4.03879746213"/>
         <!--  link  -->
         <link name="link1">
@@ -114,5 +114,6 @@
                 <mass value="0.95156"/>
                 <origin xyz="-0.001706 -0.000534 0.016649"/>
-                <inertia ixx="1.271e-2" ixy="3.344217e-6" ixz="2.5531018e-5" iyy="8.153e-4" iyz="-3.333465e-6" izz="1.244e-2"/>
+                <inertia ixx="1.271e-2" ixy="3.344217e-6" ixz="2.5531018e-5" iyy="8.153e-4" iyz="-3.333465e-6"
+                         izz="1.244e-2"/>
             </inertial>
             <visual>
@@ -139,5 +140,6 @@
                 <mass value="0.739277"/>
                 <origin xyz="0.000853 -0.001219 0.003256"/>
-                <inertia ixx="9.950e-3" ixy="-1.181569e-6" ixz="1.1018936e-5" iyy="3.150e-4" iyz="3.7875649e-5" izz="9.892e-3"/>
+                <inertia ixx="9.950e-3" ixy="-1.181569e-6" ixz="1.1018936e-5" iyy="3.150e-4" iyz="3.7875649e-5"
+                         izz="9.892e-3"/>
             </inertial>
             <visual>
@@ -164,5 +166,6 @@
                 <mass value="0.597915"/>
                 <origin xyz="0.0033 -0.051861 0.000004"/>
-                <inertia ixx="3.027e-3" ixy="-6.403167e-6" ixz="2.37196e-7" iyy="2.774e-4" iyz="-7.08963e-7" izz="3.084e-3"/>
+                <inertia ixx="3.027e-3" ixy="-6.403167e-6" ixz="2.37196e-7" iyy="2.774e-4" iyz="-7.08963e-7"
+                         izz="3.084e-3"/>
             </inertial>
             <visual>
@@ -183,5 +186,6 @@
                 <mass value="0.705206"/>
                 <origin xyz="-0.030997 0.000129 0.038143"/>
-                <inertia ixx="4.444e-3" ixy="8.7593e-7" ixz="4.924e-4" iyy="5.629e-3" iyz="-7.662224e-6" izz="1.390e-3"/>
+                <inertia ixx="4.444e-3" ixy="8.7593e-7" ixz="4.924e-4" iyy="5.629e-3" iyz="-7.662224e-6"
+                         izz="1.390e-3"/>
             </inertial>
             <visual>
@@ -214,5 +218,6 @@
                 <mass value="0.771338"/>
                 <origin xyz="0.04148 -0.000028 -0.028949"/>
-                <inertia ixx="2.206e-3" ixy="-3.0455e-8" ixz="-1.041e-4" iyy="4.988e-3" iyz="-4.58505e-7" izz="3.998e-3"/>
+                <inertia ixx="2.206e-3" ixy="-3.0455e-8" ixz="-1.041e-4" iyy="4.988e-3" iyz="-4.58505e-7"
+                         izz="3.998e-3"/>
             </inertial>
             <visual>
@@ -246,5 +251,6 @@
             <origin xyz="0 0 0.1375" rpy="0 0 0"/>
             <axis xyz="0 0 1"/>
-            <limit lower="${joint1_lower_limit}" upper="${joint1_upper_limit}" velocity="0.1" effort="3000"/>
+            <limit lower="${joint1_lower_limit}" upper="${joint1_upper_limit}" velocity="100"
+                   effort="10"/>
         </joint>
         <joint name="joint2" type="prismatic">
@@ -253,5 +259,6 @@
             <origin xyz="0. 0. 0.098707" rpy="0 0 0"/>
             <axis xyz="1 0 0"/>
-            <limit lower="${joint2_lower_limit}" upper="${joint2_upper_limit}" velocity="0.1" effort="300"/>
+            <limit lower="${joint2_lower_limit}" upper="${joint2_upper_limit}" velocity="100"
+                   effort="10"/>
         </joint>
         <joint name="joint3" type="prismatic">
@@ -260,5 +267,5 @@
             <origin xyz="0.022 0. 0.034" rpy="0 0 0"/>
             <axis xyz="1 0 0"/>
-            <limit lower="${joint3_lower_limit}" upper="${joint3_upper_limit}" velocity="0.1" effort="300"/>
+            <limit lower="${joint3_lower_limit}" upper="${joint3_upper_limit}" velocity="100" effort="10"/>
         </joint>
         <joint name="joint4" type="prismatic">
@@ -267,5 +274,6 @@
             <origin xyz="0. 0. 0.068" rpy="0 0 0"/>
             <axis xyz="0 1 0"/>
-            <limit lower="${joint4_lower_limit}" upper="${joint4_upper_limit}" velocity="0.1" effort="300"/>
+            <limit lower="${joint4_lower_limit}" upper="${joint4_upper_limit}" velocity="100"
+                   effort="10"/>
         </joint>
         <joint name="joint5" type="revolute">
@@ -274,5 +282,6 @@
             <origin xyz="0. 0. 0.069" rpy="0 0 0"/>
             <axis xyz="0 1 0"/>
-            <limit lower="${joint5_lower_limit}" upper="${joint5_upper_limit}" velocity="0.1" effort="300"/>
+            <limit lower="${joint5_lower_limit}" upper="${joint5_upper_limit}" velocity="100"
+                   effort="10"/>
         </joint>
         <joint name="joint6" type="revolute">
@@ -281,5 +290,6 @@
             <origin xyz="0.06925 0. 0" rpy="0 0 0"/>
             <axis xyz="1 0 0"/>
-            <limit lower="${joint6_lower_limit}" upper="${joint6_upper_limit}" velocity="0.1" effort="300"/>
+            <limit lower="${joint6_lower_limit}" upper="${joint6_upper_limit}" velocity="100"
+                   effort="10"/>
         </joint>
         <joint name="joint7" type="revolute">
@@ -288,5 +298,6 @@
             <origin xyz="-0.06925 0 0.255" rpy="0 0 0"/>
             <axis xyz="0 0 1"/>
-            <limit lower="${joint7_lower_limit}" upper="${joint7_upper_limit}" velocity="0.1" effort="300"/>
+            <limit lower="${joint7_lower_limit}" upper="${joint7_upper_limit}" velocity="100"
+                   effort="10"/>
         </joint>
     </xacro:macro>

Commit message: Add mini link and the controllers of mini jooint

File: urdf/engineer/arm.transmission.xacro (robot description, xacro)
@@ -4,49 +4,61 @@
         <!-- transmission -->
         <transmission name="trans_joint1">
-            <type>transmission_interface/MultiActuatorTransmission</type>
-            <actuator name="joint1_motor_left">
-                <role>main</role>
-                <mechanicalReduction>19.2032</mechanicalReduction>
-            </actuator>
-            <actuator name="joint1_motor_right">
-                <role>joint1_motor_right</role>
-                <mechanicalReduction>-19.2032</mechanicalReduction>
+            <type>transmission_interface/SimpleTransmission</type>
+            <actuator name="joint1_motor">
+                <mechanicalReduction>406.489213</mechanicalReduction>
             </actuator>
             <joint name="joint1">
                 <hardwareInterface>hardware_interface/EffortJointInterface</hardwareInterface>
-                <offset>0.603732671447</offset>
-                <mechanicalReduction>21.1677852</mechanicalReduction>
+                <offset>0</offset>
+            </joint>
+        </transmission>
+        <transmission name="trans_joint1_mime">
+            <type>transmission_interface/SimpleTransmission</type>
+            <actuator name="mime_joint1_motor">
+                <mechanicalReduction>-406.489213</mechanicalReduction>
+            </actuator>
+            <joint name="joint1_mime">
+                <hardwareInterface>hardware_interface/EffortJointInterface</hardwareInterface>
+                <offset>0</offset>
             </joint>
         </transmission>
         <transmission name="trans_joint2">
-            <type>transmission_interface/MultiActuatorTransmission</type>
-            <actuator name="joint2_motor_left">
-                <role>main</role>
-                <mechanicalReduction>19.2032</mechanicalReduction>
-            </actuator>
-            <actuator name="joint2_motor_right">
-                <role>joint1_motor_right</role>
-                <mechanicalReduction>-19.2032</mechanicalReduction>
+            <type>transmission_interface/SimpleTransmission</type>
+            <actuator name="joint2_motor">
+                <mechanicalReduction>476.977368</mechanicalReduction>
             </actuator>
             <joint name="joint2">
                 <hardwareInterface>hardware_interface/EffortJointInterface</hardwareInterface>
-                <offset>0.344452874</offset>
-                <mechanicalReduction>24.8384315</mechanicalReduction>
+                <offset>0</offset>
+            </joint>
+        </transmission>
+        <transmission name="trans_joint2_mime">
+            <type>transmission_interface/SimpleTransmission</type>
+            <actuator name="mime_joint2_motor">
+                <mechanicalReduction>-476.977368</mechanicalReduction>
+            </actuator>
+            <joint name="joint2_mime">
+                <hardwareInterface>hardware_interface/EffortJointInterface</hardwareInterface>
+                <offset>0</offset>
             </joint>
         </transmission>
         <transmission name="trans_joint3">
-            <type>transmission_interface/MultiActuatorTransmission</type>
-            <actuator name="joint3_motor_left">
-                <role>main</role>
-                <mechanicalReduction>19.2032</mechanicalReduction>
-            </actuator>
-            <actuator name="joint3_motor_right">
-                <role>joint1_motor_right</role>
-                <mechanicalReduction>-19.2032</mechanicalReduction>
+            <type>transmission_interface/SimpleTransmission</type>
+            <actuator name="joint3_motor">
+                <mechanicalReduction>1036.0854</mechanicalReduction>
             </actuator>
             <joint name="joint3">
                 <hardwareInterface>hardware_interface/EffortJointInterface</hardwareInterface>
-                <offset>0.23650836764</offset>
-                <mechanicalReduction>-53.9537441</mechanicalReduction>
+                <offset>0</offset>
+            </joint>
+        </transmission>
+        <transmission name="trans_joint3_mime">
+            <type>transmission_interface/SimpleTransmission</type>
+            <actuator name="mime_joint3_motor">
+                <mechanicalReduction>-1036.0854</mechanicalReduction>
+            </actuator>
+            <joint name="joint3_mime">
+                <hardwareInterface>hardware_interface/EffortJointInterface</hardwareInterface>
+                <offset>0</offset>
             </joint>
         </transmission>
@@ -68,5 +80,5 @@
             <joint name="joint5">
                 <hardwareInterface>hardware_interface/EffortJointInterface</hardwareInterface>
-                <offset>0.02522726716</offset>
+                <offset>0</offset>
             </joint>
         </transmission>
@@ -78,5 +90,5 @@
             <joint name="joint6">
                 <hardwareInterface>hardware_interface/EffortJointInterface</hardwareInterface>
-                <offset>0.83257516659</offset>
+                <offset>0</offset>
             </joint>
         </transmission>
@@ -88,5 +100,5 @@
             <joint name="joint7">
                 <hardwareInterface>hardware_interface/EffortJointInterface</hardwareInterface>
-                <offset>3.983091759055</offset>
+                <offset>0</offset>
             </joint>
         </transmission>

File: urdf/engineer/arm.urdf.xacro (robot description, xacro)
@@ -73,4 +73,23 @@
             </collision>
         </link>
+        <link name="link1_mime">
+            <inertial>
+                <mass value="0.1"/>
+                <origin xyz="0. 0. 0."/>
+                <inertia ixx="0" ixy="0" ixz="0" iyy="0" iyz="0" izz="0"/>
+            </inertial>
+            <visual>
+                <origin xyz="0. 0.237 -0.0175" rpy="0 0 0"/>
+                <geometry>
+                    <box size="0.01 0.01 0.1"/>
+                </geometry>
+            </visual>
+            <collision>
+                <origin xyz="0. 0 0." rpy="0 0 0"/>
+                <geometry>
+                    <box size="0. 0. 0."/>
+                </geometry>
+            </collision>
+        </link>
         <link name="link2_1">
             <inertial>
@@ -107,4 +126,23 @@
                 <geometry>
                     <box size="0.054 0.12 0.054"/>
+                </geometry>
+            </collision>
+        </link>
+        <link name="link2_1_mime">
+            <inertial>
+                <mass value="0.1"/>
+                <origin xyz="0. 0. 0."/>
+                <inertia ixx="0" ixy="0" ixz="0" iyy="0" iyz="0" izz="0"/>
+            </inertial>
+            <visual>
+                <origin xyz="-0.283 0.134 0.003" rpy="0 0 0"/>
+                <geometry>
+                    <box size="0.1 0.01 0.01"/>
+                </geometry>
+            </visual>
+            <collision>
+                <origin xyz="0. 0 0." rpy="0 0 0"/>
+                <geometry>
+                    <box size="0. 0. 0."/>
                 </geometry>
             </collision>
@@ -133,4 +171,23 @@
                 <geometry>
                     <box size="0.082 0.122 0.054"/>
+                </geometry>
+            </collision>
+        </link>
+        <link name="link2_2_mime">
+            <inertial>
+                <mass value="0.1"/>
+                <origin xyz="0. 0. 0."/>
+                <inertia ixx="0" ixy="0" ixz="0" iyy="0" iyz="0" izz="0"/>
+            </inertial>
+            <visual>
+                <origin xyz="-0.001 0 0.0015" rpy="0 0 0"/>
+                <geometry>
+                    <box size="0.1 0.01 0.01"/>
+                </geometry>
+            </visual>
+            <collision>
+                <origin xyz="0. 0 0." rpy="0 0 0"/>
+                <geometry>
+                    <box size="0. 0. 0."/>
                 </geometry>
             </collision>
@@ -253,4 +310,11 @@
             <limit lower="${joint1_lower_limit}" upper="${joint1_upper_limit}" velocity="1" effort="200"/>
         </joint>
+        <joint name="joint1_mime" type="prismatic">
+            <parent link="${connected_to}"/>
+            <child link="link1_mime"/>z
+            <origin xyz="0 0 0.1375" rpy="0 0 0"/>
+            <axis xyz="0 0 1"/>
+            <limit lower="${joint1_lower_limit}" upper="${joint1_upper_limit}" velocity="1" effort="200"/>
+        </joint>
         <joint name="joint2" type="prismatic">
             <parent link="link1"/>
@@ -260,7 +324,21 @@
             <limit lower="${joint2_lower_limit}" upper="${joint2_upper_limit}" velocity="1" effort="200"/>
         </joint>
+        <joint name="joint2_mime" type="prismatic">
+            <parent link="link1"/>
+            <child link="link2_1_mime"/>
+            <origin xyz="0. 0. 0.098707" rpy="0 0 0"/>
+            <axis xyz="1 0 0"/>
+            <limit lower="${joint2_lower_limit}" upper="${joint2_upper_limit}" velocity="1" effort="200"/>
+        </joint>
         <joint name="joint3" type="prismatic">
             <parent link="link2_1"/>
             <child link="link2_2"/>
+            <origin xyz="0.022 0. 0.034" rpy="0 0 0"/>
+            <axis xyz="1 0 0"/>
+            <limit lower="${joint3_lower_limit}" upper="${joint3_upper_limit}" velocity="1" effort="200"/>
+        </joint>
+        <joint name="joint3_mime" type="prismatic">
+            <parent link="link2_1"/>
+            <child link="link2_2_mime"/>
             <origin xyz="0.022 0. 0.034" rpy="0 0 0"/>
             <axis xyz="1 0 0"/>

File: urdf/engineer/chassis.urdf.xacro (robot description, xacro)
@@ -20,25 +20,25 @@
             </collision>
             <collision>
-                <origin xyz="0.125 0.2645 0.3" rpy="0 0 0"/>
+                <origin xyz="0.125 0.26625 0.3" rpy="0 0 0"/>
                 <geometry>
-                    <box size="0.04 0.043 0.44"/>
+                    <box size="0.04 0.0395 0.44"/>
                 </geometry>
             </collision>
             <collision>
-                <origin xyz="0.125 -0.2645 0.3" rpy="0 0 0"/>
+                <origin xyz="0.125 -0.26625 0.3" rpy="0 0 0"/>
                 <geometry>
-                    <box size="0.04 0.043 0.44"/>
+                    <box size="0.04 0.0395 0.44"/>
                 </geometry>
             </collision>
             <collision>
-                <origin xyz="-0.0965 0.272 0.3" rpy="0 0 0"/>
+                <origin xyz="-0.0965 0.27375 0.3" rpy="0 0 0"/>
                 <geometry>
-                    <box size="0.097 0.058 0.44"/>
+                    <box size="0.097 0.0545 0.44"/>
                 </geometry>
             </collision>
             <collision>
-                <origin xyz="-0.0965 -0.272 0.3" rpy="0 0 0"/>
+                <origin xyz="-0.0965 -0.27375 0.3" rpy="0 0 0"/>
                 <geometry>
-                    <box size="0.097 0.058 0.44"/>
+                    <box size="0.097 0.0545 0.44"/>
                 </geometry>
             </collision>
