Commit message: Add card and drag's link , add the params "simulation"

File: urdf/engineer/arm.transmission.xacro (robot description, xacro)
@@ -13,14 +13,4 @@
             </joint>
         </transmission>
-        <transmission name="trans_joint1_mime">
-            <type>transmission_interface/SimpleTransmission</type>
-            <actuator name="mime_joint1_motor">
-                <mechanicalReduction>-406.489213</mechanicalReduction>
-            </actuator>
-            <joint name="joint1_mime">
-                <hardwareInterface>hardware_interface/EffortJointInterface</hardwareInterface>
-                <offset>0</offset>
-            </joint>
-        </transmission>
         <transmission name="trans_joint2">
             <type>transmission_interface/SimpleTransmission</type>
@@ -33,14 +23,4 @@
             </joint>
         </transmission>
-        <transmission name="trans_joint2_mime">
-            <type>transmission_interface/SimpleTransmission</type>
-            <actuator name="mime_joint2_motor">
-                <mechanicalReduction>-476.977368</mechanicalReduction>
-            </actuator>
-            <joint name="joint2_mime">
-                <hardwareInterface>hardware_interface/EffortJointInterface</hardwareInterface>
-                <offset>0</offset>
-            </joint>
-        </transmission>
         <transmission name="trans_joint3">
             <type>transmission_interface/SimpleTransmission</type>
@@ -49,14 +29,4 @@
             </actuator>
             <joint name="joint3">
-                <hardwareInterface>hardware_interface/EffortJointInterface</hardwareInterface>
-                <offset>0</offset>
-            </joint>
-        </transmission>
-        <transmission name="trans_joint3_mime">
-            <type>transmission_interface/SimpleTransmission</type>
-            <actuator name="mime_joint3_motor">
-                <mechanicalReduction>-1036.0854</mechanicalReduction>
-            </actuator>
-            <joint name="joint3_mime">
                 <hardwareInterface>hardware_interface/EffortJointInterface</hardwareInterface>
                 <offset>0</offset>
@@ -103,4 +73,36 @@
             </joint>
         </transmission>
+        <xacro:unless value="${simulation}">
+            <transmission name="trans_joint1_mime">
+                <type>transmission_interface/SimpleTransmission</type>
+                <actuator name="joint1_mime_motor">
+                    <mechanicalReduction>-406.489213</mechanicalReduction>
+                </actuator>
+                <joint name="joint1_mime">
+                    <hardwareInterface>hardware_interface/EffortJointInterface</hardwareInterface>
+                    <offset>0</offset>
+                </joint>
+            </transmission>
+            <transmission name="trans_joint2_mime">
+                <type>transmission_interface/SimpleTransmission</type>
+                <actuator name="joint2_mime_motor">
+                    <mechanicalReduction>-476.977368</mechanicalReduction>
+                </actuator>
+                <joint name="joint2_mime">
+                    <hardwareInterface>hardware_interface/EffortJointInterface</hardwareInterface>
+                    <offset>0</offset>
+                </joint>
+            </transmission>
+            <transmission name="trans_joint3_mime">
+                <type>transmission_interface/SimpleTransmission</type>
+                <actuator name="joint3_mime_motor">
+                    <mechanicalReduction>-1036.0854</mechanicalReduction>
+                </actuator>
+                <joint name="joint3_mime">
+                    <hardwareInterface>hardware_interface/EffortJointInterface</hardwareInterface>
+                    <offset>0</offset>
+                </joint>
+            </transmission>
+        </xacro:unless>
     </xacro:macro>
 </robot>

File: urdf/engineer/arm.urdf.xacro (robot description, xacro)
@@ -1,5 +1,5 @@
 <?xml version="1.0" encoding="utf-8"?>
 <robot xmlns:xacro="http://www.ros.org/wiki/xacro" name="arm">
-    <xacro:macro name="arm" params="connected_to">
+    <xacro:macro name="arm" params="connected_to simulation">
         <xacro:property name="threshold" value="0.1"/>
         <xacro:property name="joint1_lower_limit" value="0.0005736069829"/>
@@ -73,23 +73,4 @@
             </collision>
         </link>
-        <link name="link1_mime">
-            <inertial>
-                <mass value="0.1"/>
-                <origin xyz="0. 0. 0."/>
-                <inertia ixx="0" ixy="0" ixz="0" iyy="0" iyz="0" izz="0"/>
-            </inertial>
-            <visual>
-                <origin xyz="0. 0.237 -0.0175" rpy="0 0 0"/>
-                <geometry>
-                    <box size="0.01 0.01 0.1"/>
-                </geometry>
-            </visual>
-            <collision>
-                <origin xyz="0. 0 0." rpy="0 0 0"/>
-                <geometry>
-                    <box size="0. 0. 0."/>
-                </geometry>
-            </collision>
-        </link>
         <link name="link2_1">
             <inertial>
@@ -126,23 +107,4 @@
                 <geometry>
                     <box size="0.054 0.12 0.054"/>
-                </geometry>
-            </collision>
-        </link>
-        <link name="link2_1_mime">
-            <inertial>
-                <mass value="0.1"/>
-                <origin xyz="0. 0. 0."/>
-                <inertia ixx="0" ixy="0" ixz="0" iyy="0" iyz="0" izz="0"/>
-            </inertial>
-            <visual>
-                <origin xyz="-0.283 0.134 0.003" rpy="0 0 0"/>
-                <geometry>
-                    <box size="0.1 0.01 0.01"/>
-                </geometry>
-            </visual>
-            <collision>
-                <origin xyz="0. 0 0." rpy="0 0 0"/>
-                <geometry>
-                    <box size="0. 0. 0."/>
                 </geometry>
             </collision>
@@ -171,23 +133,4 @@
                 <geometry>
                     <box size="0.082 0.122 0.054"/>
-                </geometry>
-            </collision>
-        </link>
-        <link name="link2_2_mime">
-            <inertial>
-                <mass value="0.1"/>
-                <origin xyz="0. 0. 0."/>
-                <inertia ixx="0" ixy="0" ixz="0" iyy="0" iyz="0" izz="0"/>
-            </inertial>
-            <visual>
-                <origin xyz="-0.001 0 0.0015" rpy="0 0 0"/>
-                <geometry>
-                    <box size="0.1 0.01 0.01"/>
-                </geometry>
-            </visual>
-            <collision>
-                <origin xyz="0. 0 0." rpy="0 0 0"/>
-                <geometry>
-                    <box size="0. 0. 0."/>
                 </geometry>
             </collision>
@@ -310,11 +253,4 @@
             <limit lower="${joint1_lower_limit}" upper="${joint1_upper_limit}" velocity="1" effort="200"/>
         </joint>
-        <joint name="joint1_mime" type="prismatic">
-            <parent link="${connected_to}"/>
-            <child link="link1_mime"/>z
-            <origin xyz="0 0 0.1375" rpy="0 0 0"/>
-            <axis xyz="0 0 1"/>
-            <limit lower="${joint1_lower_limit}" upper="${joint1_upper_limit}" velocity="1" effort="200"/>
-        </joint>
         <joint name="joint2" type="prismatic">
             <parent link="link1"/>
@@ -324,11 +260,4 @@
             <limit lower="${joint2_lower_limit}" upper="${joint2_upper_limit}" velocity="1" effort="200"/>
         </joint>
-        <joint name="joint2_mime" type="prismatic">
-            <parent link="link1"/>
-            <child link="link2_1_mime"/>
-            <origin xyz="0. 0. 0.098707" rpy="0 0 0"/>
-            <axis xyz="1 0 0"/>
-            <limit lower="${joint2_lower_limit}" upper="${joint2_upper_limit}" velocity="1" effort="200"/>
-        </joint>
         <joint name="joint3" type="prismatic">
             <parent link="link2_1"/>
@@ -338,11 +267,4 @@
             <limit lower="${joint3_lower_limit}" upper="${joint3_upper_limit}" velocity="1" effort="200"/>
         </joint>
-        <joint name="joint3_mime" type="prismatic">
-            <parent link="link2_1"/>
-            <child link="link2_2_mime"/>
-            <origin xyz="0.022 0. 0.034" rpy="0 0 0"/>
-            <axis xyz="1 0 0"/>
-            <limit lower="${joint3_lower_limit}" upper="${joint3_upper_limit}" velocity="1" effort="200"/>
-        </joint>
         <joint name="joint4" type="prismatic">
             <parent link="link2_2"/>
@@ -373,4 +295,84 @@
             <limit lower="${joint7_lower_limit}" upper="${joint7_upper_limit}" velocity="10" effort="200"/>
         </joint>
+        <xacro:unless value="${simulation}">
+            <link name="link1_mime">
+                <inertial>
+                    <mass value="0.1"/>
+                    <origin xyz="0. 0. 0."/>
+                    <inertia ixx="0" ixy="0" ixz="0" iyy="0" iyz="0" izz="0"/>
+                </inertial>
+                <visual>
+                    <origin xyz="0. 0.237 -0.0175" rpy="0 0 0"/>
+                    <geometry>
+                        <box size="0.01 0.01 0.1"/>
+                    </geometry>
+                </visual>
+                <collision>
+                    <origin xyz="0. 0 0." rpy="0 0 0"/>
+                    <geometry>
+                        <box size="0. 0. 0."/>
+                    </geometry>
+                </collision>
+            </link>
+            <link name="link2_1_mime">
+                <inertial>
+                    <mass value="0.1"/>
+                    <origin xyz="0. 0. 0."/>
+                    <inertia ixx="0" ixy="0" ixz="0" iyy="0" iyz="0" izz="0"/>
+                </inertial>
+                <visual>
+                    <origin xyz="-0.283 0.134 0.003" rpy="0 0 0"/>
+                    <geometry>
+                        <box size="0.1 0.01 0.01"/>
+                    </geometry>
+                </visual>
+                <collision>
+                    <origin xyz="0. 0 0." rpy="0 0 0"/>
+                    <geometry>
+                        <box size="0. 0. 0."/>
+                    </geometry>
+                </collision>
+            </link>
+            <link name="link2_2_mime">
+                <inertial>
+                    <mass value="0.1"/>
+                    <origin xyz="0. 0. 0."/>
+                    <inertia ixx="0" ixy="0" ixz="0" iyy="0" iyz="0" izz="0"/>
+                </inertial>
+                <visual>
+                    <origin xyz="-0.001 0 0.0015" rpy="0 0 0"/>
+                    <geometry>
+                        <box size="0.1 0.01 0.01"/>
+                    </geometry>
+                </visual>
+                <collision>
+                    <origin xyz="0. 0 0." rpy="0 0 0"/>
+                    <geometry>
+                        <box size="0. 0. 0."/>
+                    </geometry>
+                </collision>
+            </link>
+            <joint name="joint1_mime" type="prismatic">
+                <parent link="${connected_to}"/>
+                <child link="link1_mime"/>z
+                <origin xyz="0 0 0.1375" rpy="0 0 0"/>
+                <axis xyz="0 0 1"/>
+                <limit lower="${joint1_lower_limit}" upper="${joint1_upper_limit}" velocity="1" effort="200"/>
+            </joint>
+            <joint name="joint2_mime" type="prismatic">
+                <parent link="link1"/>
+                <child link="link2_1_mime"/>
+                <origin xyz="0. 0. 0.098707" rpy="0 0 0"/>
+                <axis xyz="1 0 0"/>
+                <limit lower="${joint2_lower_limit}" upper="${joint2_upper_limit}" velocity="1" effort="200"/>
+            </joint>
+            <joint name="joint3_mime" type="prismatic">
+                <parent link="link2_1"/>
+                <child link="link2_2_mime"/>
+                <origin xyz="0.022 0. 0.034" rpy="0 0 0"/>
+                <axis xyz="1 0 0"/>
+                <limit lower="${joint3_lower_limit}" upper="${joint3_upper_limit}" velocity="1" effort="200"/>
+            </joint>
+        </xacro:unless>
     </xacro:macro>
 </robot>

File: urdf/engineer/chassis.urdf.xacro (robot description, xacro)
@@ -1,81 +1,10 @@
 <robot xmlns:xacro="http://www.ros.org/wiki/xacro" name="chassis">
     <xacro:include filename="$(find rm_description)/urdf/common/swerve_drive.urdf.xacro"/>
-    <xacro:property name="wheel_track" value="0.416152"/>
-    <xacro:property name="wheel_base" value="0.416152"/>
+    <!-- https://upload.wikimedia.org/wikipedia/commons/5/52/Wheelbase_and_Track.png -->
+    <xacro:property name="wheel_track" value="0.42"/>
+    <xacro:property name="wheel_base" value="0.42"/>
     <xacro:property name="wheel_offset_z" value="0.06"/>
-    <xacro:macro name="chassis" params="roller_type">
+    <xacro:macro name="chassis">
         <link name="base_link">
-            <inertial>
-                <mass value="6.78192"/>
-                <origin xyz="-0.010204 -0.005935 0.071865"/>
-                <inertia ixx="4.319e-1" ixy="-3.679e-4" ixz="9.099e-3" iyy="2.759e-1" iyz="-2.652e-3" izz="3.458e-1"/>
-            </inertial>
-            <visual>
-                <origin xyz="0 0 0" rpy="0 0 0"/>
-                <geometry>
-                    <mesh filename="package://rm_description/meshes/engineer/base_link.stl" scale="0.001 0.001 0.001"/>
-                </geometry>
-            </visual>
-            <collision>
-                <origin xyz="0. 0. 0.04" rpy="0 0 0"/>
-                <geometry>
-                    <box size="0.43 0.602 0.08"/>
-                </geometry>
-            </collision>
-            <collision>
-                <origin xyz="0.125 0.26625 0.3" rpy="0 0 0"/>
-                <geometry>
-                    <box size="0.04 0.0395 0.44"/>
-                </geometry>
-            </collision>
-            <collision>
-                <origin xyz="0.125 -0.26625 0.3" rpy="0 0 0"/>
-                <geometry>
-                    <box size="0.04 0.0395 0.44"/>
-                </geometry>
-            </collision>
-            <collision>
-                <origin xyz="-0.0965 0.27375 0.3" rpy="0 0 0"/>
-                <geometry>
-                    <box size="0.097 0.0545 0.44"/>
-                </geometry>
-            </collision>
-            <collision>
-                <origin xyz="-0.0965 -0.27375 0.3" rpy="0 0 0"/>
-                <geometry>
-                    <box size="0.097 0.0545 0.44"/>
-                </geometry>
-            </collision>
-            <collision>
-                <origin xyz="-0.013 0.274 0.1055" rpy="0 0 0"/>
-                <geometry>
-                    <box size="0.07 0.054 0.051"/>
-                </geometry>
-            </collision>
-            <collision>
-                <origin xyz="-0.013 -0.274 0.1055" rpy="0 0 0"/>
-                <geometry>
-                    <box size="0.07 0.054 0.051"/>
-                </geometry>
-            </collision>
-            <collision>
-                <origin xyz="0.0285 0.2685 0.5" rpy="0 0 0"/>
-                <geometry>
-                    <box size="0.153 0.035 0.040"/>
-                </geometry>
-            </collision>
-            <collision>
-                <origin xyz="0.0285 -0.2685 0.5" rpy="0 0 0"/>
-                <geometry>
-                    <box size="0.153 0.035 0.040"/>
-                </geometry>
-            </collision>
-        </link>
-        <joint name="fixed" type="fixed">
-            <parent link="base_link"/>
-            <child link="base_chassis"/>
-            <origin xyz="0. 0. 0.04" rpy="0 0 0"/>
-        </joint>
-        <link name="base_chassis">
             <inertial>
                 <mass value="4.947"/>
@@ -86,6 +15,5 @@
                 <origin xyz="0 0 0" rpy="0 0 0"/>
                 <geometry>
-                    <mesh filename="package://rm_description/meshes/engineer/base_chassis.stl"
-                          scale="0.001 0.001 0.001"/>
+                    <mesh filename="package://rm_description/meshes/engineer/base.stl" scale="0.001 0.001 0.001"/>
                 </geometry>
             </visual>
@@ -97,11 +25,4 @@
             </collision>
         </link>
-        <joint name="jointx" type="prismatic">
-            <parent link="base_chassis"/>
-            <child link="card"/>
-            <origin xyz="-0.2825 -0.001 0.005" rpy="0 0 0"/>
-            <axis xyz="1 0 0"/>
-            <limit lower="-0.1" upper="0.1" velocity="1" effort="200"/>
-        </joint>
         <link name="card">
             <inertial>
@@ -119,18 +40,7 @@
             </visual>
             <collision>
-                <origin xyz="0.0285 -0.2685 0.5" rpy="0 0 0"/>
-                <geometry>
-                    <box size="0.153 0.035 0.040"/>
-                </geometry>
             </collision>
         </link>
-        <joint name="jointx1" type="revolute">
-            <parent link="base_chassis"/>
-            <child link="hold"/>
-            <origin xyz="-0.245 -0.000076 0.06" rpy="0 0 0"/>
-            <axis xyz="0 1 0"/>
-            <limit lower="-6.28" upper="6.28" velocity="1" effort="200"/>
-        </joint>
-        <link name="hold">
+        <link name="drag">
             <inertial>
                 <mass value="0.404078"/>
@@ -140,29 +50,63 @@
             </inertial>
             <visual>
-                <origin xyz="-0.245 -0.000076 0.06" rpy="0 0 0"/>
+                <origin xyz="0 0 0" rpy="0 0 0"/>
                 <geometry>
-                    <mesh filename="package://rm_description/meshes/engineer/hold.stl"
+                    <mesh filename="package://rm_description/meshes/engineer/drag.stl"
                           scale="0.001 0.001 0.001"/>
                 </geometry>
             </visual>
             <collision>
-                <origin xyz="0.0285 -0.2685 0.5" rpy="0 0 0"/>
-                <geometry>
-                    <box size="0.153 0.035 0.040"/>
-                </geometry>
             </collision>
         </link>
-        <xacro:swerve_drive prefix="left_front" connected_to="base_chassis"
+        <joint name="drag_joint" type="revolute">
+            <parent link="base_link"/>
+            <child link="drag"/>
+            <origin xyz="-0.245 -0.000076 0.06" rpy="0 0 0"/>
+            <axis xyz="0 1 0"/>
+            <limit lower="-6.28" upper="6.28" velocity="1" effort="200"/>
+        </joint>
+        <joint name="card_joint" type="prismatic">
+            <parent link="base_link"/>
+            <child link="card"/>
+            <origin xyz="-0.001 -0.2475 0.005" rpy="0 0 0"/>
+            <axis xyz="0 1 0"/>
+            <limit lower="-0.1" upper="0.1" velocity="1" effort="200"/>
+        </joint>
+        <transmission name="trans_card_joint">
+            <type>transmission_interface/SimpleTransmission</type>
+            <actuator name="card_joint_motor">
+                <mechanicalReduction>1</mechanicalReduction>
+            </actuator>
+            <joint name="card_joint">
+                <offset>0</offset>
+                <hardwareInterface>hardware_interface/EffortJointInterface</hardwareInterface>
+            </joint>
+        </transmission>
+        <transmission name="trans_drag_joint">
+            <type>transmission_interface/SimpleTransmission</type>
+            <actuator name="drag_joint_motor">
+                <mechanicalReduction>1</mechanicalReduction>
+            </actuator>
+            <joint name="drag_joint">
+                <offset>0</offset>
+                <hardwareInterface>hardware_interface/EffortJointInterface</hardwareInterface>
+            </joint>
+        </transmission>
+        <xacro:swerve_drive prefix="left_front" connected_to="base_link"
                             wheel_x_offset="${wheel_track/2}" wheel_y_offset="${wheel_base/2}"
                             wheel_z_offset="${wheel_offset_z}"/>
-        <xacro:swerve_drive prefix="right_front" connected_to="base_chassis"
+        <xacro:swerve_drive prefix="right_front" connected_to="base_link"
                             wheel_x_offset="${wheel_track/2}" wheel_y_offset="${-wheel_base/2}"
                             wheel_z_offset="${wheel_offset_z}"/>
-        <xacro:swerve_drive prefix="left_back" connected_to="base_chassis"
+        <xacro:swerve_drive prefix="left_back" connected_to="base_link"
                             wheel_x_offset="${-wheel_track/2}" wheel_y_offset="${wheel_base/2}"
                             wheel_z_offset="${wheel_offset_z}"/>
-        <xacro:swerve_drive prefix="right_back" connected_to="base_chassis"
+        <xacro:swerve_drive prefix="right_back" connected_to="base_link"
                             wheel_x_offset="${-wheel_track/2}" wheel_y_offset="${-wheel_base/2}"
                             wheel_z_offset="${wheel_offset_z}"/>
+        <xacro:swerve_transmission prefix="left_front" wheel_reduction="13.733" pivot_offset="0"/>
+        <xacro:swerve_transmission prefix="right_front" wheel_reduction="-13.733" pivot_offset="1.861"/>
+        <xacro:swerve_transmission prefix="left_back" wheel_reduction="13.733" pivot_offset="1.585"/>
+        <xacro:swerve_transmission prefix="right_back" wheel_reduction="-13.733" pivot_offset="6.283"/>
     </xacro:macro>
 </robot>

File: urdf/engineer/engineer.urdf.xacro (robot description, xacro)
@@ -4,12 +4,11 @@
     <xacro:arg name="load_arm" default="true"/>
     <xacro:arg name="use_simulation" default="true"/>
-    <xacro:arg name="roller_type" default="simple"/>
     <xacro:if value="$(arg load_chassis)">
         <xacro:include filename="$(find rm_description)/urdf/engineer/chassis.urdf.xacro"/>
-        <xacro:chassis roller_type="$(arg roller_type)"/>
+        <xacro:chassis/>
     </xacro:if>
     <xacro:if value="$(arg load_arm)">
         <xacro:include filename="$(find rm_description)/urdf/engineer/arm.urdf.xacro"/>
-        <xacro:arm connected_to="base_link"/>
+        <xacro:arm connected_to="base_link" simulation="$(arg use_simulation)"/>
         <xacro:include filename="$(find rm_description)/urdf/engineer/arm.transmission.xacro"/>
         <xacro:arm_transmission simulation="$(arg use_simulation)"/>
