Commit message: Modified mechanical reduction and add softy controller

File: urdf/engineer/arm.transmission.xacro (robot description, xacro)
@@ -6,9 +6,9 @@
             <type>transmission_interface/SimpleTransmission</type>
             <actuator name="joint1_motor">
-                <mechanicalReduction>406.489213</mechanicalReduction>
+                <mechanicalReduction>738.231957</mechanicalReduction>
             </actuator>
             <joint name="joint1">
                 <hardwareInterface>hardware_interface/EffortJointInterface</hardwareInterface>
-                <offset>0</offset>
+                <offset>-0.003164659</offset>
             </joint>
         </transmission>
@@ -16,9 +16,9 @@
             <type>transmission_interface/SimpleTransmission</type>
             <actuator name="joint2_motor">
-                <mechanicalReduction>476.977368</mechanicalReduction>
+                <mechanicalReduction>434.2541</mechanicalReduction>
             </actuator>
             <joint name="joint2">
                 <hardwareInterface>hardware_interface/EffortJointInterface</hardwareInterface>
-                <offset>0</offset>
+                <offset>0.380457155</offset>
             </joint>
         </transmission>
@@ -26,9 +26,9 @@
             <type>transmission_interface/SimpleTransmission</type>
             <actuator name="joint3_motor">
-                <mechanicalReduction>1036.0854</mechanicalReduction>
+                <mechanicalReduction>-868.508184</mechanicalReduction>
             </actuator>
             <joint name="joint3">
                 <hardwareInterface>hardware_interface/EffortJointInterface</hardwareInterface>
-                <offset>0</offset>
+                <offset>0.2554111</offset>
             </joint>
         </transmission>
@@ -36,9 +36,9 @@
             <type>transmission_interface/SimpleTransmission</type>
             <actuator name="joint4_motor">
-                <mechanicalReduction>328.29</mechanicalReduction>
+                <mechanicalReduction>319.8835</mechanicalReduction>
             </actuator>
             <joint name="joint4">
                 <hardwareInterface>hardware_interface/EffortJointInterface</hardwareInterface>
-                <offset>0.3415371896670</offset>
+                <offset>-0.298261683</offset>
             </joint>
         </transmission>
@@ -50,5 +50,5 @@
             <joint name="joint5">
                 <hardwareInterface>hardware_interface/EffortJointInterface</hardwareInterface>
-                <offset>0</offset>
+                <offset>0.0460992</offset>
             </joint>
         </transmission>
@@ -60,5 +60,5 @@
             <joint name="joint6">
                 <hardwareInterface>hardware_interface/EffortJointInterface</hardwareInterface>
-                <offset>0</offset>
+                <offset>0.82689375</offset>
             </joint>
         </transmission>
@@ -70,5 +70,5 @@
             <joint name="joint7">
                 <hardwareInterface>hardware_interface/EffortJointInterface</hardwareInterface>
-                <offset>0</offset>
+                <offset>0.92119356</offset>
             </joint>
         </transmission>
@@ -77,9 +77,9 @@
                 <type>transmission_interface/SimpleTransmission</type>
                 <actuator name="mimic_joint1_motor">
-                    <mechanicalReduction>-406.489213</mechanicalReduction>
+                    <mechanicalReduction>-738.231957</mechanicalReduction>
                 </actuator>
                 <joint name="mimic_joint1">
                     <hardwareInterface>hardware_interface/EffortJointInterface</hardwareInterface>
-                    <offset>0</offset>
+                    <offset>-0.000870644</offset>
                 </joint>
             </transmission>
@@ -87,9 +87,9 @@
                 <type>transmission_interface/SimpleTransmission</type>
                 <actuator name="mimic_joint2_motor">
-                    <mechanicalReduction>-476.977368</mechanicalReduction>
+                    <mechanicalReduction>-434.2541</mechanicalReduction>
                 </actuator>
                 <joint name="mimic_joint2">
                     <hardwareInterface>hardware_interface/EffortJointInterface</hardwareInterface>
-                    <offset>0</offset>
+                    <offset>0.383102959</offset>
                 </joint>
             </transmission>
@@ -97,9 +97,9 @@
                 <type>transmission_interface/SimpleTransmission</type>
                 <actuator name="mimic_joint3_motor">
-                    <mechanicalReduction>-1036.0854</mechanicalReduction>
+                    <mechanicalReduction>868.508184</mechanicalReduction>
                 </actuator>
                 <joint name="mimic_joint3">
                     <hardwareInterface>hardware_interface/EffortJointInterface</hardwareInterface>
-                    <offset>0</offset>
+                    <offset>0.241729</offset>
                 </joint>
             </transmission>

File: urdf/engineer/arm.urdf.xacro (robot description, xacro)
@@ -2,19 +2,26 @@
 <robot xmlns:xacro="http://www.ros.org/wiki/xacro" name="arm">
     <xacro:macro name="arm" params="connected_to simulation">
-        <xacro:property name="threshold" value="0.1"/>
-        <xacro:property name="joint1_lower_limit" value="0.0005736069829"/>
-        <xacro:property name="joint1_upper_limit" value="0.6351414275302"/>
-        <xacro:property name="joint2_upper_limit" value="0.3438321773"/>
-        <xacro:property name="joint2_lower_limit" value="-0.2253643418193"/>
-        <xacro:property name="joint3_upper_limit" value="0.2362959079343"/>
-        <xacro:property name="joint3_lower_limit" value="-0.2253360962"/>
-        <xacro:property name="joint4_upper_limit" value="0.34152550806"/>
-        <xacro:property name="joint4_lower_limit" value="-0.296310718475"/>
-        <xacro:property name="joint5_upper_limit" value="-0.00022605078282"/>
-        <xacro:property name="joint5_lower_limit" value="-3.23240560816"/>
-        <xacro:property name="joint6_upper_limit" value="0.798170237718"/>
-        <xacro:property name="joint6_lower_limit" value="-4.2362368464"/>
-        <xacro:property name="joint7_upper_limit" value="3.979137624343"/>
-        <xacro:property name="joint7_lower_limit" value="-1.26312636630"/>
+        <xacro:property name="revolute_threshold" value="0.2"/>
+        <xacro:property name="threshold" value="0.01"/>
+        <xacro:property name="joint1_upper_limit" value="0.2759"/>
+        <xacro:property name="joint1_lower_limit" value="-0.0014"/>
+        <xacro:property name="joint2_upper_limit" value="0.38"/>
+        <xacro:property name="joint2_lower_limit" value="-0.35"/>
+        <xacro:property name="joint3_upper_limit" value="0.26"/>
+        <xacro:property name="joint3_lower_limit" value="-0.23"/>
+        <xacro:property name="joint4_upper_limit" value="0.2929"/>
+        <xacro:property name="joint4_lower_limit" value="-0.30"/>
+        <xacro:property name="joint5_upper_limit" value="0.06"/>
+        <xacro:property name="joint5_lower_limit" value="-3.22"/>
+        <xacro:property name="joint6_upper_limit" value="0.84"/>
+        <xacro:property name="joint6_lower_limit" value="-0.6"/>
+        <xacro:property name="joint7_upper_limit" value="0.95"/>
+        <xacro:property name="joint7_lower_limit" value="-4.38"/>
+        <xacro:property name="mimic_joint1_upper_limit" value="0.275"/>
+        <xacro:property name="mimic_joint1_lower_limit" value="0"/>
+        <xacro:property name="mimic_joint2_upper_limit" value="0.38"/>
+        <xacro:property name="mimic_joint2_lower_limit" value="-0.348"/>
+        <xacro:property name="mimic_joint3_upper_limit" value="0.24"/>
+        <xacro:property name="mimic_joint3_lower_limit" value="-0.24"/>
         <!--  link  -->
         <link name="link1">
@@ -251,5 +258,8 @@
             <origin xyz="0 0 0.1375" rpy="0 0 0"/>
             <axis xyz="0 0 1"/>
-            <limit lower="${joint1_lower_limit}" upper="${joint1_upper_limit}" velocity="1" effort="200"/>
+            <limit lower="${joint1_lower_limit}" upper="${joint1_upper_limit}" velocity="10" effort="200"/>
+            <safety_controller k_position="8000" k_velocity="15"
+                               soft_lower_limit="${joint1_lower_limit+0.003}"
+                               soft_upper_limit="${joint1_upper_limit-0.003}"/>
         </joint>
         <joint name="joint2" type="prismatic">
@@ -258,5 +268,8 @@
             <origin xyz="0. 0. 0.098707" rpy="0 0 0"/>
             <axis xyz="1 0 0"/>
-            <limit lower="${joint2_lower_limit}" upper="${joint2_upper_limit}" velocity="1" effort="200"/>
+            <limit lower="${joint2_lower_limit}" upper="${joint2_upper_limit}" velocity="10" effort="200"/>
+            <safety_controller k_position="8000" k_velocity="15"
+                               soft_lower_limit="${joint2_lower_limit+0.002}"
+                               soft_upper_limit="${joint2_upper_limit-0.002}"/>
         </joint>
         <joint name="joint3" type="prismatic">
@@ -265,5 +278,8 @@
             <origin xyz="0.022 0. 0.034" rpy="0 0 0"/>
             <axis xyz="1 0 0"/>
-            <limit lower="${joint3_lower_limit}" upper="${joint3_upper_limit}" velocity="1" effort="200"/>
+            <limit lower="${joint3_lower_limit}" upper="${joint3_upper_limit}" velocity="10" effort="200"/>
+            <safety_controller k_position="4000" k_velocity="10"
+                               soft_lower_limit="${joint3_lower_limit+0.01}"
+                               soft_upper_limit="${joint3_upper_limit-0.01}"/>
         </joint>
         <joint name="joint4" type="prismatic">
@@ -272,5 +288,8 @@
             <origin xyz="0. 0. 0.068" rpy="0 0 0"/>
             <axis xyz="0 1 0"/>
-            <limit lower="${joint4_lower_limit}" upper="${joint4_upper_limit}" velocity="1" effort="200"/>
+            <limit lower="${joint4_lower_limit}" upper="${joint4_upper_limit}" velocity="10" effort="200"/>
+            <safety_controller k_position="4000" k_velocity="10"
+                               soft_lower_limit="${joint4_lower_limit+0.005}"
+                               soft_upper_limit="${joint4_upper_limit-0.01}"/>
         </joint>
         <joint name="joint5" type="revolute">
@@ -279,5 +298,8 @@
             <origin xyz="0. 0. 0.069" rpy="0 0 0"/>
             <axis xyz="0 1 0"/>
-            <limit lower="${joint5_lower_limit}" upper="${joint5_upper_limit}" velocity="10" effort="200"/>
+            <limit lower="${joint5_lower_limit}" upper="${joint5_upper_limit}" velocity="30" effort="200"/>
+            <safety_controller k_position="20" k_velocity="2.5"
+                               soft_lower_limit="${joint5_lower_limit+revolute_threshold}"
+                               soft_upper_limit="${joint5_upper_limit-revolute_threshold}"/>
         </joint>
         <joint name="joint6" type="revolute">
@@ -286,5 +308,8 @@
             <origin xyz="0.06925 0. 0" rpy="0 0 0"/>
             <axis xyz="1 0 0"/>
-            <limit lower="${joint6_lower_limit}" upper="${joint6_upper_limit}" velocity="10" effort="200"/>
+            <limit lower="${joint6_lower_limit}" upper="${joint6_upper_limit}" velocity="30" effort="200"/>
+            <safety_controller k_position="20" k_velocity="2.5"
+                               soft_lower_limit="${joint6_lower_limit+revolute_threshold}"
+                               soft_upper_limit="${joint6_upper_limit-revolute_threshold}"/>
         </joint>
         <joint name="joint7" type="revolute">
@@ -293,5 +318,8 @@
             <origin xyz="-0.06925 0 0.255" rpy="0 0 0"/>
             <axis xyz="0 0 1"/>
-            <limit lower="${joint7_lower_limit}" upper="${joint7_upper_limit}" velocity="10" effort="200"/>
+            <limit lower="${joint7_lower_limit}" upper="${joint7_upper_limit}" velocity="30" effort="200"/>
+            <safety_controller k_position="20" k_velocity="2.5"
+                               soft_lower_limit="${joint7_lower_limit+revolute_threshold}"
+                               soft_upper_limit="${joint7_upper_limit-revolute_threshold}"/>
         </joint>
         <xacro:unless value="${simulation}">
@@ -356,21 +384,31 @@
                 <parent link="${connected_to}"/>
                 <child link="mimic_link1"/>
-                <origin xyz="0 0 0.1375" rpy="0 0 0"/>
+                <origin xyz="0 0 0.21375" rpy="0 0 0"/>
                 <axis xyz="0 0 1"/>
-                <limit lower="${joint1_lower_limit}" upper="${joint1_upper_limit}" velocity="1" effort="200"/>
+                <limit lower="${joint1_lower_limit}" upper="${joint1_upper_limit}" velocity="10" effort="200"/>
+                <safety_controller k_position="8000" k_velocity="15"
+                                   soft_lower_limit="${mimic_joint1_lower_limit+0.001}"
+                                   soft_upper_limit="${mimic_joint1_upper_limit-0.001}"/>
             </joint>
             <joint name="mimic_joint2" type="prismatic">
                 <parent link="link1"/>
-                <child link="mimiclink2_1"/>
-                <origin xyz="0. 0. 0.098707" rpy="0 0 0"/>
+                <child link="mimic_link2_1"/>
+                <origin xyz="0. 0. 15.098707" rpy="0 0 0"/>
                 <axis xyz="1 0 0"/>
-                <limit lower="${joint2_lower_limit}" upper="${joint2_upper_limit}" velocity="1" effort="200"/>
+                <limit lower="${joint2_lower_limit}" upper="${joint2_upper_limit}" velocity="10" effort="200"/>
+                <safety_controller k_position="8000" k_velocity="15"
+                                   soft_lower_limit="${mimic_joint2_lower_limit+0.005}"
+                                   soft_upper_limit="${mimic_joint2_upper_limit-0.002}"/>
             </joint>
             <joint name="mimic_joint3" type="prismatic">
                 <parent link="link2_1"/>
                 <child link="mimic_link2_2"/>
-                <origin xyz="0.022 0. 0.034" rpy="0 0 0"/>
+                <origin xyz="0.022 0. 10.034" rpy="0 0 0"/>
                 <axis xyz="1 0 0"/>
-                <limit lower="${joint3_lower_limit}" upper="${joint3_upper_limit}" velocity="1" effort="200"/>
+                <limit lower="${mimic_joint3_lower_limit}" upper="${mimic_joint3_upper_limit}" velocity="10"
+                       effort="200"/>
+                <safety_controller k_position="8000" k_velocity="15"
+                                   soft_lower_limit="${mimic_joint3_lower_limit+0.005}"
+                                   soft_upper_limit="${mimic_joint3_upper_limit-0.005}"/>
             </joint>
         </xacro:unless>

Commit message: Update joint's limit

File: urdf/engineer/arm.transmission.xacro (robot description, xacro)
@@ -70,5 +70,5 @@
             <joint name="joint7">
                 <hardwareInterface>hardware_interface/EffortJointInterface</hardwareInterface>
-                <offset>0.92119356</offset>
+                <offset>0.8493</offset>
             </joint>
         </transmission>

File: urdf/engineer/arm.urdf.xacro (robot description, xacro)
@@ -6,13 +6,13 @@
         <xacro:property name="joint1_upper_limit" value="0.2759"/>
         <xacro:property name="joint1_lower_limit" value="-0.0014"/>
-        <xacro:property name="joint2_upper_limit" value="0.38"/>
+        <xacro:property name="joint2_upper_limit" value="0.392"/>
         <xacro:property name="joint2_lower_limit" value="-0.35"/>
-        <xacro:property name="joint3_upper_limit" value="0.26"/>
+        <xacro:property name="joint3_upper_limit" value="0.265"/>
         <xacro:property name="joint3_lower_limit" value="-0.23"/>
         <xacro:property name="joint4_upper_limit" value="0.2929"/>
         <xacro:property name="joint4_lower_limit" value="-0.30"/>
-        <xacro:property name="joint5_upper_limit" value="0.06"/>
+        <xacro:property name="joint5_upper_limit" value="0.29"/>
         <xacro:property name="joint5_lower_limit" value="-3.22"/>
-        <xacro:property name="joint6_upper_limit" value="0.84"/>
+        <xacro:property name="joint6_upper_limit" value="1.32"/>
         <xacro:property name="joint6_lower_limit" value="-0.6"/>
         <xacro:property name="joint7_upper_limit" value="0.95"/>
@@ -20,7 +20,7 @@
         <xacro:property name="mimic_joint1_upper_limit" value="0.275"/>
         <xacro:property name="mimic_joint1_lower_limit" value="0"/>
-        <xacro:property name="mimic_joint2_upper_limit" value="0.38"/>
+        <xacro:property name="mimic_joint2_upper_limit" value="0.381"/>
         <xacro:property name="mimic_joint2_lower_limit" value="-0.348"/>
-        <xacro:property name="mimic_joint3_upper_limit" value="0.24"/>
+        <xacro:property name="mimic_joint3_upper_limit" value="0.241"/>
         <xacro:property name="mimic_joint3_lower_limit" value="-0.24"/>
         <!--  link  -->
@@ -259,7 +259,7 @@
             <axis xyz="0 0 1"/>
             <limit lower="${joint1_lower_limit}" upper="${joint1_upper_limit}" velocity="10" effort="200"/>
-            <safety_controller k_position="8000" k_velocity="15"
-                               soft_lower_limit="${joint1_lower_limit+0.003}"
-                               soft_upper_limit="${joint1_upper_limit-0.003}"/>
+            <!--            <safety_controller k_position="8000" k_velocity="15"-->
+            <!--                               soft_lower_limit="${joint1_lower_limit+0.003}"-->
+            <!--                               soft_upper_limit="${joint1_upper_limit-0.003}"/>-->
         </joint>
         <joint name="joint2" type="prismatic">
@@ -269,7 +269,7 @@
             <axis xyz="1 0 0"/>
             <limit lower="${joint2_lower_limit}" upper="${joint2_upper_limit}" velocity="10" effort="200"/>
-            <safety_controller k_position="8000" k_velocity="15"
-                               soft_lower_limit="${joint2_lower_limit+0.002}"
-                               soft_upper_limit="${joint2_upper_limit-0.002}"/>
+            <!--            <safety_controller k_position="8000" k_velocity="15"-->
+            <!--                               soft_lower_limit="${joint2_lower_limit+0.002}"-->
+            <!--                               soft_upper_limit="${joint2_upper_limit-0.002}"/>-->
         </joint>
         <joint name="joint3" type="prismatic">
@@ -279,7 +279,7 @@
             <axis xyz="1 0 0"/>
             <limit lower="${joint3_lower_limit}" upper="${joint3_upper_limit}" velocity="10" effort="200"/>
-            <safety_controller k_position="4000" k_velocity="10"
-                               soft_lower_limit="${joint3_lower_limit+0.01}"
-                               soft_upper_limit="${joint3_upper_limit-0.01}"/>
+            <!--            <safety_controller k_position="4000" k_velocity="10"-->
+            <!--                               soft_lower_limit="${joint3_lower_limit+0.01}"-->
+            <!--                               soft_upper_limit="${joint3_upper_limit-0.01}"/>-->
         </joint>
         <joint name="joint4" type="prismatic">
@@ -289,7 +289,7 @@
             <axis xyz="0 1 0"/>
             <limit lower="${joint4_lower_limit}" upper="${joint4_upper_limit}" velocity="10" effort="200"/>
-            <safety_controller k_position="4000" k_velocity="10"
-                               soft_lower_limit="${joint4_lower_limit+0.005}"
-                               soft_upper_limit="${joint4_upper_limit-0.01}"/>
+            <!--            <safety_controller k_position="4000" k_velocity="10"-->
+            <!--                               soft_lower_limit="${joint4_lower_limit+0.005}"-->
+            <!--                               soft_upper_limit="${joint4_upper_limit-0.01}"/>-->
         </joint>
         <joint name="joint5" type="revolute">
@@ -299,7 +299,7 @@
             <axis xyz="0 1 0"/>
             <limit lower="${joint5_lower_limit}" upper="${joint5_upper_limit}" velocity="30" effort="200"/>
-            <safety_controller k_position="20" k_velocity="2.5"
-                               soft_lower_limit="${joint5_lower_limit+revolute_threshold}"
-                               soft_upper_limit="${joint5_upper_limit-revolute_threshold}"/>
+            <!--            <safety_controller k_position="20" k_velocity="2.5"-->
+            <!--                               soft_lower_limit="${joint5_lower_limit+revolute_threshold}"-->
+            <!--                               soft_upper_limit="${joint5_upper_limit-revolute_threshold}"/>-->
         </joint>
         <joint name="joint6" type="revolute">
@@ -309,7 +309,7 @@
             <axis xyz="1 0 0"/>
             <limit lower="${joint6_lower_limit}" upper="${joint6_upper_limit}" velocity="30" effort="200"/>
-            <safety_controller k_position="20" k_velocity="2.5"
-                               soft_lower_limit="${joint6_lower_limit+revolute_threshold}"
-                               soft_upper_limit="${joint6_upper_limit-revolute_threshold}"/>
+            <!--            <safety_controller k_position="20" k_velocity="2.5"-->
+            <!--                               soft_lower_limit="${joint6_lower_limit+revolute_threshold}"-->
+            <!--                               soft_upper_limit="${joint6_upper_limit-revolute_threshold}"/>-->
         </joint>
         <joint name="joint7" type="revolute">
@@ -319,7 +319,4 @@
             <axis xyz="0 0 1"/>
             <limit lower="${joint7_lower_limit}" upper="${joint7_upper_limit}" velocity="30" effort="200"/>
-            <safety_controller k_position="20" k_velocity="2.5"
-                               soft_lower_limit="${joint7_lower_limit+revolute_threshold}"
-                               soft_upper_limit="${joint7_upper_limit-revolute_threshold}"/>
         </joint>
         <xacro:unless value="${simulation}">
@@ -387,7 +384,4 @@
                 <axis xyz="0 0 1"/>
                 <limit lower="${joint1_lower_limit}" upper="${joint1_upper_limit}" velocity="10" effort="200"/>
-                <safety_controller k_position="8000" k_velocity="15"
-                                   soft_lower_limit="${mimic_joint1_lower_limit+0.001}"
-                                   soft_upper_limit="${mimic_joint1_upper_limit-0.001}"/>
             </joint>
             <joint name="mimic_joint2" type="prismatic">
