Commit message: Update engineer's model

File: urdf/engineer/arm.transmission.xacro (robot description, xacro)
@@ -6,9 +6,9 @@
             <type>transmission_interface/SimpleTransmission</type>
             <actuator name="joint1_motor">
-                <mechanicalReduction>738.231957</mechanicalReduction>
+                <mechanicalReduction>883.300222</mechanicalReduction>
             </actuator>
             <joint name="joint1">
                 <hardwareInterface>hardware_interface/EffortJointInterface</hardwareInterface>
-                <offset>-0.003164659</offset>
+                <offset>0.015</offset>
             </joint>
         </transmission>
@@ -16,9 +16,9 @@
             <type>transmission_interface/SimpleTransmission</type>
             <actuator name="joint2_motor">
-                <mechanicalReduction>434.2541</mechanicalReduction>
+                <mechanicalReduction>497.500437</mechanicalReduction>
             </actuator>
             <joint name="joint2">
                 <hardwareInterface>hardware_interface/EffortJointInterface</hardwareInterface>
-                <offset>0.380457155</offset>
+                <offset>-0.313196</offset>
             </joint>
         </transmission>
@@ -26,9 +26,9 @@
             <type>transmission_interface/SimpleTransmission</type>
             <actuator name="joint3_motor">
-                <mechanicalReduction>-868.508184</mechanicalReduction>
+                <mechanicalReduction>-995.000875</mechanicalReduction>
             </actuator>
             <joint name="joint3">
                 <hardwareInterface>hardware_interface/EffortJointInterface</hardwareInterface>
-                <offset>0.2554111</offset>
+                <offset>-0.188893</offset>
             </joint>
         </transmission>
@@ -36,9 +36,9 @@
             <type>transmission_interface/SimpleTransmission</type>
             <actuator name="joint4_motor">
-                <mechanicalReduction>319.8835</mechanicalReduction>
+                <mechanicalReduction>328.093719</mechanicalReduction>
             </actuator>
             <joint name="joint4">
                 <hardwareInterface>hardware_interface/EffortJointInterface</hardwareInterface>
-                <offset>-0.298261683</offset>
+                <offset>-0.29131929</offset>
             </joint>
         </transmission>
@@ -50,5 +50,5 @@
             <joint name="joint5">
                 <hardwareInterface>hardware_interface/EffortJointInterface</hardwareInterface>
-                <offset>0.0460992</offset>
+                <offset>0.010503</offset>
             </joint>
         </transmission>
@@ -60,5 +60,5 @@
             <joint name="joint6">
                 <hardwareInterface>hardware_interface/EffortJointInterface</hardwareInterface>
-                <offset>0.82689375</offset>
+                <offset>0.85218130</offset>
             </joint>
         </transmission>
@@ -70,5 +70,5 @@
             <joint name="joint7">
                 <hardwareInterface>hardware_interface/EffortJointInterface</hardwareInterface>
-                <offset>0.8493</offset>
+                <offset>0.87897618</offset>
             </joint>
         </transmission>
@@ -77,9 +77,9 @@
                 <type>transmission_interface/SimpleTransmission</type>
                 <actuator name="mimic_joint1_motor">
-                    <mechanicalReduction>-738.231957</mechanicalReduction>
+                    <mechanicalReduction>-883.300222</mechanicalReduction>
                 </actuator>
                 <joint name="mimic_joint1">
                     <hardwareInterface>hardware_interface/EffortJointInterface</hardwareInterface>
-                    <offset>-0.000870644</offset>
+                    <offset>0.015</offset>
                 </joint>
             </transmission>
@@ -87,9 +87,9 @@
                 <type>transmission_interface/SimpleTransmission</type>
                 <actuator name="mimic_joint2_motor">
-                    <mechanicalReduction>-434.2541</mechanicalReduction>
+                    <mechanicalReduction>-497.500437</mechanicalReduction>
                 </actuator>
                 <joint name="mimic_joint2">
                     <hardwareInterface>hardware_interface/EffortJointInterface</hardwareInterface>
-                    <offset>0.383102959</offset>
+                    <offset>-0.3062994</offset>
                 </joint>
             </transmission>
@@ -97,9 +97,9 @@
                 <type>transmission_interface/SimpleTransmission</type>
                 <actuator name="mimic_joint3_motor">
-                    <mechanicalReduction>868.508184</mechanicalReduction>
+                    <mechanicalReduction>995.000875</mechanicalReduction>
                 </actuator>
                 <joint name="mimic_joint3">
                     <hardwareInterface>hardware_interface/EffortJointInterface</hardwareInterface>
-                    <offset>0.241729</offset>
+                    <offset>-0.1930778828</offset>
                 </joint>
             </transmission>

File: urdf/engineer/arm.urdf.xacro (robot description, xacro)
@@ -2,26 +2,25 @@
 <robot xmlns:xacro="http://www.ros.org/wiki/xacro" name="arm">
     <xacro:macro name="arm" params="connected_to simulation">
-        <xacro:property name="revolute_threshold" value="0.2"/>
-        <xacro:property name="threshold" value="0.01"/>
-        <xacro:property name="joint1_upper_limit" value="0.2759"/>
-        <xacro:property name="joint1_lower_limit" value="-0.0014"/>
-        <xacro:property name="joint2_upper_limit" value="0.392"/>
-        <xacro:property name="joint2_lower_limit" value="-0.35"/>
-        <xacro:property name="joint3_upper_limit" value="0.265"/>
-        <xacro:property name="joint3_lower_limit" value="-0.23"/>
-        <xacro:property name="joint4_upper_limit" value="0.2929"/>
+        <xacro:property name="threshold" value="0.15"/>
+        <xacro:property name="joint1_upper_limit" value="0.25"/>
+        <xacro:property name="joint1_lower_limit" value="0"/>
+        <xacro:property name="joint2_upper_limit" value="0.34"/>
+        <xacro:property name="joint2_lower_limit" value="-0.32"/>
+        <xacro:property name="joint3_upper_limit" value="0.26"/>
+        <xacro:property name="joint3_lower_limit" value="-0.20"/>
+        <xacro:property name="joint4_upper_limit" value="0.33"/>
         <xacro:property name="joint4_lower_limit" value="-0.30"/>
-        <xacro:property name="joint5_upper_limit" value="0.29"/>
-        <xacro:property name="joint5_lower_limit" value="-3.22"/>
-        <xacro:property name="joint6_upper_limit" value="1.32"/>
-        <xacro:property name="joint6_lower_limit" value="-0.6"/>
+        <xacro:property name="joint5_upper_limit" value="0.1"/>
+        <xacro:property name="joint5_lower_limit" value="-3.4"/>
+        <xacro:property name="joint6_upper_limit" value="0.9"/>
+        <xacro:property name="joint6_lower_limit" value="-0.9"/>
         <xacro:property name="joint7_upper_limit" value="0.95"/>
-        <xacro:property name="joint7_lower_limit" value="-4.38"/>
-        <xacro:property name="mimic_joint1_upper_limit" value="0.275"/>
+        <xacro:property name="joint7_lower_limit" value="-4.50"/>
+        <xacro:property name="mimic_joint1_upper_limit" value="0.25"/>
         <xacro:property name="mimic_joint1_lower_limit" value="0"/>
-        <xacro:property name="mimic_joint2_upper_limit" value="0.381"/>
-        <xacro:property name="mimic_joint2_lower_limit" value="-0.348"/>
-        <xacro:property name="mimic_joint3_upper_limit" value="0.241"/>
-        <xacro:property name="mimic_joint3_lower_limit" value="-0.24"/>
+        <xacro:property name="mimic_joint2_upper_limit" value="0.34"/>
+        <xacro:property name="mimic_joint2_lower_limit" value="-0.32"/>
+        <xacro:property name="mimic_joint3_upper_limit" value="0.21"/>
+        <xacro:property name="mimic_joint3_lower_limit" value="-0.2"/>
         <!--  link  -->
         <link name="link1">
@@ -258,8 +257,5 @@
             <origin xyz="0 0 0.1375" rpy="0 0 0"/>
             <axis xyz="0 0 1"/>
-            <limit lower="${joint1_lower_limit}" upper="${joint1_upper_limit}" velocity="10" effort="200"/>
-            <!--            <safety_controller k_position="8000" k_velocity="15"-->
-            <!--                               soft_lower_limit="${joint1_lower_limit+0.003}"-->
-            <!--                               soft_upper_limit="${joint1_upper_limit-0.003}"/>-->
+            <limit lower="${joint1_lower_limit}" upper="${joint1_upper_limit}" velocity="5" effort="200"/>
         </joint>
         <joint name="joint2" type="prismatic">
@@ -268,8 +264,5 @@
             <origin xyz="0. 0. 0.098707" rpy="0 0 0"/>
             <axis xyz="1 0 0"/>
-            <limit lower="${joint2_lower_limit}" upper="${joint2_upper_limit}" velocity="10" effort="200"/>
-            <!--            <safety_controller k_position="8000" k_velocity="15"-->
-            <!--                               soft_lower_limit="${joint2_lower_limit+0.002}"-->
-            <!--                               soft_upper_limit="${joint2_upper_limit-0.002}"/>-->
+            <limit lower="${joint2_lower_limit}" upper="${joint2_upper_limit}" velocity="5" effort="200"/>
         </joint>
         <joint name="joint3" type="prismatic">
@@ -278,8 +271,8 @@
             <origin xyz="0.022 0. 0.034" rpy="0 0 0"/>
             <axis xyz="1 0 0"/>
-            <limit lower="${joint3_lower_limit}" upper="${joint3_upper_limit}" velocity="10" effort="200"/>
-            <!--            <safety_controller k_position="4000" k_velocity="10"-->
-            <!--                               soft_lower_limit="${joint3_lower_limit+0.01}"-->
-            <!--                               soft_upper_limit="${joint3_upper_limit-0.01}"/>-->
+            <limit lower="${joint3_lower_limit}" upper="${joint3_upper_limit}" velocity="5" effort="200"/>
+            <safety_controller k_position="1800" k_velocity="18"
+                               soft_lower_limit="${joint3_lower_limit+0.018}"
+                               soft_upper_limit="${joint3_upper_limit-0.03}"/>
         </joint>
         <joint name="joint4" type="prismatic">
@@ -288,8 +281,8 @@
             <origin xyz="0. 0. 0.068" rpy="0 0 0"/>
             <axis xyz="0 1 0"/>
-            <limit lower="${joint4_lower_limit}" upper="${joint4_upper_limit}" velocity="10" effort="200"/>
-            <!--            <safety_controller k_position="4000" k_velocity="10"-->
-            <!--                               soft_lower_limit="${joint4_lower_limit+0.005}"-->
-            <!--                               soft_upper_limit="${joint4_upper_limit-0.01}"/>-->
+            <limit lower="${joint4_lower_limit}" upper="${joint4_upper_limit}" velocity="5" effort="200"/>
+            <safety_controller k_position="800" k_velocity="10"
+                               soft_lower_limit="${joint4_lower_limit+0.014}"
+                               soft_upper_limit="${joint4_upper_limit-0.046}"/>
         </joint>
         <joint name="joint5" type="revolute">
@@ -298,8 +291,8 @@
             <origin xyz="0. 0. 0.069" rpy="0 0 0"/>
             <axis xyz="0 1 0"/>
-            <limit lower="${joint5_lower_limit}" upper="${joint5_upper_limit}" velocity="30" effort="200"/>
-            <!--            <safety_controller k_position="20" k_velocity="2.5"-->
-            <!--                               soft_lower_limit="${joint5_lower_limit+revolute_threshold}"-->
-            <!--                               soft_upper_limit="${joint5_upper_limit-revolute_threshold}"/>-->
+            <limit lower="${joint5_lower_limit}" upper="${joint5_upper_limit}" velocity="5" effort="200"/>
+            <safety_controller k_position="100" k_velocity="3"
+                               soft_lower_limit="${joint5_lower_limit+threshold}"
+                               soft_upper_limit="${joint5_upper_limit-threshold}"/>
         </joint>
         <joint name="joint6" type="revolute">
@@ -308,8 +301,8 @@
             <origin xyz="0.06925 0. 0" rpy="0 0 0"/>
             <axis xyz="1 0 0"/>
-            <limit lower="${joint6_lower_limit}" upper="${joint6_upper_limit}" velocity="30" effort="200"/>
-            <!--            <safety_controller k_position="20" k_velocity="2.5"-->
-            <!--                               soft_lower_limit="${joint6_lower_limit+revolute_threshold}"-->
-            <!--                               soft_upper_limit="${joint6_upper_limit-revolute_threshold}"/>-->
+            <limit lower="${joint6_lower_limit}" upper="${joint6_upper_limit}" velocity="5" effort="200"/>
+            <safety_controller k_position="100" k_velocity="3"
+                               soft_lower_limit="${joint6_lower_limit+threshold}"
+                               soft_upper_limit="${joint6_upper_limit-threshold}"/>
         </joint>
         <joint name="joint7" type="revolute">
@@ -318,5 +311,8 @@
             <origin xyz="-0.06925 0 0.255" rpy="0 0 0"/>
             <axis xyz="0 0 1"/>
-            <limit lower="${joint7_lower_limit}" upper="${joint7_upper_limit}" velocity="30" effort="200"/>
+            <limit lower="${joint7_lower_limit}" upper="${joint7_upper_limit}" velocity="5" effort="200"/>
+            <safety_controller k_position="100" k_velocity="3"
+                               soft_lower_limit="${joint7_lower_limit+threshold}"
+                               soft_upper_limit="${joint7_upper_limit-threshold}"/>
         </joint>
         <xacro:unless value="${simulation}">
@@ -383,26 +379,20 @@
                 <origin xyz="0 0 0.21375" rpy="0 0 0"/>
                 <axis xyz="0 0 1"/>
-                <limit lower="${joint1_lower_limit}" upper="${joint1_upper_limit}" velocity="10" effort="200"/>
+                <limit lower="${joint1_lower_limit}" upper="${joint1_upper_limit}" velocity="5" effort="200"/>
             </joint>
             <joint name="mimic_joint2" type="prismatic">
                 <parent link="link1"/>
                 <child link="mimic_link2_1"/>
-                <origin xyz="0. 0. 15.098707" rpy="0 0 0"/>
+                <origin xyz="0. 0. 0.098707" rpy="0 0 0"/>
                 <axis xyz="1 0 0"/>
-                <limit lower="${joint2_lower_limit}" upper="${joint2_upper_limit}" velocity="10" effort="200"/>
-                <safety_controller k_position="8000" k_velocity="15"
-                                   soft_lower_limit="${mimic_joint2_lower_limit+0.005}"
-                                   soft_upper_limit="${mimic_joint2_upper_limit-0.002}"/>
+                <limit lower="${joint2_lower_limit}" upper="${joint2_upper_limit}" velocity="5" effort="200"/>
             </joint>
             <joint name="mimic_joint3" type="prismatic">
                 <parent link="link2_1"/>
                 <child link="mimic_link2_2"/>
-                <origin xyz="0.022 0. 10.034" rpy="0 0 0"/>
+                <origin xyz="0.022 0. 0.034" rpy="0 0 0"/>
                 <axis xyz="1 0 0"/>
-                <limit lower="${mimic_joint3_lower_limit}" upper="${mimic_joint3_upper_limit}" velocity="10"
+                <limit lower="${mimic_joint3_lower_limit}" upper="${mimic_joint3_upper_limit}" velocity="5"
                        effort="200"/>
-                <safety_controller k_position="8000" k_velocity="15"
-                                   soft_lower_limit="${mimic_joint3_lower_limit+0.005}"
-                                   soft_upper_limit="${mimic_joint3_upper_limit-0.005}"/>
             </joint>
         </xacro:unless>

File: urdf/engineer/chassis.urdf.xacro (robot description, xacro)
@@ -123,5 +123,5 @@
             </inertial>
             <visual>
-                <origin xyz="0 0 0" rpy="0 0 0"/>
+                <origin xyz="0 0 0" rpy="0 0 -1.57"/>
                 <geometry>
                     <mesh filename="package://rm_description/meshes/engineer/card.stl" scale="0.001 0.001 0.001"/>
@@ -130,5 +130,5 @@
             <collision>
                 <geometry>
-                    <mesh filename="package://rm_description/meshes/engineer/card_collision.stl"
+                    <mesh filename="package://rm_description/meshes/engineer/card_collision1.stl"
                           scale="0.001 0.001 0.001"/>
                 </geometry>
@@ -137,7 +137,8 @@
         <link name="drag">
             <inertial>
-                <mass value="0.252375"/>
-                <origin xyz="-0.230445 -0.072148 0.051026"/>
-                <inertia ixx="3.688e-3" ixy="-3.738e-3" ixz="2.667e-3" iyy="1.480e-2" iyz="1.299e-3" izz="1.663e-2"/>
+                <mass value="0.404605"/>
+                <origin xyz="0.053283 0.032371 0.017125"/>
+                <inertia ixx="5.893e-3" ixy="1.346e-4" ixz="-8.957569e-5" iyy="2.879e-3" iyz="-4.020e-4"
+                         izz="8.206e-3"/>
             </inertial>
             <visual>
@@ -149,7 +150,8 @@
             </visual>
             <collision>
-                <origin xyz="-0.041518 0.077 0.017" rpy="0 0 0"/>
-                <geometry>
-                    <box size="0.112768 0.009 0.018"/>
+                <origin xyz="0 0 0" rpy="0 0 0"/>
+                <geometry>
+                    <mesh filename="package://rm_description/meshes/engineer/drag_collision.stl"
+                          scale="0.001 0.001 0.001"/>
                 </geometry>
             </collision>
@@ -164,5 +166,5 @@
             <parent link="base_link"/>
             <child link="card"/>
-            <origin xyz="0. 0.175076 -0.008" rpy="0 0 0"/>
+            <origin xyz="0.244 -0.0585 0.036" rpy="0 0 -1.57"/>
             <axis xyz="1 0 0"/>
             <limit lower="-1000000" upper="1000000" velocity="1" effort="200"/>
@@ -171,12 +173,12 @@
             <parent link="base_link"/>
             <child link="drag"/>
-            <origin xyz="-0.245 -0.000076 0.06" rpy="0 0 0"/>
+            <origin xyz="-0.245 0 0.06" rpy="0 0 3.14"/>
             <axis xyz="0 1 0"/>
-            <limit lower="-6.28" upper="6.28" velocity="1" effort="200"/>
+            <limit lower="-1.6" upper="-0.01" velocity="1" effort="200"/>
         </joint>
         <transmission name="trans_card_joint">
             <type>transmission_interface/SimpleTransmission</type>
             <actuator name="card_joint_motor">
-                <mechanicalReduction>50.895</mechanicalReduction>
+                <mechanicalReduction>36</mechanicalReduction>
             </actuator>
             <joint name="card_joint">
@@ -188,8 +190,8 @@
             <type>transmission_interface/SimpleTransmission</type>
             <actuator name="drag_joint_motor">
-                <mechanicalReduction>1</mechanicalReduction>
+                <mechanicalReduction>2</mechanicalReduction>
             </actuator>
             <joint name="drag_joint">
-                <offset>0</offset>
+                <offset>-1.625664</offset>
                 <hardwareInterface>hardware_interface/EffortJointInterface</hardwareInterface>
             </joint>

File: urdf/engineer/gimbal.urdf.xacro (robot description, xacro)
@@ -5,8 +5,8 @@
         <link name="gimbal_base">
             <inertial>
-                <mass value="0.2"/>
-                <origin xyz="-0.034 0.002 0.036"/>
-                <inertia ixx="4.878e-4" ixy="1.941e-5" ixz="2.44e-4" iyy="8.322e-4"
-                         iyz="-1.812e-5" izz="4.513e-4"/>
+                <mass value="0.163485"/>
+                <origin xyz="0.000652 0.002177 0.009113"/>
+                <inertia ixx="7.4761869e-5" ixy="-1.177056e-6" ixz="-2.348598e-6" iyy="7.440176e-5"
+                         iyz="6.29861e-6" izz="6.3915e-5"/>
             </inertial>
             <visual>
@@ -17,18 +17,11 @@
                 </geometry>
             </visual>
-            <collision>
-                <origin xyz="0 0 0" rpy="0 0 0"/>
-                <geometry>
-                    <mesh filename="package://rm_description/meshes/engineer/gimbal_base.stl"
-                          scale="0.001 0.001 0.001"/>
-                </geometry>
-            </collision>
         </link>
         <link name="yaw">
             <inertial>
-                <mass value="0.2"/>
-                <origin xyz="-0.034 0.002 0.036"/>
-                <inertia ixx="4.878e-4" ixy="1.941e-5" ixz="2.44e-4" iyy="8.322e-4"
-                         iyz="-1.812e-5" izz="4.513e-4"/>
+                <mass value="0.074489"/>
+                <origin xyz="0.000003 -0.001925 0.013798"/>
+                <inertia ixx="1.672e-4" ixy="-0.42e-9" ixz="1.5288e-8" iyy="5.1826669e-5"
+                         iyz="-5.33194e-7" izz="1.439e-4"/>
             </inertial>
             <visual>
@@ -38,17 +31,11 @@
                 </geometry>
             </visual>
-            <collision>
-                <origin xyz="0 0 0" rpy="0 0 0"/>
-                <geometry>
-                    <mesh filename="package://rm_description/meshes/engineer/yaw.stl" scale="0.001 0.001 0.001"/>
-                </geometry>
-            </collision>
         </link>
         <link name="pitch">
             <inertial>
-                <mass value="0.644"/>
-                <origin xyz="0.029 0.000617 0.0376"/>
-                <inertia ixx="1.8216e-3" ixy="5.514e-6" ixz="1.58e-4" iyy="5.68e-3"
-                         iyz="-6.628e-6" izz="4.396e-3"/>
+                <mass value="0.28963"/>
+                <origin xyz="0.001291 0.005233 0.001395"/>
+                <inertia ixx="2.976e-4" ixy="5.294138e-6" ixz="-5.514329e-6" iyy="1.889e-4"
+                         iyz="3.085924e-6" izz="4.132e-4"/>
             </inertial>
             <visual>
@@ -58,10 +45,4 @@
                 </geometry>
             </visual>
-            <collision>
-                <origin xyz="0 0 0" rpy="0 0 0"/>
-                <geometry>
-                    <mesh filename="package://rm_description/meshes/engineer/pitch.stl" scale="0.001 0.001 0.001"/>
-                </geometry>
-            </collision>
         </link>
         <xacro:unless value="${connected_to == ''}">
@@ -96,5 +77,5 @@
             </actuator>
             <joint name="yaw_joint">
-                <offset>0</offset>
+                <offset>3.48597</offset>
                 <hardwareInterface>hardware_interface/EffortJointInterface</hardwareInterface>
             </joint>
@@ -103,8 +84,8 @@
             <type>transmission_interface/SimpleTransmission</type>
             <actuator name="pitch_joint_motor">
-                <mechanicalReduction>-1</mechanicalReduction>
+                <mechanicalReduction>1</mechanicalReduction>
             </actuator>
             <joint name="pitch_joint">
-                <offset>0</offset>
+                <offset>0.75088</offset>
                 <hardwareInterface>hardware_interface/EffortJointInterface</hardwareInterface>
             </joint>
