Commit message: Update engineer joint's limit and add softy controller

File: urdf/engineer/arm.transmission.xacro (robot description, xacro)
@@ -10,5 +10,5 @@
             <joint name="joint1">
                 <hardwareInterface>hardware_interface/EffortJointInterface</hardwareInterface>
-                <offset>0.015</offset>
+                <offset>-0.002099</offset>
             </joint>
         </transmission>
@@ -16,9 +16,9 @@
             <type>transmission_interface/SimpleTransmission</type>
             <actuator name="joint2_motor">
-                <mechanicalReduction>497.500437</mechanicalReduction>
+                <mechanicalReduction>-497.500437</mechanicalReduction>
             </actuator>
             <joint name="joint2">
                 <hardwareInterface>hardware_interface/EffortJointInterface</hardwareInterface>
-                <offset>-0.313196</offset>
+                <offset>0.294773</offset>
             </joint>
         </transmission>
@@ -26,9 +26,9 @@
             <type>transmission_interface/SimpleTransmission</type>
             <actuator name="joint3_motor">
-                <mechanicalReduction>-995.000875</mechanicalReduction>
+                <mechanicalReduction>995.000875</mechanicalReduction>
             </actuator>
             <joint name="joint3">
                 <hardwareInterface>hardware_interface/EffortJointInterface</hardwareInterface>
-                <offset>-0.188893</offset>
+                <offset>0.312881</offset>
             </joint>
         </transmission>
@@ -36,9 +36,9 @@
             <type>transmission_interface/SimpleTransmission</type>
             <actuator name="joint4_motor">
-                <mechanicalReduction>328.093719</mechanicalReduction>
+                <mechanicalReduction>-328.093719</mechanicalReduction>
             </actuator>
             <joint name="joint4">
                 <hardwareInterface>hardware_interface/EffortJointInterface</hardwareInterface>
-                <offset>-0.29131929</offset>
+                <offset>-0.31346</offset>
             </joint>
         </transmission>
@@ -46,9 +46,9 @@
             <type>transmission_interface/SimpleTransmission</type>
             <actuator name="joint5_motor">
-                <mechanicalReduction>50.895</mechanicalReduction>
+                <mechanicalReduction>-50.895</mechanicalReduction>
             </actuator>
             <joint name="joint5">
                 <hardwareInterface>hardware_interface/EffortJointInterface</hardwareInterface>
-                <offset>0.010503</offset>
+                <offset>-0.009373</offset>
             </joint>
         </transmission>
@@ -56,9 +56,9 @@
             <type>transmission_interface/SimpleTransmission</type>
             <actuator name="joint6_motor">
-                <mechanicalReduction>50.895</mechanicalReduction>
+                <mechanicalReduction>-50.895</mechanicalReduction>
             </actuator>
             <joint name="joint6">
                 <hardwareInterface>hardware_interface/EffortJointInterface</hardwareInterface>
-                <offset>0.85218130</offset>
+                <offset>-0.780477</offset>
             </joint>
         </transmission>
@@ -70,5 +70,5 @@
             <joint name="joint7">
                 <hardwareInterface>hardware_interface/EffortJointInterface</hardwareInterface>
-                <offset>0.87897618</offset>
+                <offset>-1.359663</offset>
             </joint>
         </transmission>
@@ -81,5 +81,5 @@
                 <joint name="mimic_joint1">
                     <hardwareInterface>hardware_interface/EffortJointInterface</hardwareInterface>
-                    <offset>0.015</offset>
+                    <offset>-0.002099</offset>
                 </joint>
             </transmission>
@@ -87,9 +87,9 @@
                 <type>transmission_interface/SimpleTransmission</type>
                 <actuator name="mimic_joint2_motor">
-                    <mechanicalReduction>-497.500437</mechanicalReduction>
+                    <mechanicalReduction>497.500437</mechanicalReduction>
                 </actuator>
                 <joint name="mimic_joint2">
                     <hardwareInterface>hardware_interface/EffortJointInterface</hardwareInterface>
-                    <offset>-0.3062994</offset>
+                    <offset>0.294773</offset>
                 </joint>
             </transmission>
@@ -97,9 +97,9 @@
                 <type>transmission_interface/SimpleTransmission</type>
                 <actuator name="mimic_joint3_motor">
-                    <mechanicalReduction>995.000875</mechanicalReduction>
+                    <mechanicalReduction>-995.000875</mechanicalReduction>
                 </actuator>
                 <joint name="mimic_joint3">
                     <hardwareInterface>hardware_interface/EffortJointInterface</hardwareInterface>
-                    <offset>-0.1930778828</offset>
+                    <offset>0.312881</offset>
                 </joint>
             </transmission>
