Commit message: Update chassis's inertial

File: urdf/engineer/chassis.urdf.xacro (robot description, xacro)
@@ -8,7 +8,7 @@
         <link name="base_link">
             <inertial>
-                <mass value="12.252018"/>
-                <origin xyz="0.004494 0.012027 0.169606"/>
-                <inertia ixx="1.047e0" ixy="-4.114e-3" ixz="-1.395e-2" iyy="8.849e-1" iyz="-1.357e-2" izz="6.167e-1"/>
+                <mass value="14.321805"/>
+                <origin xyz="-0.011828 -0.007426 0.160123"/>
+                <inertia ixx="1.06e0" ixy="1.071e-3" ixz="3.011e-2" iyy="9.494e-1" iyz="2.344e-2" izz="7.430e-1"/>
             </inertial>
             <visual>
@@ -19,97 +19,8 @@
             </visual>
             <collision>
-                <origin xyz="-0.0486 0.2515 0.5235" rpy="0 0 0"/>
+                <origin xyz="0 0 0" rpy="0 0 0"/>
                 <geometry>
-                    <box size="0.0984 0.055 0.067"/>
-                </geometry>
-            </collision>
-            <collision>
-                <origin xyz="-0.0486 -0.2515 0.5235" rpy="0 0 0"/>
-                <geometry>
-                    <box size="0.0984 0.055 0.067"/>
-                </geometry>
-            </collision>
-            <collision>
-                <origin xyz="0.125 0.24675 0.285" rpy="0 0 0"/>
-                <geometry>
-                    <box size="0.04 0.0365 0.41"/>
-                </geometry>
-            </collision>
-            <collision>
-                <origin xyz="-0.125 0.24675 0.285" rpy="0 0 0"/>
-                <geometry>
-                    <box size="0.04 0.0365 0.41"/>
-                </geometry>
-            </collision>
-            <collision>
-                <origin xyz="0.125 -0.24675 0.285" rpy="0 0 0"/>
-                <geometry>
-                    <box size="0.04 0.0365 0.41"/>
-                </geometry>
-            </collision>
-            <collision>
-                <origin xyz="-0.125 -0.24675 0.285" rpy="0 0 0"/>
-                <geometry>
-                    <box size="0.04 0.0365 0.41"/>
-                </geometry>
-            </collision>
-            <collision>
-                <origin xyz="0.125 0. 0.06" rpy="0 0 0"/>
-                <geometry>
-                    <box size="0.04 0.59 0.04"/>
-                </geometry>
-            </collision>
-            <collision>
-                <origin xyz="-0.125 0. 0.06" rpy="0 0 0"/>
-                <geometry>
-                    <box size="0.04 0.59 0.04"/>
-                </geometry>
-            </collision>
-            <collision>
-                <origin xyz="0. 0.115076 0.02" rpy="0 0 0"/>
-                <geometry>
-                    <box size="0.55 0.04 0.04"/>
-                </geometry>
-            </collision>
-            <collision>
-                <origin xyz="0. -0.115076 0.02" rpy="0 0 0"/>
-                <geometry>
-                    <box size="0.55 0.04 0.04"/>
-                </geometry>
-            </collision>
-            <collision>
-                <origin xyz="0.285 0.185 0.03" rpy="0 0 0"/>
-                <geometry>
-                    <box size="0.02 0.22 0.02"/>
-                </geometry>
-            </collision>
-            <collision>
-                <origin xyz="-0.285 0.185 0.03" rpy="0 0 0"/>
-                <geometry>
-                    <box size="0.02 0.22 0.02"/>
-                </geometry>
-            </collision>
-            <collision>
-                <origin xyz="0.285 -0.185 0.03" rpy="0 0 0"/>
-                <geometry>
-                    <box size="0.02 0.22 0.02"/>
-                </geometry>
-            </collision>
-            <collision>
-                <origin xyz="-0.285 -0.185 0.03" rpy="0 0 0"/>
-                <geometry>
-                    <box size="0.02 0.22 0.02"/>
-                </geometry>
-            </collision>
-            <collision>
-                <origin xyz="0. 0.285 0.03" rpy="0 0 0"/>
-                <geometry>
-                    <box size="0.59 0.02 0.02"/>
-                </geometry>
-            </collision>
-            <collision>
-                <origin xyz="0. -0.285 0.03" rpy="0 0 0"/>
-                <geometry>
-                    <box size="0.59 0.02 0.02"/>
+                    <mesh filename="package://rm_description/meshes/engineer/base_collision.stl"
+                          scale="0.001 0.001 0.001"/>
                 </geometry>
             </collision>
@@ -128,10 +39,4 @@
                 </geometry>
             </visual>
-            <collision>
-                <geometry>
-                    <mesh filename="package://rm_description/meshes/engineer/card_collision1.stl"
-                          scale="0.001 0.001 0.001"/>
-                </geometry>
-            </collision>
         </link>
         <link name="drag">
@@ -149,36 +54,23 @@
                 </geometry>
             </visual>
-            <collision>
-                <origin xyz="0 0 0" rpy="0 0 0"/>
-                <geometry>
-                    <mesh filename="package://rm_description/meshes/engineer/drag_collision.stl"
-                          scale="0.001 0.001 0.001"/>
-                </geometry>
-            </collision>
-            <collision>
-                <origin xyz="-0.041518 -0.077 0.017" rpy="0 0 0"/>
-                <geometry>
-                    <box size="0.112768 0.009 0.018"/>
-                </geometry>
-            </collision>
         </link>
-        <joint name="card_joint" type="revolute">
+        <joint name="card_joint" type="prismatic">
             <parent link="base_link"/>
             <child link="card"/>
-            <origin xyz="0.244 -0.0585 0.036" rpy="0 0 -1.57"/>
-            <axis xyz="1 0 0"/>
-            <limit lower="-1000000" upper="1000000" velocity="1" effort="200"/>
+            <origin xyz="0.244 0. 0.036" rpy="0 0 -1.57"/>
+            <axis xyz="0 1 0"/>
+            <limit lower="0" upper="0.36" velocity="1" effort="200"/>
         </joint>
         <joint name="drag_joint" type="revolute">
             <parent link="base_link"/>
             <child link="drag"/>
-            <origin xyz="-0.245 0 0.06" rpy="0 0 3.14"/>
+            <origin xyz="0.245 0 0.06" rpy="0 0 0"/>
             <axis xyz="0 1 0"/>
-            <limit lower="-1.6" upper="-0.01" velocity="1" effort="200"/>
+            <limit lower="-10" upper="10" velocity="1" effort="200"/>
         </joint>
         <transmission name="trans_card_joint">
             <type>transmission_interface/SimpleTransmission</type>
             <actuator name="card_joint_motor">
-                <mechanicalReduction>36</mechanicalReduction>
+                <mechanicalReduction>1800</mechanicalReduction>
             </actuator>
             <joint name="card_joint">
@@ -193,5 +85,5 @@
             </actuator>
             <joint name="drag_joint">
-                <offset>-1.625664</offset>
+                <offset>-1.5749</offset>
                 <hardwareInterface>hardware_interface/EffortJointInterface</hardwareInterface>
             </joint>

Commit message: Update base_link's collision and joint's limit

File: urdf/engineer/chassis.urdf.xacro (robot description, xacro)
@@ -23,4 +23,16 @@
                     <mesh filename="package://rm_description/meshes/engineer/base_collision.stl"
                           scale="0.001 0.001 0.001"/>
+                </geometry>
+            </collision>
+            <collision>
+                <origin xyz="0 0.251 0.447" rpy="0 0 0"/>
+                <geometry>
+                    <box size="0.28 0.035 0.567"/>
+                </geometry>
+            </collision>
+            <collision>
+                <origin xyz="0 -0.251 0.447" rpy="0 0 0"/>
+                <geometry>
+                    <box size="0.28 0.035 0.567"/>
                 </geometry>
             </collision>
@@ -60,5 +72,5 @@
             <origin xyz="0.244 0. 0.036" rpy="0 0 -1.57"/>
             <axis xyz="0 1 0"/>
-            <limit lower="0" upper="0.36" velocity="1" effort="200"/>
+            <limit lower="-2" upper="0.6" velocity="1" effort="200"/>
         </joint>
         <joint name="drag_joint" type="revolute">
@@ -67,5 +79,5 @@
             <origin xyz="0.245 0 0.06" rpy="0 0 0"/>
             <axis xyz="0 1 0"/>
-            <limit lower="-10" upper="10" velocity="1" effort="200"/>
+            <limit lower="-0.1" upper="0.1" velocity="1" effort="200"/>
         </joint>
         <transmission name="trans_card_joint">
@@ -101,8 +113,8 @@
                             x_offset="${-wheel_track/2}" y_offset="${-wheel_base/2}"
                             z_offset="${wheel_offset_z}"/>
-        <xacro:swerve_transmission prefix="left_front" wheel_reduction="13" pivot_offset="6.288554632"/>
-        <xacro:swerve_transmission prefix="right_front" wheel_reduction="13" pivot_offset="3.11052562"/>
-        <xacro:swerve_transmission prefix="left_back" wheel_reduction="13" pivot_offset="2.101043076"/>
-        <xacro:swerve_transmission prefix="right_back" wheel_reduction="13" pivot_offset="5.472377256"/>
+        <xacro:swerve_transmission prefix="left_front" wheel_reduction="-13" pivot_offset="1.3086453"/>
+        <xacro:swerve_transmission prefix="right_front" wheel_reduction="-13" pivot_offset="6.238694172"/>
+        <xacro:swerve_transmission prefix="left_back" wheel_reduction="-13" pivot_offset="7.3548013"/>
+        <xacro:swerve_transmission prefix="right_back" wheel_reduction="-13" pivot_offset="2.3304011"/>
     </xacro:macro>
 </robot>

Commit message: Modified the card_joint's lower_limit

File: urdf/engineer/chassis.urdf.xacro (robot description, xacro)
@@ -72,5 +72,5 @@
             <origin xyz="0.244 0. 0.036" rpy="0 0 -1.57"/>
             <axis xyz="0 1 0"/>
-            <limit lower="-2" upper="0.6" velocity="1" effort="200"/>
+            <limit lower="-0.01" upper="0.6" velocity="1" effort="200"/>
         </joint>
         <joint name="drag_joint" type="revolute">

Commit message: Update the limit

File: urdf/engineer/chassis.urdf.xacro (robot description, xacro)
@@ -79,5 +79,5 @@
             <origin xyz="0.245 0 0.06" rpy="0 0 0"/>
             <axis xyz="0 1 0"/>
-            <limit lower="-0.1" upper="0.1" velocity="1" effort="200"/>
+            <limit lower="-10" upper="20" velocity="1" effort="200"/>
         </joint>
         <transmission name="trans_card_joint">
@@ -97,5 +97,5 @@
             </actuator>
             <joint name="drag_joint">
-                <offset>-1.5749</offset>
+                <offset>0</offset>
                 <hardwareInterface>hardware_interface/EffortJointInterface</hardwareInterface>
             </joint>

File: urdf/engineer/gimbal.urdf.xacro (robot description, xacro)
@@ -64,8 +64,5 @@
                     rpy="0 0 0"/>
             <dynamics damping="0.0" friction="0.1"/>
-            <limit effort="0.25" velocity="1000" lower="-4.3" upper="0.3"/>
-            <safety_controller k_position="0.8" k_velocity="0.04"
-                               soft_lower_limit="-4.25"
-                               soft_upper_limit="0.25"/>
+            <limit effort="0.25" velocity="1000" lower="-4.26" upper="0.45"/>
             <parent link="gimbal_base"/>
             <child link="yaw"/>
@@ -75,5 +72,5 @@
             <origin xyz="0.  0. 0.056 " rpy="0 0 0"/>
             <dynamics damping="0.0" friction="0.1"/>
-            <limit effort="1.2" velocity="30" lower="-1" upper="1"/>
+            <limit effort="0.045" velocity="30" lower="-1000" upper="1000"/>
             <parent link="yaw"/>
             <child link="pitch"/>
@@ -86,5 +83,5 @@
             </actuator>
             <joint name="yaw_joint">
-                <offset>0.03911</offset>
+                <offset>0.467</offset>
                 <hardwareInterface>hardware_interface/EffortJointInterface</hardwareInterface>
             </joint>
@@ -96,5 +93,5 @@
             </actuator>
             <joint name="pitch_joint">
-                <offset>0.777728</offset>
+                <offset>0.74321</offset>
                 <hardwareInterface>hardware_interface/EffortJointInterface</hardwareInterface>
             </joint>

Commit message: Increase card and drag's velocity

File: urdf/engineer/chassis.urdf.xacro (robot description, xacro)
@@ -72,5 +72,5 @@
             <origin xyz="0.244 0. 0.036" rpy="0 0 -1.57"/>
             <axis xyz="0 1 0"/>
-            <limit lower="-0.01" upper="0.6" velocity="1" effort="200"/>
+            <limit lower="-0.01" upper="0.6" velocity="3" effort="200"/>
         </joint>
         <joint name="drag_joint" type="revolute">
@@ -79,5 +79,5 @@
             <origin xyz="0.245 0 0.06" rpy="0 0 0"/>
             <axis xyz="0 1 0"/>
-            <limit lower="-10" upper="20" velocity="1" effort="200"/>
+            <limit lower="-10" upper="20" velocity="6" effort="200"/>
         </joint>
         <transmission name="trans_card_joint">

Commit message: Update gimbal's limit

File: urdf/engineer/chassis.urdf.xacro (robot description, xacro)
@@ -113,8 +113,8 @@
                             x_offset="${-wheel_track/2}" y_offset="${-wheel_base/2}"
                             z_offset="${wheel_offset_z}"/>
-        <xacro:swerve_transmission prefix="left_front" wheel_reduction="13" pivot_offset="-1.806482"/>
-        <xacro:swerve_transmission prefix="right_front" wheel_reduction="13" pivot_offset="0.7317981"/>
-        <xacro:swerve_transmission prefix="left_back" wheel_reduction="13" pivot_offset="-2.032005516"/>
-        <xacro:swerve_transmission prefix="right_back" wheel_reduction="13" pivot_offset="0.807739452"/>
+        <xacro:swerve_transmission prefix="left_front" wheel_reduction="13" pivot_offset="4.481304"/>
+        <xacro:swerve_transmission prefix="right_front" wheel_reduction="13" pivot_offset="0.733332"/>
+        <xacro:swerve_transmission prefix="left_back" wheel_reduction="13" pivot_offset="4.25117"/>
+        <xacro:swerve_transmission prefix="right_back" wheel_reduction="13" pivot_offset="0.80697"/>
     </xacro:macro>
 </robot>

File: urdf/engineer/gimbal.urdf.xacro (robot description, xacro)
@@ -3,4 +3,9 @@
     <!-- safety_distance: Minimum safety distance in [m] by which the collision volumes are expanded and which is enforced during robot motions -->
     <xacro:macro name="gimbal" params="connected_to:='' xyz:='0 0 0' rpy:='0 0 0' simulation">
+        <xacro:property name="threshold" value="0.03"/>
+        <xacro:property name="yaw_lower_limit" value="-4.235"/>
+        <xacro:property name="yaw_upper_limit" value="0.48"/>
+        <xacro:property name="pitch_lower_limit" value="-1.07"/>
+        <xacro:property name="pitch_upper_limit" value="0.76"/>
         <link name="gimbal_base">
             <inertial>
@@ -64,5 +69,8 @@
                     rpy="0 0 0"/>
             <dynamics damping="0.0" friction="0.1"/>
-            <limit effort="0.25" velocity="1000" lower="-5" upper="0"/>
+            <limit effort="1.2" velocity="13.82" lower="${yaw_lower_limit}" upper="${yaw_upper_limit}"/>
+            <safety_controller k_position="100" k_velocity="0.1"
+                               soft_lower_limit="${yaw_lower_limit+threshold}"
+                               soft_upper_limit="${yaw_upper_limit-threshold}"/>
             <parent link="gimbal_base"/>
             <child link="yaw"/>
@@ -72,5 +80,8 @@
             <origin xyz="0.  0. 0.056 " rpy="0 0 0"/>
             <dynamics damping="0.0" friction="0.1"/>
-            <limit effort="0.045" velocity="30" lower="-1000" upper="1000"/>
+            <limit effort="1.2" velocity="13.82" lower="${pitch_lower_limit}" upper="${pitch_upper_limit}"/>
+            <safety_controller k_position="100" k_velocity="0.1"
+                               soft_lower_limit="${pitch_lower_limit+threshold}"
+                               soft_upper_limit="${pitch_upper_limit-threshold}"/>
             <parent link="yaw"/>
             <child link="pitch"/>

Commit message: Delete unnecessary collision of base_link

File: urdf/engineer/chassis.urdf.xacro (robot description, xacro)
@@ -23,16 +23,4 @@
                     <mesh filename="package://rm_description/meshes/engineer/base_collision.stl"
                           scale="0.001 0.001 0.001"/>
-                </geometry>
-            </collision>
-            <collision>
-                <origin xyz="0 0.251 0.387" rpy="0 0 0"/>
-                <geometry>
-                    <box size="0.43 0.0387 0.567"/>
-                </geometry>
-            </collision>
-            <collision>
-                <origin xyz="0 -0.251 0.407" rpy="0 0 0"/>
-                <geometry>
-                    <box size="0.43 0.0387 0.567"/>
                 </geometry>
             </collision>

Commit message: Improve the steps list

File: urdf/engineer/chassis.urdf.xacro (robot description, xacro)
@@ -47,4 +47,22 @@
                 <geometry>
                     <box size="0.061 0.042 0.4"/>
+                </geometry>
+            </collision>
+            <collision>
+                <origin xyz="-0.175 0.247 0.275" rpy="0 0 0"/>
+                <geometry>
+                    <box size="0.061 0.042 0.4"/>
+                </geometry>
+            </collision>
+            <collision>
+                <origin xyz="0. -0.255 0.51" rpy="0 0 0"/>
+                <geometry>
+                    <box size="0.386 0.06 0.06"/>
+                </geometry>
+            </collision>
+            <collision>
+                <origin xyz="0. 0.255 0.51" rpy="0 0 0"/>
+                <geometry>
+                    <box size="0.386 0.06 0.06"/>
                 </geometry>
             </collision>

File: urdf/engineer/gimbal.urdf.xacro (robot description, xacro)
@@ -3,9 +3,9 @@
     <!-- safety_distance: Minimum safety distance in [m] by which the collision volumes are expanded and which is enforced during robot motions -->
     <xacro:macro name="gimbal" params="connected_to:='' xyz:='0 0 0' rpy:='0 0 0' simulation">
-        <xacro:property name="threshold" value="0.03"/>
-        <xacro:property name="yaw_lower_limit" value="-4.235"/>
-        <xacro:property name="yaw_upper_limit" value="0.48"/>
-        <xacro:property name="pitch_lower_limit" value="-1.07"/>
-        <xacro:property name="pitch_upper_limit" value="0.76"/>
+        <xacro:property name="threshold" value="0.04"/>
+        <xacro:property name="yaw_lower_limit" value="-4.18"/>
+        <xacro:property name="yaw_upper_limit" value="0.88"/>
+        <xacro:property name="pitch_lower_limit" value="-0.91"/>
+        <xacro:property name="pitch_upper_limit" value="0.91"/>
         <link name="gimbal_base">
             <inertial>
@@ -70,7 +70,4 @@
             <dynamics damping="0.0" friction="0.1"/>
             <limit effort="900" velocity="0.17" lower="${yaw_lower_limit}" upper="${yaw_upper_limit}"/>
-            <safety_controller k_position="100" k_velocity="0.1"
-                               soft_lower_limit="${yaw_lower_limit+threshold}"
-                               soft_upper_limit="${yaw_upper_limit-threshold}"/>
             <parent link="gimbal_base"/>
             <child link="yaw"/>
@@ -81,7 +78,4 @@
             <dynamics damping="0.0" friction="0.1"/>
             <limit effort="900" velocity="0.17" lower="${pitch_lower_limit}" upper="${pitch_upper_limit}"/>
-            <safety_controller k_position="100" k_velocity="0.1"
-                               soft_lower_limit="${pitch_lower_limit+threshold}"
-                               soft_upper_limit="${pitch_upper_limit-threshold}"/>
             <parent link="yaw"/>
             <child link="pitch"/>
@@ -94,5 +88,5 @@
             </actuator>
             <joint name="yaw_joint">
-                <offset>0.467</offset>
+                <offset>0.7524</offset>
                 <hardwareInterface>hardware_interface/EffortJointInterface</hardwareInterface>
             </joint>
@@ -104,5 +98,5 @@
             </actuator>
             <joint name="pitch_joint">
-                <offset>0.74321</offset>
+                <offset>0.9019</offset>
                 <hardwareInterface>hardware_interface/EffortJointInterface</hardwareInterface>
             </joint>

Commit message: Update new collision

File: urdf/engineer/chassis.urdf.xacro (robot description, xacro)
@@ -34,5 +34,5 @@
                 <origin xyz="0.175 0.247 0.275" rpy="0 0 0"/>
                 <geometry>
-                    <box size="0.061 0.042 0.4"/>
+                    <box size="0.081 0.042 0.4"/>
                 </geometry>
             </collision>
@@ -40,5 +40,5 @@
                 <origin xyz="-0.175 -0.247 0.275" rpy="0 0 0"/>
                 <geometry>
-                    <box size="0.061 0.042 0.4"/>
+                    <box size="0.081 0.042 0.4"/>
                 </geometry>
             </collision>
@@ -46,5 +46,5 @@
                 <origin xyz="0.175 -0.247 0.275" rpy="0 0 0"/>
                 <geometry>
-                    <box size="0.061 0.042 0.4"/>
+                    <box size="0.081 0.042 0.4"/>
                 </geometry>
             </collision>
@@ -52,5 +52,5 @@
                 <origin xyz="-0.175 0.247 0.275" rpy="0 0 0"/>
                 <geometry>
-                    <box size="0.061 0.042 0.4"/>
+                    <box size="0.081 0.042 0.4"/>
                 </geometry>
             </collision>
@@ -58,5 +58,5 @@
                 <origin xyz="0. -0.255 0.51" rpy="0 0 0"/>
                 <geometry>
-                    <box size="0.386 0.06 0.06"/>
+                    <box size="0.41 0.06 0.09"/>
                 </geometry>
             </collision>
@@ -64,8 +64,7 @@
                 <origin xyz="0. 0.255 0.51" rpy="0 0 0"/>
                 <geometry>
-                    <box size="0.386 0.06 0.06"/>
+                    <box size="0.41 0.06 0.09"/>
                 </geometry>
             </collision>
-            <selfCollide>true</selfCollide>
         </link>
         <link name="card">
