Commit message: Update the joint's limit

File: urdf/engineer/arm.urdf.xacro (robot description, xacro)
@@ -3,18 +3,18 @@
     <xacro:macro name="arm" params="connected_to">
         <xacro:property name="threshold" value="0.1"/>
-        <xacro:property name="joint1_lower_limit" value="0"/>
-        <xacro:property name="joint1_upper_limit" value="0.3"/>
-        <xacro:property name="joint2_lower_limit" value="-0.253350256769"/>
-        <xacro:property name="joint2_upper_limit" value="0.385167154"/>
-        <xacro:property name="joint3_lower_limit" value="-0.229388728029366"/>
-        <xacro:property name="joint3_upper_limit" value="0.281850996668"/>
-        <xacro:property name="joint4_lower_limit" value="-0.40983099899072"/>
-        <xacro:property name="joint4_upper_limit" value="0.43667063"/>
-        <xacro:property name="joint5_lower_limit" value="-3.42203741234"/>
-        <xacro:property name="joint5_upper_limit" value="0.047983045788"/>
-        <xacro:property name="joint6_lower_limit" value="-4.327149605070"/>
-        <xacro:property name="joint6_upper_limit" value="0.593107173715"/>
-        <xacro:property name="joint7_lower_limit" value="-1.507979833"/>
-        <xacro:property name="joint7_upper_limit" value="4.03879746213"/>
+        <xacro:property name="joint1_lower_limit" value="0.0045"/>
+        <xacro:property name="joint1_upper_limit" value="0.6274"/>
+        <xacro:property name="joint2_upper_limit" value="0.34363"/>
+        <xacro:property name="joint2_lower_limit" value="-0.2124"/>
+        <xacro:property name="joint3_upper_limit" value="0.2360"/>
+        <xacro:property name="joint3_lower_limit" value="-0.2219"/>
+        <xacro:property name="joint4_upper_limit" value="0.34125"/>
+        <xacro:property name="joint4_lower_limit" value="-0.295"/>
+        <xacro:property name="joint5_upper_limit" value="0"/>
+        <xacro:property name="joint5_lower_limit" value="-3.2301"/>
+        <xacro:property name="joint6_upper_limit" value="0.8005"/>
+        <xacro:property name="joint6_lower_limit" value="-4.2"/>
+        <xacro:property name="joint7_upper_limit" value="3.99"/>
+        <xacro:property name="joint7_lower_limit" value="-1.26"/>
         <!--  link  -->
         <link name="link1">
@@ -251,6 +251,5 @@
             <origin xyz="0 0 0.1375" rpy="0 0 0"/>
             <axis xyz="0 0 1"/>
-            <limit lower="${joint1_lower_limit}" upper="${joint1_upper_limit}" velocity="100"
-                   effort="10"/>
+            <limit lower="${joint1_lower_limit}" upper="${joint1_upper_limit}" velocity="200" effort="20"/>
         </joint>
         <joint name="joint2" type="prismatic">
@@ -259,6 +258,5 @@
             <origin xyz="0. 0. 0.098707" rpy="0 0 0"/>
             <axis xyz="1 0 0"/>
-            <limit lower="${joint2_lower_limit}" upper="${joint2_upper_limit}" velocity="100"
-                   effort="10"/>
+            <limit lower="${joint2_lower_limit}" upper="${joint2_upper_limit}" velocity="200" effort="20"/>
         </joint>
         <joint name="joint3" type="prismatic">
@@ -267,5 +265,5 @@
             <origin xyz="0.022 0. 0.034" rpy="0 0 0"/>
             <axis xyz="1 0 0"/>
-            <limit lower="${joint3_lower_limit}" upper="${joint3_upper_limit}" velocity="100" effort="10"/>
+            <limit lower="${joint3_lower_limit}" upper="${joint3_upper_limit}" velocity="200" effort="20"/>
         </joint>
         <joint name="joint4" type="prismatic">
@@ -274,6 +272,5 @@
             <origin xyz="0. 0. 0.068" rpy="0 0 0"/>
             <axis xyz="0 1 0"/>
-            <limit lower="${joint4_lower_limit}" upper="${joint4_upper_limit}" velocity="100"
-                   effort="10"/>
+            <limit lower="${joint4_lower_limit}" upper="${joint4_upper_limit}" velocity="200" effort="20"/>
         </joint>
         <joint name="joint5" type="revolute">
@@ -282,6 +279,5 @@
             <origin xyz="0. 0. 0.069" rpy="0 0 0"/>
             <axis xyz="0 1 0"/>
-            <limit lower="${joint5_lower_limit}" upper="${joint5_upper_limit}" velocity="100"
-                   effort="10"/>
+            <limit lower="${joint5_lower_limit}" upper="${joint5_upper_limit}" velocity="200" effort="20"/>
         </joint>
         <joint name="joint6" type="revolute">
@@ -290,6 +286,5 @@
             <origin xyz="0.06925 0. 0" rpy="0 0 0"/>
             <axis xyz="1 0 0"/>
-            <limit lower="${joint6_lower_limit}" upper="${joint6_upper_limit}" velocity="100"
-                   effort="10"/>
+            <limit lower="${joint6_lower_limit}" upper="${joint6_upper_limit}" velocity="200" effort="20"/>
         </joint>
         <joint name="joint7" type="revolute">
@@ -298,6 +293,5 @@
             <origin xyz="-0.06925 0 0.255" rpy="0 0 0"/>
             <axis xyz="0 0 1"/>
-            <limit lower="${joint7_lower_limit}" upper="${joint7_upper_limit}" velocity="100"
-                   effort="10"/>
+            <limit lower="${joint7_lower_limit}" upper="${joint7_upper_limit}" velocity="200" effort="20"/>
         </joint>
     </xacro:macro>

Commit message: Update the joint's limit and max vel effort

File: urdf/engineer/arm.urdf.xacro (robot description, xacro)
@@ -3,18 +3,18 @@
     <xacro:macro name="arm" params="connected_to">
         <xacro:property name="threshold" value="0.1"/>
-        <xacro:property name="joint1_lower_limit" value="0.0045"/>
-        <xacro:property name="joint1_upper_limit" value="0.6274"/>
-        <xacro:property name="joint2_upper_limit" value="0.34363"/>
-        <xacro:property name="joint2_lower_limit" value="-0.2124"/>
-        <xacro:property name="joint3_upper_limit" value="0.2360"/>
-        <xacro:property name="joint3_lower_limit" value="-0.2219"/>
-        <xacro:property name="joint4_upper_limit" value="0.34125"/>
-        <xacro:property name="joint4_lower_limit" value="-0.295"/>
-        <xacro:property name="joint5_upper_limit" value="0"/>
-        <xacro:property name="joint5_lower_limit" value="-3.2301"/>
-        <xacro:property name="joint6_upper_limit" value="0.8005"/>
-        <xacro:property name="joint6_lower_limit" value="-4.2"/>
-        <xacro:property name="joint7_upper_limit" value="3.99"/>
-        <xacro:property name="joint7_lower_limit" value="-1.26"/>
+        <xacro:property name="joint1_lower_limit" value="0.0005736069829"/>
+        <xacro:property name="joint1_upper_limit" value="0.6351414275302"/>
+        <xacro:property name="joint2_upper_limit" value="0.3438321773"/>
+        <xacro:property name="joint2_lower_limit" value="-0.2253643418193"/>
+        <xacro:property name="joint3_upper_limit" value="0.2362959079343"/>
+        <xacro:property name="joint3_lower_limit" value="-0.2253360962"/>
+        <xacro:property name="joint4_upper_limit" value="0.34152550806"/>
+        <xacro:property name="joint4_lower_limit" value="-0.296310718475"/>
+        <xacro:property name="joint5_upper_limit" value="-0.00022605078282"/>
+        <xacro:property name="joint5_lower_limit" value="-3.23240560816"/>
+        <xacro:property name="joint6_upper_limit" value="0.798170237718"/>
+        <xacro:property name="joint6_lower_limit" value="-4.2362368464"/>
+        <xacro:property name="joint7_upper_limit" value="3.979137624343"/>
+        <xacro:property name="joint7_lower_limit" value="-1.26312636630"/>
         <!--  link  -->
         <link name="link1">
@@ -251,5 +251,5 @@
             <origin xyz="0 0 0.1375" rpy="0 0 0"/>
             <axis xyz="0 0 1"/>
-            <limit lower="${joint1_lower_limit}" upper="${joint1_upper_limit}" velocity="200" effort="20"/>
+            <limit lower="${joint1_lower_limit}" upper="${joint1_upper_limit}" velocity="1" effort="200"/>
         </joint>
         <joint name="joint2" type="prismatic">
@@ -258,5 +258,5 @@
             <origin xyz="0. 0. 0.098707" rpy="0 0 0"/>
             <axis xyz="1 0 0"/>
-            <limit lower="${joint2_lower_limit}" upper="${joint2_upper_limit}" velocity="200" effort="20"/>
+            <limit lower="${joint2_lower_limit}" upper="${joint2_upper_limit}" velocity="1" effort="200"/>
         </joint>
         <joint name="joint3" type="prismatic">
@@ -265,5 +265,5 @@
             <origin xyz="0.022 0. 0.034" rpy="0 0 0"/>
             <axis xyz="1 0 0"/>
-            <limit lower="${joint3_lower_limit}" upper="${joint3_upper_limit}" velocity="200" effort="20"/>
+            <limit lower="${joint3_lower_limit}" upper="${joint3_upper_limit}" velocity="1" effort="200"/>
         </joint>
         <joint name="joint4" type="prismatic">
@@ -272,5 +272,5 @@
             <origin xyz="0. 0. 0.068" rpy="0 0 0"/>
             <axis xyz="0 1 0"/>
-            <limit lower="${joint4_lower_limit}" upper="${joint4_upper_limit}" velocity="200" effort="20"/>
+            <limit lower="${joint4_lower_limit}" upper="${joint4_upper_limit}" velocity="1" effort="200"/>
         </joint>
         <joint name="joint5" type="revolute">
@@ -279,19 +279,19 @@
             <origin xyz="0. 0. 0.069" rpy="0 0 0"/>
             <axis xyz="0 1 0"/>
-            <limit lower="${joint5_lower_limit}" upper="${joint5_upper_limit}" velocity="200" effort="20"/>
-        </joint>
-        <joint name="joint6" type="revolute">
+            <limit lower="${joint5_lower_limit}" upper="${joint5_upper_limit}" velocity="10" effort="200"/>
+        </joint>
+        <joint name="joint6" type="revolute">50.895
             <parent link="link4"/>
             <child link="link5"/>
             <origin xyz="0.06925 0. 0" rpy="0 0 0"/>
             <axis xyz="1 0 0"/>
-            <limit lower="${joint6_lower_limit}" upper="${joint6_upper_limit}" velocity="200" effort="20"/>
-        </joint>
-        <joint name="joint7" type="revolute">
+            <limit lower="${joint6_lower_limit}" upper="${joint6_upper_limit}" velocity="10" effort="200"/>
+        </joint>
+        <joint name="joint7" type="revolute">19.2032
             <parent link="link5"/>
             <child link="link6"/>
             <origin xyz="-0.06925 0 0.255" rpy="0 0 0"/>
             <axis xyz="0 0 1"/>
-            <limit lower="${joint7_lower_limit}" upper="${joint7_upper_limit}" velocity="200" effort="20"/>
+            <limit lower="${joint7_lower_limit}" upper="${joint7_upper_limit}" velocity="10" effort="200"/>
         </joint>
     </xacro:macro>

Commit message: Add hold card and chassis's urdf

File: urdf/engineer/arm.urdf.xacro (robot description, xacro)
@@ -359,5 +359,5 @@
             <limit lower="${joint5_lower_limit}" upper="${joint5_upper_limit}" velocity="10" effort="200"/>
         </joint>
-        <joint name="joint6" type="revolute">50.895
+        <joint name="joint6" type="revolute">
             <parent link="link4"/>
             <child link="link5"/>
@@ -366,5 +366,5 @@
             <limit lower="${joint6_lower_limit}" upper="${joint6_upper_limit}" velocity="10" effort="200"/>
         </joint>
-        <joint name="joint7" type="revolute">19.2032
+        <joint name="joint7" type="revolute">
             <parent link="link5"/>
             <child link="link6"/>

File: urdf/engineer/chassis.urdf.xacro (robot description, xacro)
@@ -1,3 +1,7 @@
 <robot xmlns:xacro="http://www.ros.org/wiki/xacro" name="chassis">
+    <xacro:include filename="$(find rm_description)/urdf/common/swerve_drive.urdf.xacro"/>
+    <xacro:property name="wheel_track" value="0.416152"/>
+    <xacro:property name="wheel_base" value="0.416152"/>
+    <xacro:property name="wheel_offset_z" value="0.06"/>
     <xacro:macro name="chassis" params="roller_type">
         <link name="base_link">
@@ -68,4 +72,97 @@
             </collision>
         </link>
+        <joint name="fixed" type="fixed">
+            <parent link="base_link"/>
+            <child link="base_chassis"/>
+            <origin xyz="0. 0. 0.04" rpy="0 0 0"/>
+        </joint>
+        <link name="base_chassis">
+            <inertial>
+                <mass value="4.947"/>
+                <origin xyz="0.012487 0.000034 0.341608"/>
+                <inertia ixx="1.617e3" ixy="-3.511e-4" ixz="-2.127e1" iyy="1.616e3" iyz="-1.559e-2" izz="1.723e3"/>
+            </inertial>
+            <visual>
+                <origin xyz="0 0 0" rpy="0 0 0"/>
+                <geometry>
+                    <mesh filename="package://rm_description/meshes/engineer/base_chassis.stl"
+                          scale="0.001 0.001 0.001"/>
+                </geometry>
+            </visual>
+            <collision>
+                <origin xyz="0.0285 -0.2685 0.5" rpy="0 0 0"/>
+                <geometry>
+                    <box size="0.153 0.035 0.040"/>
+                </geometry>
+            </collision>
+        </link>
+        <joint name="jointx" type="prismatic">
+            <parent link="base_chassis"/>
+            <child link="card"/>
+            <origin xyz="-0.2825 -0.001 0.005" rpy="0 0 0"/>
+            <axis xyz="1 0 0"/>
+            <limit lower="-0.1" upper="0.1" velocity="1" effort="200"/>
+        </joint>
+        <link name="card">
+            <inertial>
+                <mass value="0.404078"/>
+                <origin xyz="0.006702 0.071531 0.019438"/>
+                <inertia ixx="3.645e-3" ixy="-2.951e-4" ixz="-8.7675418e-5" iyy="1.235e-3" iyz="-8.535e-4"
+                         izz="4.126e-3"/>
+            </inertial>
+            <visual>
+                <origin xyz="0 0 0" rpy="0 0 0"/>
+                <geometry>
+                    <mesh filename="package://rm_description/meshes/engineer/card.stl"
+                          scale="0.001 0.001 0.001"/>
+                </geometry>
+            </visual>
+            <collision>
+                <origin xyz="0.0285 -0.2685 0.5" rpy="0 0 0"/>
+                <geometry>
+                    <box size="0.153 0.035 0.040"/>
+                </geometry>
+            </collision>
+        </link>
+        <joint name="jointx1" type="revolute">
+            <parent link="base_chassis"/>
+            <child link="hold"/>
+            <origin xyz="-0.245 -0.000076 0.06" rpy="0 0 0"/>
+            <axis xyz="0 1 0"/>
+            <limit lower="-6.28" upper="6.28" velocity="1" effort="200"/>
+        </joint>
+        <link name="hold">
+            <inertial>
+                <mass value="0.404078"/>
+                <origin xyz="0.006702 0.071531 0.019438"/>
+                <inertia ixx="3.645e-3" ixy="-2.951e-4" ixz="-8.7675418e-5" iyy="1.235e-3" iyz="-8.535e-4"
+                         izz="4.126e-3"/>
+            </inertial>
+            <visual>
+                <origin xyz="-0.245 -0.000076 0.06" rpy="0 0 0"/>
+                <geometry>
+                    <mesh filename="package://rm_description/meshes/engineer/hold.stl"
+                          scale="0.001 0.001 0.001"/>
+                </geometry>
+            </visual>
+            <collision>
+                <origin xyz="0.0285 -0.2685 0.5" rpy="0 0 0"/>
+                <geometry>
+                    <box size="0.153 0.035 0.040"/>
+                </geometry>
+            </collision>
+        </link>
+        <xacro:swerve_drive prefix="left_front" connected_to="base_chassis"
+                            wheel_x_offset="${wheel_track/2}" wheel_y_offset="${wheel_base/2}"
+                            wheel_z_offset="${wheel_offset_z}"/>
+        <xacro:swerve_drive prefix="right_front" connected_to="base_chassis"
+                            wheel_x_offset="${wheel_track/2}" wheel_y_offset="${-wheel_base/2}"
+                            wheel_z_offset="${wheel_offset_z}"/>
+        <xacro:swerve_drive prefix="left_back" connected_to="base_chassis"
+                            wheel_x_offset="${-wheel_track/2}" wheel_y_offset="${wheel_base/2}"
+                            wheel_z_offset="${wheel_offset_z}"/>
+        <xacro:swerve_drive prefix="right_back" connected_to="base_chassis"
+                            wheel_x_offset="${-wheel_track/2}" wheel_y_offset="${-wheel_base/2}"
+                            wheel_z_offset="${wheel_offset_z}"/>
     </xacro:macro>
 </robot>
