Commit message: Add gpio_controller

File: urdf/engineer/arm.urdf.xacro (robot description, xacro)
@@ -6,14 +6,14 @@
         <xacro:property name="joint2_upper_limit" value="0.3"/>
         <xacro:property name="joint2_lower_limit" value="-0.35"/>
-        <xacro:property name="joint3_upper_limit" value="0.32"/>
+        <xacro:property name="joint3_upper_limit" value="0.31"/>
         <xacro:property name="joint3_lower_limit" value="-0.12"/>
-        <xacro:property name="joint4_upper_limit" value="0.32"/>
-        <xacro:property name="joint4_lower_limit" value="-0.32"/>
-        <xacro:property name="joint5_upper_limit" value="3.3"/>
+        <xacro:property name="joint4_upper_limit" value="0.31"/>
+        <xacro:property name="joint4_lower_limit" value="-0.31"/>
+        <xacro:property name="joint5_upper_limit" value="3.8445"/>
         <xacro:property name="joint5_lower_limit" value="0"/>
-        <xacro:property name="joint6_upper_limit" value="0.75"/>
-        <xacro:property name="joint6_lower_limit" value="-0.75"/>
+        <xacro:property name="joint6_upper_limit" value="0.9"/>
+        <xacro:property name="joint6_lower_limit" value="-0.9"/>
         <xacro:property name="joint7_upper_limit" value="4"/>
-        <xacro:property name="joint7_lower_limit" value="-1.4"/>
+        <xacro:property name="joint7_lower_limit" value="-1"/>
         <!--  link  -->
         <link name="link1">
@@ -97,10 +97,4 @@
                     <mesh filename="package://rm_description/meshes/engineer/link3_collision.stl"
                           scale="0.001 0.001 0.001"/>
-                </geometry>
-            </collision>
-            <collision>
-                <origin xyz="-0.04 0.153351 -0.02" rpy="0 0 0"/>
-                <geometry>
-                    <box size="0.06 0.1 0.06"/>
                 </geometry>
             </collision>
@@ -174,5 +168,5 @@
             <origin xyz="0 0 0.233" rpy="0 0 0"/>
             <axis xyz="0 0 1"/>
-            <limit lower="${joint1_lower_limit}" upper="${joint1_upper_limit}" velocity="3" effort="200"/>
+            <limit lower="${joint1_lower_limit}" upper="${joint1_upper_limit}" velocity="1.068" effort="180"/>
         </joint>
         <joint name="joint2" type="prismatic">
@@ -181,8 +175,5 @@
             <origin xyz="-0.014 0. 0.0542" rpy="0 0 0"/>
             <axis xyz="1 0 0"/>
-            <limit lower="${joint2_lower_limit}" upper="${joint2_upper_limit}" velocity="3" effort="300"/>
-            <safety_controller k_position="1800" k_velocity="15"
-                               soft_lower_limit="${joint2_lower_limit+0.01}"
-                               soft_upper_limit="${joint2_upper_limit-0.01}"/>
+            <limit lower="${joint2_lower_limit}" upper="${joint2_upper_limit}" velocity="1.9" effort="120"/>
         </joint>
         <joint name="joint3" type="prismatic">
@@ -191,8 +182,5 @@
             <origin xyz="-0.11 0. 0.013" rpy="0 0 0"/>
             <axis xyz="1 0 0"/>
-            <limit lower="${joint3_lower_limit}" upper="${joint3_upper_limit}" velocity="2" effort="300"/>
-            <safety_controller k_position="1800" k_velocity="18"
-                               soft_lower_limit="${joint3_lower_limit+0.008}"
-                               soft_upper_limit="${joint3_upper_limit-0.008}"/>
+            <limit lower="${joint3_lower_limit}" upper="${joint3_upper_limit}" velocity="0.95" effort="210"/>
         </joint>
         <joint name="joint4" type="prismatic">
@@ -201,8 +189,5 @@
             <origin xyz="0. 0. 0.078" rpy="0 0 0"/>
             <axis xyz="0 1 0"/>
-            <limit lower="${joint4_lower_limit}" upper="${joint4_upper_limit}" velocity="4.5" effort="200"/>
-            <safety_controller k_position="800" k_velocity="10"
-                               soft_lower_limit="${joint4_lower_limit+0.02}"
-                               soft_upper_limit="${joint4_upper_limit-0.02}"/>
+            <limit lower="${joint4_lower_limit}" upper="${joint4_upper_limit}" velocity="1.437" effort="105"/>
         </joint>
         <joint name="joint5" type="revolute">
@@ -211,7 +196,7 @@
             <origin xyz="0. 0. 0.02" rpy="0 0 0"/>
             <axis xyz="0 1 0"/>
-            <limit lower="${joint5_lower_limit}" upper="${joint5_upper_limit}" velocity="28.675" effort="8"/>
+            <limit lower="${joint5_lower_limit}" upper="${joint5_upper_limit}" velocity="18.53" effort="15"/>
             <safety_controller k_position="12" k_velocity="5"
-                               soft_lower_limit="${joint5_lower_limit+0}"
+                               soft_lower_limit="${joint5_lower_limit+0.03}"
                                soft_upper_limit="${joint5_upper_limit-0.1}"/>
         </joint>
@@ -221,5 +206,5 @@
             <origin xyz="-0.0585 0. 0.04875" rpy="0 0 0"/>
             <axis xyz="1 0 0"/>
-            <limit lower="${joint6_lower_limit}" upper="${joint6_upper_limit}" velocity="28.675" effort="8"/>
+            <limit lower="${joint6_lower_limit}" upper="${joint6_upper_limit}" velocity="18.53" effort="15"/>
             <safety_controller k_position="12" k_velocity="5"
                                soft_lower_limit="${joint6_lower_limit+0.1}"
@@ -231,8 +216,8 @@
             <origin xyz="0.05825 0 0.233" rpy="0 0 0"/>
             <axis xyz="0 0 1"/>
-            <limit lower="${joint7_lower_limit}" upper="${joint7_upper_limit}" velocity="76" effort="3"/>
-            <safety_controller k_position="5" k_velocity="2"
-                               soft_lower_limit="${joint7_lower_limit+0.30}"
-                               soft_upper_limit="${joint7_upper_limit-0.30}"/>
+            <limit lower="${joint7_lower_limit}" upper="${joint7_upper_limit}" velocity="49.0887" effort="7"/>
+            <safety_controller k_position="8" k_velocity="1"
+                               soft_lower_limit="${joint7_lower_limit+0.2}"
+                               soft_upper_limit="${joint7_upper_limit-0.2}"/>
         </joint>
         <xacro:unless value="${simulation}">
@@ -299,5 +284,5 @@
                 <origin xyz="0 0 10.21375" rpy="0 0 0"/>
                 <axis xyz="0 0 1"/>
-                <limit lower="${joint1_lower_limit}" upper="${joint1_upper_limit}" velocity="2" effort="200"/>
+                <limit lower="${joint1_lower_limit}" upper="${joint1_upper_limit}" velocity="1.068" effort="180"/>
             </joint>
             <joint name="mimic_joint2" type="prismatic">
@@ -306,8 +291,5 @@
                 <origin xyz="0. 0. 30.098707" rpy="0 0 0"/>
                 <axis xyz="1 0 0"/>
-                <limit lower="${joint2_lower_limit}" upper="${joint2_upper_limit}" velocity="3" effort="300"/>
-                <safety_controller k_position="1800" k_velocity="15"
-                                   soft_lower_limit="${joint2_lower_limit+0.01}"
-                                   soft_upper_limit="${joint2_upper_limit-0.01}"/>
+                <limit lower="${joint2_lower_limit}" upper="${joint2_upper_limit}" velocity="1.9" effort="120"/>
             </joint>
             <joint name="mimic_joint3" type="prismatic">
@@ -316,8 +298,5 @@
                 <origin xyz="0.022 0. 20.034" rpy="0 0 0"/>
                 <axis xyz="1 0 0"/>
-                <limit lower="${joint3_lower_limit}" upper="${joint3_upper_limit}" velocity="2" effort="300"/>
-                <safety_controller k_position="1800" k_velocity="18"
-                                   soft_lower_limit="${joint3_lower_limit+0.008}"
-                                   soft_upper_limit="${joint3_upper_limit-0.008}"/>
+                <limit lower="${joint3_lower_limit}" upper="${joint3_upper_limit}" velocity="0.95" effort="210"/>
             </joint>
         </xacro:unless>

Commit message: Update joint's velocity and effort

File: urdf/engineer/arm.urdf.xacro (robot description, xacro)
@@ -168,5 +168,5 @@
             <origin xyz="0 0 0.233" rpy="0 0 0"/>
             <axis xyz="0 0 1"/>
-            <limit lower="${joint1_lower_limit}" upper="${joint1_upper_limit}" velocity="1.068" effort="180"/>
+            <limit lower="${joint1_lower_limit}" upper="${joint1_upper_limit}" velocity="1.068" effort="230"/>
         </joint>
         <joint name="joint2" type="prismatic">
@@ -175,5 +175,5 @@
             <origin xyz="-0.014 0. 0.0542" rpy="0 0 0"/>
             <axis xyz="1 0 0"/>
-            <limit lower="${joint2_lower_limit}" upper="${joint2_upper_limit}" velocity="1.9" effort="120"/>
+            <limit lower="${joint2_lower_limit}" upper="${joint2_upper_limit}" velocity="1.93" effort="129"/>
         </joint>
         <joint name="joint3" type="prismatic">
@@ -182,5 +182,5 @@
             <origin xyz="-0.11 0. 0.013" rpy="0 0 0"/>
             <axis xyz="1 0 0"/>
-            <limit lower="${joint3_lower_limit}" upper="${joint3_upper_limit}" velocity="0.95" effort="210"/>
+            <limit lower="${joint3_lower_limit}" upper="${joint3_upper_limit}" velocity="0.965" effort="258"/>
         </joint>
         <joint name="joint4" type="prismatic">
@@ -189,5 +189,5 @@
             <origin xyz="0. 0. 0.078" rpy="0 0 0"/>
             <axis xyz="0 1 0"/>
-            <limit lower="${joint4_lower_limit}" upper="${joint4_upper_limit}" velocity="1.437" effort="105"/>
+            <limit lower="${joint4_lower_limit}" upper="${joint4_upper_limit}" velocity="1.4625" effort="170"/>
         </joint>
         <joint name="joint5" type="revolute">
@@ -196,5 +196,5 @@
             <origin xyz="0. 0. 0.02" rpy="0 0 0"/>
             <axis xyz="0 1 0"/>
-            <limit lower="${joint5_lower_limit}" upper="${joint5_upper_limit}" velocity="18.53" effort="15"/>
+            <limit lower="${joint5_lower_limit}" upper="${joint5_upper_limit}" velocity="18.53" effort="13.3"/>
             <safety_controller k_position="12" k_velocity="5"
                                soft_lower_limit="${joint5_lower_limit+0.03}"
@@ -206,5 +206,5 @@
             <origin xyz="-0.0585 0. 0.04875" rpy="0 0 0"/>
             <axis xyz="1 0 0"/>
-            <limit lower="${joint6_lower_limit}" upper="${joint6_upper_limit}" velocity="18.53" effort="15"/>
+            <limit lower="${joint6_lower_limit}" upper="${joint6_upper_limit}" velocity="18.53" effort="13.3"/>
             <safety_controller k_position="12" k_velocity="5"
                                soft_lower_limit="${joint6_lower_limit+0.1}"
@@ -216,5 +216,5 @@
             <origin xyz="0.05825 0 0.233" rpy="0 0 0"/>
             <axis xyz="0 0 1"/>
-            <limit lower="${joint7_lower_limit}" upper="${joint7_upper_limit}" velocity="49.0887" effort="7"/>
+            <limit lower="${joint7_lower_limit}" upper="${joint7_upper_limit}" velocity="49.0887" effort="5"/>
             <safety_controller k_position="8" k_velocity="1"
                                soft_lower_limit="${joint7_lower_limit+0.2}"
@@ -284,5 +284,5 @@
                 <origin xyz="0 0 10.21375" rpy="0 0 0"/>
                 <axis xyz="0 0 1"/>
-                <limit lower="${joint1_lower_limit}" upper="${joint1_upper_limit}" velocity="1.068" effort="180"/>
+                <limit lower="${joint1_lower_limit}" upper="${joint1_upper_limit}" velocity="1.068" effort="230"/>
             </joint>
             <joint name="mimic_joint2" type="prismatic">
@@ -291,5 +291,5 @@
                 <origin xyz="0. 0. 30.098707" rpy="0 0 0"/>
                 <axis xyz="1 0 0"/>
-                <limit lower="${joint2_lower_limit}" upper="${joint2_upper_limit}" velocity="1.9" effort="120"/>
+                <limit lower="${joint2_lower_limit}" upper="${joint2_upper_limit}" velocity="1.93" effort="129"/>
             </joint>
             <joint name="mimic_joint3" type="prismatic">
@@ -298,5 +298,5 @@
                 <origin xyz="0.022 0. 20.034" rpy="0 0 0"/>
                 <axis xyz="1 0 0"/>
-                <limit lower="${joint3_lower_limit}" upper="${joint3_upper_limit}" velocity="0.95" effort="210"/>
+                <limit lower="${joint3_lower_limit}" upper="${joint3_upper_limit}" velocity="0.965" effort="258"/>
             </joint>
         </xacro:unless>

Commit message: Add uwb's collision to base link

File: urdf/engineer/arm.urdf.xacro (robot description, xacro)
@@ -6,5 +6,5 @@
         <xacro:property name="joint2_upper_limit" value="0.3"/>
         <xacro:property name="joint2_lower_limit" value="-0.35"/>
-        <xacro:property name="joint3_upper_limit" value="0.31"/>
+        <xacro:property name="joint3_upper_limit" value="0.3"/>
         <xacro:property name="joint3_lower_limit" value="-0.12"/>
         <xacro:property name="joint4_upper_limit" value="0.31"/>
@@ -169,4 +169,7 @@
             <axis xyz="0 0 1"/>
             <limit lower="${joint1_lower_limit}" upper="${joint1_upper_limit}" velocity="1.068" effort="230"/>
+            <safety_controller k_position="80000." k_velocity="800."
+                               soft_lower_limit="${joint1_lower_limit+0.0005}"
+                               soft_upper_limit="${joint1_upper_limit-0.001}"/>
         </joint>
         <joint name="joint2" type="prismatic">
@@ -175,5 +178,8 @@
             <origin xyz="-0.014 0. 0.0542" rpy="0 0 0"/>
             <axis xyz="1 0 0"/>
-            <limit lower="${joint2_lower_limit}" upper="${joint2_upper_limit}" velocity="1.93" effort="129"/>
+            <limit lower="${joint2_lower_limit}" upper="${joint2_upper_limit}" velocity="1.93" effort="110"/>
+            <safety_controller k_position="50000." k_velocity="600."
+                               soft_lower_limit="${joint2_lower_limit+0.008}"
+                               soft_upper_limit="${joint2_upper_limit-0.008}"/>
         </joint>
         <joint name="joint3" type="prismatic">
@@ -183,4 +189,7 @@
             <axis xyz="1 0 0"/>
             <limit lower="${joint3_lower_limit}" upper="${joint3_upper_limit}" velocity="0.965" effort="258"/>
+            <safety_controller k_position="80000." k_velocity="1000."
+                               soft_lower_limit="${joint3_lower_limit+0.002}"
+                               soft_upper_limit="${joint3_upper_limit-0.004}"/>
         </joint>
         <joint name="joint4" type="prismatic">
@@ -190,4 +199,7 @@
             <axis xyz="0 1 0"/>
             <limit lower="${joint4_lower_limit}" upper="${joint4_upper_limit}" velocity="1.4625" effort="170"/>
+            <safety_controller k_position="8000." k_velocity="400."
+                               soft_lower_limit="${joint4_lower_limit+0.01}"
+                               soft_upper_limit="${joint4_upper_limit-0.01}"/>
         </joint>
         <joint name="joint5" type="revolute">
@@ -197,7 +209,7 @@
             <axis xyz="0 1 0"/>
             <limit lower="${joint5_lower_limit}" upper="${joint5_upper_limit}" velocity="18.53" effort="13.3"/>
-            <safety_controller k_position="12" k_velocity="5"
+            <safety_controller k_position="300." k_velocity="3."
                                soft_lower_limit="${joint5_lower_limit+0.03}"
-                               soft_upper_limit="${joint5_upper_limit-0.1}"/>
+                               soft_upper_limit="${joint5_upper_limit-0.03}"/>
         </joint>
         <joint name="joint6" type="revolute">
@@ -207,7 +219,7 @@
             <axis xyz="1 0 0"/>
             <limit lower="${joint6_lower_limit}" upper="${joint6_upper_limit}" velocity="18.53" effort="13.3"/>
-            <safety_controller k_position="12" k_velocity="5"
-                               soft_lower_limit="${joint6_lower_limit+0.1}"
-                               soft_upper_limit="${joint6_upper_limit-0.1}"/>
+            <safety_controller k_position="100." k_velocity="3."
+                               soft_lower_limit="${joint6_lower_limit+0.01}"
+                               soft_upper_limit="${joint6_upper_limit-0.01}"/>
         </joint>
         <joint name="joint7" type="revolute">
@@ -216,6 +228,6 @@
             <origin xyz="0.05825 0 0.233" rpy="0 0 0"/>
             <axis xyz="0 0 1"/>
-            <limit lower="${joint7_lower_limit}" upper="${joint7_upper_limit}" velocity="49.0887" effort="5"/>
-            <safety_controller k_position="8" k_velocity="1"
+            <limit lower="${joint7_lower_limit}" upper="${joint7_upper_limit}" velocity="50" effort="5"/>
+            <safety_controller k_position="50." k_velocity="0.6"
                                soft_lower_limit="${joint7_lower_limit+0.2}"
                                soft_upper_limit="${joint7_upper_limit-0.2}"/>
@@ -285,4 +297,7 @@
                 <axis xyz="0 0 1"/>
                 <limit lower="${joint1_lower_limit}" upper="${joint1_upper_limit}" velocity="1.068" effort="230"/>
+                <safety_controller k_position="80000." k_velocity="800."
+                                   soft_lower_limit="${joint1_lower_limit+0.0005}"
+                                   soft_upper_limit="${joint1_upper_limit-0.001}"/>
             </joint>
             <joint name="mimic_joint2" type="prismatic">
@@ -291,5 +306,8 @@
                 <origin xyz="0. 0. 30.098707" rpy="0 0 0"/>
                 <axis xyz="1 0 0"/>
-                <limit lower="${joint2_lower_limit}" upper="${joint2_upper_limit}" velocity="1.93" effort="129"/>
+                <limit lower="${joint2_lower_limit}" upper="${joint2_upper_limit}" velocity="1.93" effort="110"/>
+                <safety_controller k_position="50000." k_velocity="600."
+                                   soft_lower_limit="${joint2_lower_limit+0.008}"
+                                   soft_upper_limit="${joint2_upper_limit-0.008}"/>
             </joint>
             <joint name="mimic_joint3" type="prismatic">
@@ -299,4 +317,7 @@
                 <axis xyz="1 0 0"/>
                 <limit lower="${joint3_lower_limit}" upper="${joint3_upper_limit}" velocity="0.965" effort="258"/>
+                <safety_controller k_position="80000." k_velocity="1000."
+                                   soft_lower_limit="${joint3_lower_limit+0.002}"
+                                   soft_upper_limit="${joint3_upper_limit-0.004}"/>
             </joint>
         </xacro:unless>

File: urdf/engineer/chassis.urdf.xacro (robot description, xacro)
@@ -26,13 +26,13 @@
             </collision>
             <collision>
-                <origin xyz="0 0.251 0.447" rpy="0 0 0"/>
+                <origin xyz="0 0.251 0.387" rpy="0 0 0"/>
                 <geometry>
-                    <box size="0.28 0.035 0.567"/>
+                    <box size="0.43 0.0387 0.567"/>
                 </geometry>
             </collision>
             <collision>
-                <origin xyz="0 -0.251 0.447" rpy="0 0 0"/>
+                <origin xyz="0 -0.251 0.407" rpy="0 0 0"/>
                 <geometry>
-                    <box size="0.28 0.035 0.567"/>
+                    <box size="0.43 0.0387 0.567"/>
                 </geometry>
             </collision>
@@ -113,8 +113,8 @@
                             x_offset="${-wheel_track/2}" y_offset="${-wheel_base/2}"
                             z_offset="${wheel_offset_z}"/>
-        <xacro:swerve_transmission prefix="left_front" wheel_reduction="-13" pivot_offset="1.3086453"/>
-        <xacro:swerve_transmission prefix="right_front" wheel_reduction="-13" pivot_offset="6.238694172"/>
-        <xacro:swerve_transmission prefix="left_back" wheel_reduction="-13" pivot_offset="7.3548013"/>
-        <xacro:swerve_transmission prefix="right_back" wheel_reduction="-13" pivot_offset="2.3304011"/>
+        <xacro:swerve_transmission prefix="left_front" wheel_reduction="13" pivot_offset="-1.806482"/>
+        <xacro:swerve_transmission prefix="right_front" wheel_reduction="13" pivot_offset="0.7317981"/>
+        <xacro:swerve_transmission prefix="left_back" wheel_reduction="13" pivot_offset="-2.032005516"/>
+        <xacro:swerve_transmission prefix="right_back" wheel_reduction="13" pivot_offset="0.807739452"/>
     </xacro:macro>
 </robot>
