Commit message: Combined the joint and its mimic's effort and velocity

File: urdf/engineer/arm.urdf.xacro (robot description, xacro)
@@ -16,4 +16,10 @@
         <xacro:property name="joint7_upper_limit" value="4"/>
         <xacro:property name="joint7_lower_limit" value="-1"/>
+        <xacro:property name="joint1_velocity" value="1.068"/>
+        <xacro:property name="joint1_effort" value="230"/>
+        <xacro:property name="joint2_velocity" value="1.93"/>
+        <xacro:property name="joint2_effort" value="110"/>
+        <xacro:property name="joint3_velocity" value="0.965"/>
+        <xacro:property name="joint3_effort" value="258"/>
         <!--  link  -->
         <link name="link1">
@@ -168,5 +174,6 @@
             <origin xyz="0 0 0.233" rpy="0 0 0"/>
             <axis xyz="0 0 1"/>
-            <limit lower="${joint1_lower_limit}" upper="${joint1_upper_limit}" velocity="1.068" effort="230"/>
+            <limit lower="${joint1_lower_limit}" upper="${joint1_upper_limit}" velocity="${joint1_velocity}"
+                   effort="${joint1_effort}"/>
             <safety_controller k_position="40000." k_velocity="800."
                                soft_lower_limit="${joint1_lower_limit+0.0005}"
@@ -178,5 +185,6 @@
             <origin xyz="-0.014 0. 0.0542" rpy="0 0 0"/>
             <axis xyz="1 0 0"/>
-            <limit lower="${joint2_lower_limit}" upper="${joint2_upper_limit}" velocity="1.93" effort="110"/>
+            <limit lower="${joint2_lower_limit}" upper="${joint2_upper_limit}" velocity="${joint2_velocity}"
+                   effort="${joint2_effort}"/>
             <safety_controller k_position="50000." k_velocity="600."
                                soft_lower_limit="${joint2_lower_limit+0.008}"
@@ -188,5 +196,6 @@
             <origin xyz="-0.11 0. 0.013" rpy="0 0 0"/>
             <axis xyz="1 0 0"/>
-            <limit lower="${joint3_lower_limit}" upper="${joint3_upper_limit}" velocity="0.965" effort="258"/>
+            <limit lower="${joint3_lower_limit}" upper="${joint3_upper_limit}" velocity="${joint3_velocity}"
+                   effort="${joint3_effort}"/>
             <safety_controller k_position="80000." k_velocity="1000."
                                soft_lower_limit="${joint3_lower_limit+0.002}"
@@ -296,5 +305,6 @@
                 <origin xyz="0 0 10.21375" rpy="0 0 0"/>
                 <axis xyz="0 0 1"/>
-                <limit lower="${joint1_lower_limit}" upper="${joint1_upper_limit}" velocity="1.068" effort="230"/>
+                <limit lower="${joint1_lower_limit}" upper="${joint1_upper_limit}" velocity="${joint1_velocity}"
+                       effort="${joint1_effort}"/>
                 <safety_controller k_position="80000." k_velocity="800."
                                    soft_lower_limit="${joint1_lower_limit+0.0005}"
@@ -306,5 +316,6 @@
                 <origin xyz="0. 0. 30.098707" rpy="0 0 0"/>
                 <axis xyz="1 0 0"/>
-                <limit lower="${joint2_lower_limit}" upper="${joint2_upper_limit}" velocity="1.93" effort="110"/>
+                <limit lower="${joint2_lower_limit}" upper="${joint2_upper_limit}" velocity="${joint2_velocity}"
+                       effort="${joint2_effort}"/>
                 <safety_controller k_position="50000." k_velocity="600."
                                    soft_lower_limit="${joint2_lower_limit+0.008}"
@@ -316,5 +327,6 @@
                 <origin xyz="0.022 0. 20.034" rpy="0 0 0"/>
                 <axis xyz="1 0 0"/>
-                <limit lower="${joint3_lower_limit}" upper="${joint3_upper_limit}" velocity="0.965" effort="258"/>
+                <limit lower="${joint3_lower_limit}" upper="${joint3_upper_limit}" velocity="${joint3_velocity}"
+                       effort="${joint3_effort}"/>
                 <safety_controller k_position="80000." k_velocity="1000."
                                    soft_lower_limit="${joint3_lower_limit+0.002}"

Commit message: Update joint's limit and vel

File: urdf/engineer/arm.urdf.xacro (robot description, xacro)
@@ -2,9 +2,9 @@
 <robot xmlns:xacro="http://www.ros.org/wiki/xacro" name="arm">
     <xacro:macro name="arm" params="connected_to simulation">
-        <xacro:property name="joint1_upper_limit" value="0.25"/>
+        <xacro:property name="joint1_upper_limit" value="0.224"/>
         <xacro:property name="joint1_lower_limit" value="0"/>
-        <xacro:property name="joint2_upper_limit" value="0.3"/>
+        <xacro:property name="joint2_upper_limit" value="0.33"/>
         <xacro:property name="joint2_lower_limit" value="-0.35"/>
-        <xacro:property name="joint3_upper_limit" value="0.3"/>
+        <xacro:property name="joint3_upper_limit" value="0.31"/>
         <xacro:property name="joint3_lower_limit" value="-0.12"/>
         <xacro:property name="joint4_upper_limit" value="0.31"/>
@@ -176,7 +176,7 @@
             <limit lower="${joint1_lower_limit}" upper="${joint1_upper_limit}" velocity="${joint1_velocity}"
                    effort="${joint1_effort}"/>
-            <safety_controller k_position="40000." k_velocity="800."
-                               soft_lower_limit="${joint1_lower_limit+0.0005}"
-                               soft_upper_limit="${joint1_upper_limit-0.001}"/>
+            <safety_controller k_position="6000." k_velocity="200."
+                               soft_lower_limit="${joint1_lower_limit+0.0001}"
+                               soft_upper_limit="${joint1_upper_limit-0.0001}"/>
         </joint>
         <joint name="joint2" type="prismatic">
@@ -188,6 +188,6 @@
                    effort="${joint2_effort}"/>
             <safety_controller k_position="50000." k_velocity="600."
-                               soft_lower_limit="${joint2_lower_limit+0.008}"
-                               soft_upper_limit="${joint2_upper_limit-0.008}"/>
+                               soft_lower_limit="${joint2_lower_limit+0.003}"
+                               soft_upper_limit="${joint2_upper_limit-0.003}"/>
         </joint>
         <joint name="joint3" type="prismatic">
@@ -199,6 +199,6 @@
                    effort="${joint3_effort}"/>
             <safety_controller k_position="80000." k_velocity="1000."
-                               soft_lower_limit="${joint3_lower_limit+0.002}"
-                               soft_upper_limit="${joint3_upper_limit-0.004}"/>
+                               soft_lower_limit="${joint3_lower_limit+0.001}"
+                               soft_upper_limit="${joint3_upper_limit-0.001}"/>
         </joint>
         <joint name="joint4" type="prismatic">
@@ -209,6 +209,6 @@
             <limit lower="${joint4_lower_limit}" upper="${joint4_upper_limit}" velocity="1.4625" effort="170"/>
             <safety_controller k_position="8000." k_velocity="400."
-                               soft_lower_limit="${joint4_lower_limit+0.01}"
-                               soft_upper_limit="${joint4_upper_limit-0.01}"/>
+                               soft_lower_limit="${joint4_lower_limit+0.005}"
+                               soft_upper_limit="${joint4_upper_limit-0.005}"/>
         </joint>
         <joint name="joint5" type="revolute">
@@ -307,7 +307,7 @@
                 <limit lower="${joint1_lower_limit}" upper="${joint1_upper_limit}" velocity="${joint1_velocity}"
                        effort="${joint1_effort}"/>
-                <safety_controller k_position="80000." k_velocity="800."
-                                   soft_lower_limit="${joint1_lower_limit+0.0005}"
-                                   soft_upper_limit="${joint1_upper_limit-0.001}"/>
+                <safety_controller k_position="6000." k_velocity="200."
+                                   soft_lower_limit="${joint1_lower_limit+0.0001}"
+                                   soft_upper_limit="${joint1_upper_limit-0.0001}"/>
             </joint>
             <joint name="mimic_joint2" type="prismatic">
@@ -319,6 +319,6 @@
                        effort="${joint2_effort}"/>
                 <safety_controller k_position="50000." k_velocity="600."
-                                   soft_lower_limit="${joint2_lower_limit+0.008}"
-                                   soft_upper_limit="${joint2_upper_limit-0.008}"/>
+                                   soft_lower_limit="${joint2_lower_limit+0.003}"
+                                   soft_upper_limit="${joint2_upper_limit-0.003}"/>
             </joint>
             <joint name="mimic_joint3" type="prismatic">
@@ -330,6 +330,6 @@
                        effort="${joint3_effort}"/>
                 <safety_controller k_position="80000." k_velocity="1000."
-                                   soft_lower_limit="${joint3_lower_limit+0.002}"
-                                   soft_upper_limit="${joint3_upper_limit-0.004}"/>
+                                   soft_lower_limit="${joint3_lower_limit+0.001}"
+                                   soft_upper_limit="${joint3_upper_limit-0.001}"/>
             </joint>
         </xacro:unless>

File: urdf/engineer/gimbal.urdf.xacro (robot description, xacro)
@@ -64,5 +64,8 @@
                     rpy="0 0 0"/>
             <dynamics damping="0.0" friction="0.1"/>
-            <limit effort="1.2" velocity="30" lower="-4.3" upper="0.3"/>
+            <limit effort="0.25" velocity="1000" lower="-4.3" upper="0.3"/>
+            <safety_controller k_position="0.8" k_velocity="0.04"
+                               soft_lower_limit="-4.25"
+                               soft_upper_limit="0.25"/>
             <parent link="gimbal_base"/>
             <child link="yaw"/>
@@ -72,5 +75,5 @@
             <origin xyz="0.  0. 0.056 " rpy="0 0 0"/>
             <dynamics damping="0.0" friction="0.1"/>
-            <limit effort="1.2" velocity="30" lower="-0.8" upper="0.8"/>
+            <limit effort="1.2" velocity="30" lower="-1" upper="1"/>
             <parent link="yaw"/>
             <child link="pitch"/>

Commit message: Increase the collision of joint2's motor

File: urdf/engineer/arm.urdf.xacro (robot description, xacro)
@@ -2,5 +2,5 @@
 <robot xmlns:xacro="http://www.ros.org/wiki/xacro" name="arm">
     <xacro:macro name="arm" params="connected_to simulation">
-        <xacro:property name="joint1_upper_limit" value="0.224"/>
+        <xacro:property name="joint1_upper_limit" value="0.24"/>
         <xacro:property name="joint1_lower_limit" value="0"/>
         <xacro:property name="joint2_upper_limit" value="0.33"/>
@@ -14,6 +14,6 @@
         <xacro:property name="joint6_upper_limit" value="0.9"/>
         <xacro:property name="joint6_lower_limit" value="-0.9"/>
-        <xacro:property name="joint7_upper_limit" value="4"/>
-        <xacro:property name="joint7_lower_limit" value="-1"/>
+        <xacro:property name="joint7_upper_limit" value="4.5"/>
+        <xacro:property name="joint7_lower_limit" value="-1.3"/>
         <xacro:property name="joint1_velocity" value="1.068"/>
         <xacro:property name="joint1_effort" value="230"/>
@@ -61,4 +61,16 @@
                     <mesh filename="package://rm_description/meshes/engineer/link2_1_collision.stl"
                           scale="0.001 0.001 0.001"/>
+                </geometry>
+            </collision>
+            <collision>
+                <origin xyz="0.29 0.175 -0.025" rpy="0 0 0"/>
+                <geometry>
+                    <box size="0.08 0.12 0.1"/>
+                </geometry>
+            </collision>
+            <collision>
+                <origin xyz="0.29 -0.175 -0.025" rpy="0 0 0"/>
+                <geometry>
+                    <box size="0.08 0.12 0.1"/>
                 </geometry>
             </collision>

Commit message: Update joint's effort and vel's limit

File: urdf/engineer/arm.urdf.xacro (robot description, xacro)
@@ -16,10 +16,10 @@
         <xacro:property name="joint7_upper_limit" value="4.5"/>
         <xacro:property name="joint7_lower_limit" value="-1.3"/>
-        <xacro:property name="joint1_velocity" value="1.068"/>
-        <xacro:property name="joint1_effort" value="230"/>
-        <xacro:property name="joint2_velocity" value="1.93"/>
-        <xacro:property name="joint2_effort" value="110"/>
-        <xacro:property name="joint3_velocity" value="0.965"/>
-        <xacro:property name="joint3_effort" value="258"/>
+        <xacro:property name="joint1_velocity" value="1.2"/>
+        <xacro:property name="joint1_effort" value="609.75"/>
+        <xacro:property name="joint2_velocity" value="1.9"/>
+        <xacro:property name="joint2_effort" value="110.00"/>
+        <xacro:property name="joint3_velocity" value="0.964"/>
+        <xacro:property name="joint3_effort" value="258.00"/>
         <!--  link  -->
         <link name="link1">
@@ -219,5 +219,5 @@
             <origin xyz="0. 0. 0.078" rpy="0 0 0"/>
             <axis xyz="0 1 0"/>
-            <limit lower="${joint4_lower_limit}" upper="${joint4_upper_limit}" velocity="1.4625" effort="170"/>
+            <limit lower="${joint4_lower_limit}" upper="${joint4_upper_limit}" velocity="2.92" effort="85.47"/>
             <safety_controller k_position="8000." k_velocity="400."
                                soft_lower_limit="${joint4_lower_limit+0.005}"
@@ -229,5 +229,5 @@
             <origin xyz="0. 0. 0.02" rpy="0 0 0"/>
             <axis xyz="0 1 0"/>
-            <limit lower="${joint5_lower_limit}" upper="${joint5_upper_limit}" velocity="18.53" effort="13.3"/>
+            <limit lower="${joint5_lower_limit}" upper="${joint5_upper_limit}" velocity="18.8" effort="13.3"/>
             <safety_controller k_position="300." k_velocity="3."
                                soft_lower_limit="${joint5_lower_limit+0.05}"
@@ -239,5 +239,5 @@
             <origin xyz="-0.0585 0. 0.04875" rpy="0 0 0"/>
             <axis xyz="1 0 0"/>
-            <limit lower="${joint6_lower_limit}" upper="${joint6_upper_limit}" velocity="18.53" effort="13.3"/>
+            <limit lower="${joint6_lower_limit}" upper="${joint6_upper_limit}" velocity="18.8" effort="13.3"/>
             <safety_controller k_position="100." k_velocity="3."
                                soft_lower_limit="${joint6_lower_limit+0.01}"

Commit message: Fixed the wrong stl of link4

File: urdf/engineer/arm.urdf.xacro (robot description, xacro)
@@ -42,4 +42,5 @@
                 </geometry>
             </collision>
+            <selfCollide>true</selfCollide>
         </link>
         <link name="link2_1">
@@ -75,4 +76,5 @@
                 </geometry>
             </collision>
+            <selfCollide>true</selfCollide>
         </link>
         <link name="link2_2">
@@ -96,4 +98,5 @@
                 </geometry>
             </collision>
+            <selfCollide>true</selfCollide>
         </link>
         <link name="link3">
@@ -117,4 +120,5 @@
                 </geometry>
             </collision>
+            <selfCollide>true</selfCollide>
         </link>
         <link name="link4">
@@ -132,10 +136,16 @@
             </visual>
             <collision>
-                <origin xyz="0 0 0" rpy="0 0 0"/>
-                <geometry>
-                    <mesh filename="package://rm_description/meshes/engineer/link4_collision.stl"
-                          scale="0.001 0.001 0.001"/>
-                </geometry>
-            </collision>
+                <origin xyz="-0.0145 0 0" rpy="0 0 0"/>
+                <geometry>
+                    <box size="0.0825 0.1015 0.078"/>
+                </geometry>
+            </collision>
+            <collision>
+                <origin xyz="0. 0.0878 0" rpy="0 0 0"/>
+                <geometry>
+                    <box size="0.0495 0.071 0.0495"/>
+                </geometry>
+            </collision>
+            <selfCollide>true</selfCollide>
         </link>
         <link name="link5">
@@ -159,4 +169,5 @@
                 </geometry>
             </collision>
+            <selfCollide>true</selfCollide>
         </link>
         <link name="link6">
@@ -180,4 +191,5 @@
                 </geometry>
             </collision>
+            <selfCollide>true</selfCollide>
         </link>
         <joint name="joint1" type="prismatic">
@@ -191,4 +203,5 @@
                                soft_lower_limit="${joint1_lower_limit+0.0001}"
                                soft_upper_limit="${joint1_upper_limit-0.0001}"/>
+            <dynamics damping="0.0" friction="0.1"/>
         </joint>
         <joint name="joint2" type="prismatic">
@@ -202,4 +215,5 @@
                                soft_lower_limit="${joint2_lower_limit+0.003}"
                                soft_upper_limit="${joint2_upper_limit-0.003}"/>
+            <dynamics damping="0.0" friction="0.1"/>
         </joint>
         <joint name="joint3" type="prismatic">
@@ -213,4 +227,5 @@
                                soft_lower_limit="${joint3_lower_limit+0.001}"
                                soft_upper_limit="${joint3_upper_limit-0.001}"/>
+            <dynamics damping="0.0" friction="0.1"/>
         </joint>
         <joint name="joint4" type="prismatic">
@@ -223,9 +238,10 @@
                                soft_lower_limit="${joint4_lower_limit+0.005}"
                                soft_upper_limit="${joint4_upper_limit-0.005}"/>
+            <dynamics damping="0.0" friction="0.1"/>
         </joint>
         <joint name="joint5" type="revolute">
             <parent link="link3"/>
             <child link="link4"/>
-            <origin xyz="0. 0. 0.02" rpy="0 0 0"/>
+            <origin xyz="0. 0. 0.06" rpy="0 0 0"/>
             <axis xyz="0 1 0"/>
             <limit lower="${joint5_lower_limit}" upper="${joint5_upper_limit}" velocity="18.8" effort="13.3"/>
@@ -233,9 +249,10 @@
                                soft_lower_limit="${joint5_lower_limit+0.05}"
                                soft_upper_limit="${joint5_upper_limit-0.05}"/>
+            <dynamics damping="0.0" friction="0.1"/>
         </joint>
         <joint name="joint6" type="revolute">
             <parent link="link4"/>
             <child link="link5"/>
-            <origin xyz="-0.0585 0. 0.04875" rpy="0 0 0"/>
+            <origin xyz="-0.06 0. 0." rpy="0 0 0"/>
             <axis xyz="1 0 0"/>
             <limit lower="${joint6_lower_limit}" upper="${joint6_upper_limit}" velocity="18.8" effort="13.3"/>
@@ -243,9 +260,10 @@
                                soft_lower_limit="${joint6_lower_limit+0.01}"
                                soft_upper_limit="${joint6_upper_limit-0.01}"/>
+            <dynamics damping="0.0" friction="0.1"/>
         </joint>
         <joint name="joint7" type="revolute">
             <parent link="link5"/>
             <child link="link6"/>
-            <origin xyz="0.05825 0 0.233" rpy="0 0 0"/>
+            <origin xyz="0.06 0 0.253" rpy="0 0 0"/>
             <axis xyz="0 0 1"/>
             <limit lower="${joint7_lower_limit}" upper="${joint7_upper_limit}" velocity="50" effort="5"/>
@@ -253,4 +271,5 @@
                                soft_lower_limit="${joint7_lower_limit+0.2}"
                                soft_upper_limit="${joint7_upper_limit-0.2}"/>
+            <dynamics damping="0.0" friction="0.1"/>
         </joint>
         <xacro:unless value="${simulation}">

File: urdf/engineer/chassis.urdf.xacro (robot description, xacro)
@@ -37,4 +37,5 @@
                 </geometry>
             </collision>
+            <selfCollide>true</selfCollide>
         </link>
         <link name="card">

Commit message: Update arm and chassis's collision

File: urdf/engineer/arm.urdf.xacro (robot description, xacro)
@@ -193,4 +193,5 @@
             <selfCollide>true</selfCollide>
         </link>
+        <link name="tools_link"/>
         <joint name="joint1" type="prismatic">
             <parent link="${connected_to}"/>
@@ -272,4 +273,9 @@
                                soft_upper_limit="${joint7_upper_limit-0.2}"/>
             <dynamics damping="0.0" friction="0.1"/>
+        </joint>
+        <joint name="tools_joint" type="fixed">
+            <parent link="link6"/>
+            <child link="tools_link"/>
+            <origin xyz="0.154 0 0.137" rpy="0 0 0"/>
         </joint>
         <xacro:unless value="${simulation}">

File: urdf/engineer/chassis.urdf.xacro (robot description, xacro)
@@ -23,4 +23,28 @@
                     <mesh filename="package://rm_description/meshes/engineer/base_collision.stl"
                           scale="0.001 0.001 0.001"/>
+                </geometry>
+            </collision>
+            <collision>
+                <origin xyz="0.175 -0.247 0.275" rpy="0 0 0"/>
+                <geometry>
+                    <box size="0.061 0.042 0.4"/>
+                </geometry>
+            </collision>
+            <collision>
+                <origin xyz="0.175 0.247 0.275" rpy="0 0 0"/>
+                <geometry>
+                    <box size="0.061 0.042 0.4"/>
+                </geometry>
+            </collision>
+            <collision>
+                <origin xyz="-0.175 -0.247 0.275" rpy="0 0 0"/>
+                <geometry>
+                    <box size="0.061 0.042 0.4"/>
+                </geometry>
+            </collision>
+            <collision>
+                <origin xyz="0.175 -0.247 0.275" rpy="0 0 0"/>
+                <geometry>
+                    <box size="0.061 0.042 0.4"/>
                 </geometry>
             </collision>

Commit message: Update tools_link position

File: urdf/engineer/arm.urdf.xacro (robot description, xacro)
@@ -277,5 +277,5 @@
             <parent link="link6"/>
             <child link="tools_link"/>
-            <origin xyz="0.154 0 0.137" rpy="0 0 0"/>
+            <origin xyz="0.112 0 0.154" rpy="0 0 0"/>
         </joint>
         <xacro:unless value="${simulation}">
