Commit message: Modified the collision

File: urdf/engineer/arm.urdf.xacro (robot description, xacro)
@@ -98,5 +98,10 @@
                 </geometry>
             </collision>
-            <selfCollide>true</selfCollide>
+            <collision>
+                <origin xyz="-0.056 0.24 0.03" rpy="0 0 0"/>
+                <geometry>
+                    <box size="0.063 0.05 0.043"/>
+                </geometry>
+            </collision>
         </link>
         <link name="link3">
@@ -118,4 +123,10 @@
                     <mesh filename="package://rm_description/meshes/engineer/link3_collision.stl"
                           scale="0.001 0.001 0.001"/>
+                </geometry>
+            </collision>
+            <collision>
+                <origin xyz="-0.06 0. -0.03" rpy="0 0 0"/>
+                <geometry>
+                    <box size="0.063 0.4 0.083"/>
                 </geometry>
             </collision>

File: urdf/engineer/chassis.urdf.xacro (robot description, xacro)
@@ -34,5 +34,5 @@
                 <origin xyz="0.175 0.247 0.275" rpy="0 0 0"/>
                 <geometry>
-                    <box size="0.081 0.042 0.4"/>
+                    <box size="0.091 0.05 0.45"/>
                 </geometry>
             </collision>
@@ -40,5 +40,5 @@
                 <origin xyz="-0.175 -0.247 0.275" rpy="0 0 0"/>
                 <geometry>
-                    <box size="0.081 0.042 0.4"/>
+                    <box size="0.091 0.05 0.45"/>
                 </geometry>
             </collision>
@@ -46,5 +46,5 @@
                 <origin xyz="0.175 -0.247 0.275" rpy="0 0 0"/>
                 <geometry>
-                    <box size="0.081 0.042 0.4"/>
+                    <box size="0.091 0.05 0.45"/>
                 </geometry>
             </collision>
@@ -52,5 +52,5 @@
                 <origin xyz="-0.175 0.247 0.275" rpy="0 0 0"/>
                 <geometry>
-                    <box size="0.081 0.042 0.4"/>
+                    <box size="0.091 0.05 0.45"/>
                 </geometry>
             </collision>
