Commit message: Add gimbal's urdf

File: urdf/engineer/gimbal.urdf.xacro (robot description, xacro)
@@ -17,4 +17,11 @@
                 </geometry>
             </visual>
+            <collision>
+                <origin xyz="0 0 0" rpy="0 0 0"/>
+                <geometry>
+                    <mesh filename="package://rm_description/meshes/engineer/gimbal_collision.stl"
+                          scale="0.001 0.001 0.001"/>
+                </geometry>
+            </collision>
         </link>
         <link name="yaw">
@@ -57,6 +64,5 @@
                     rpy="0 0 0"/>
             <dynamics damping="0.0" friction="0.1"/>
-            <limit effort="0.2" velocity="10" lower="-0.6197" upper="3.4545"/>
-            <!--            <safety_controller k_position="2" k_velocity="0.02" soft_lower_limit="-0.519" soft_upper_limit="3.35"/>-->
+            <limit effort="1.2" velocity="30" lower="-4.3" upper="0.3"/>
             <parent link="gimbal_base"/>
             <child link="yaw"/>
@@ -66,5 +72,5 @@
             <origin xyz="0.  0. 0.056 " rpy="0 0 0"/>
             <dynamics damping="0.0" friction="0.1"/>
-            <limit effort="0.2" velocity="10" lower="-0.47247" upper="1.25862"/>
+            <limit effort="1.2" velocity="30" lower="-0.8" upper="0.8"/>
             <parent link="yaw"/>
             <child link="pitch"/>
@@ -77,5 +83,5 @@
             </actuator>
             <joint name="yaw_joint">
-                <offset>3.48597</offset>
+                <offset>0.03911</offset>
                 <hardwareInterface>hardware_interface/EffortJointInterface</hardwareInterface>
             </joint>
@@ -87,5 +93,5 @@
             </actuator>
             <joint name="pitch_joint">
-                <offset>0.75088</offset>
+                <offset>0.777728</offset>
                 <hardwareInterface>hardware_interface/EffortJointInterface</hardwareInterface>
             </joint>

Commit message: Modified yaw joint's limit

File: urdf/engineer/gimbal.urdf.xacro (robot description, xacro)
@@ -64,5 +64,5 @@
                     rpy="0 0 0"/>
             <dynamics damping="0.0" friction="0.1"/>
-            <limit effort="0.25" velocity="1000" lower="-4.26" upper="0.45"/>
+            <limit effort="0.25" velocity="1000" lower="-5" upper="0"/>
             <parent link="gimbal_base"/>
             <child link="yaw"/>

Commit message: Fix gimbal's motor vel and effort

File: urdf/engineer/gimbal.urdf.xacro (robot description, xacro)
@@ -69,5 +69,5 @@
                     rpy="0 0 0"/>
             <dynamics damping="0.0" friction="0.1"/>
-            <limit effort="1.2" velocity="13.82" lower="${yaw_lower_limit}" upper="${yaw_upper_limit}"/>
+            <limit effort="900" velocity="0.17" lower="${yaw_lower_limit}" upper="${yaw_upper_limit}"/>
             <safety_controller k_position="100" k_velocity="0.1"
                                soft_lower_limit="${yaw_lower_limit+threshold}"
@@ -80,5 +80,5 @@
             <origin xyz="0.  0. 0.056 " rpy="0 0 0"/>
             <dynamics damping="0.0" friction="0.1"/>
-            <limit effort="1.2" velocity="13.82" lower="${pitch_lower_limit}" upper="${pitch_upper_limit}"/>
+            <limit effort="900" velocity="0.17" lower="${pitch_lower_limit}" upper="${pitch_upper_limit}"/>
             <safety_controller k_position="100" k_velocity="0.1"
                                soft_lower_limit="${pitch_lower_limit+threshold}"

Commit message: Modified the gimbal's limit

File: urdf/engineer/gimbal.urdf.xacro (robot description, xacro)
@@ -3,9 +3,9 @@
     <!-- safety_distance: Minimum safety distance in [m] by which the collision volumes are expanded and which is enforced during robot motions -->
     <xacro:macro name="gimbal" params="connected_to:='' xyz:='0 0 0' rpy:='0 0 0' simulation">
-        <xacro:property name="threshold" value="0.04"/>
-        <xacro:property name="yaw_lower_limit" value="-4.18"/>
-        <xacro:property name="yaw_upper_limit" value="0.88"/>
-        <xacro:property name="pitch_lower_limit" value="-0.91"/>
-        <xacro:property name="pitch_upper_limit" value="0.91"/>
+        <xacro:property name="threshold" value="0.05"/>
+        <xacro:property name="yaw_lower_limit" value="-4.3"/>
+        <xacro:property name="yaw_upper_limit" value="0.77"/>
+        <xacro:property name="pitch_lower_limit" value="-0.96"/>
+        <xacro:property name="pitch_upper_limit" value="0.87"/>
         <link name="gimbal_base">
             <inertial>
@@ -69,5 +69,5 @@
                     rpy="0 0 0"/>
             <dynamics damping="0.0" friction="0.1"/>
-            <limit effort="900" velocity="0.17" lower="${yaw_lower_limit}" upper="${yaw_upper_limit}"/>
+            <limit effort="0.15" velocity="900" lower="${yaw_lower_limit}" upper="${yaw_upper_limit}"/>
             <parent link="gimbal_base"/>
             <child link="yaw"/>
@@ -77,5 +77,5 @@
             <origin xyz="0.  0. 0.056 " rpy="0 0 0"/>
             <dynamics damping="0.0" friction="0.1"/>
-            <limit effort="900" velocity="0.17" lower="${pitch_lower_limit}" upper="${pitch_upper_limit}"/>
+            <limit effort="0.15" velocity="900" lower="${pitch_lower_limit}" upper="${pitch_upper_limit}"/>
             <parent link="yaw"/>
             <child link="pitch"/>
@@ -88,5 +88,5 @@
             </actuator>
             <joint name="yaw_joint">
-                <offset>0.7524</offset>
+                <offset>0.7639</offset>
                 <hardwareInterface>hardware_interface/EffortJointInterface</hardwareInterface>
             </joint>
@@ -98,5 +98,5 @@
             </actuator>
             <joint name="pitch_joint">
-                <offset>0.9019</offset>
+                <offset>0.83141</offset>
                 <hardwareInterface>hardware_interface/EffortJointInterface</hardwareInterface>
             </joint>
