Commit message: Updated new verision sentry's urdf.

File: urdf/sentry/upper_gimbal.urdf.xacro (robot description, xacro)
@@ -14,8 +14,8 @@
         </visual>
         <inertial>
-            <mass value="934.339e-3"/>
-            <origin xyz="-0.08e-3 -61.185e-3 90.777e-3" rpy="0 0 0"/>
-            <inertia ixx="1.880e-2" ixy="-6662.219e-9" ixz="7064.827e-9" iyy="1.083e-2"
-                     iyz="7.150e-3" izz="9.057e-3"/>
+            <mass value="599.396e-3"/>
+            <origin xyz="-67.151e-3 7.823e-3 37.636e-3" rpy="0 0 0"/>
+            <inertia ixx="3.787e-4" ixy="46745.03e-9" ixz="5459.222e-9" iyy="8.443e-4"
+                     iyz="1835.055e-9" izz="6.561e-4"/>
         </inertial>
         <collision>
@@ -31,5 +31,5 @@
         <child link="upper_yaw"/>
         <axis xyz="0 0 1"/>
-        <origin xyz="0 0 83.4e-3"/>
+        <origin xyz="0 -24.464e-3 228.5e-3"/>
         <dynamics damping="0" friction="0.1"/>
         <limit effort="1.2" velocity="13.82" lower="${yaw_lower_limit}" upper="${yaw_upper_limit}"/>
@@ -39,59 +39,59 @@
     </joint>
     <link name="upper_pitch">
-        <inertial>
-            <mass value="1227.797e-3"/>
-            <origin xyz="15.667e-3 -0.268e-3 27.267e-3"/>
-            <inertia ixx="4.484e-3" ixy="813.964e-9" ixz="2.786e-4" iyy="6.599e-3"
-                     iyz="-6822.846e-9" izz="5.343E-3"/>
-        </inertial>
-        <visual>
-            <origin xyz="0 0 0" rpy="0 0 0"/>
-            <geometry>
-                <mesh filename="package://rm_description/meshes/sentry/upper_pitch.stl" scale="0.001 0.001 0.001"/>
-            </geometry>
-        </visual>
-        <collision>
-            <origin xyz="0 0 0" rpy="0 0 0"/>
-            <geometry>
-                <mesh filename="package://rm_description/meshes/sentry/upper_pitch.stl" scale="0.001 0.001 0.001"/>
-            </geometry>
-        </collision>
+      <inertial>
+        <mass value="584.157e-3"/>
+        <origin xyz="31.362e-3 0.689e-3 36.945e-3"/>
+        <inertia ixx="1.030e-3" ixy="18463.46e-9" ixz="9.122e-4" iyy="4.507e-3"
+                 iyz="8105.967e-9" izz="4.096e-3"/>
+      </inertial>
+      <visual>
+        <origin xyz="0 0 0" rpy="0 0 0"/>
+        <geometry>
+          <mesh filename="package://rm_description/meshes/sentry/upper_pitch.stl" scale="0.001 0.001 0.001"/>
+        </geometry>
+      </visual>
+      <collision>
+        <origin xyz="0 0 0" rpy="0 0 0"/>
+        <geometry>
+          <mesh filename="package://rm_description/meshes/sentry/upper_pitch.stl" scale="0.001 0.001 0.001"/>
+        </geometry>
+      </collision>
     </link>
     <joint name="upper_pitch_joint" type="revolute">
-        <parent link="upper_yaw"/>
-        <child link="upper_pitch"/>
-        <axis xyz="0 1 0"/>
-        <origin xyz="0 0 0.125"/>
-        <dynamics damping="0" friction="0.1"/>
-        <limit effort="1.2" velocity="13.82" lower="${pitch_lower_limit}" upper="${pitch_upper_limit}"/>
-        <safety_controller k_position="100" k_velocity="0.1"
-                           soft_lower_limit="${pitch_lower_limit+threshold}"
-                           soft_upper_limit="${pitch_upper_limit-threshold}"/>
+      <parent link="upper_yaw"/>
+      <child link="upper_pitch"/>
+      <axis xyz="0 1 0"/>
+      <origin xyz="0 0 87.993e-3"/>
+      <dynamics damping="0" friction="0.1"/>
+      <limit effort="1.2" velocity="13.82" lower="${pitch_lower_limit}" upper="${pitch_upper_limit}"/>
+      <safety_controller k_position="100" k_velocity="0.1"
+                         soft_lower_limit="${pitch_lower_limit+threshold}"
+                         soft_upper_limit="${pitch_upper_limit-threshold}"/>
     </joint>
-    <!--  <link name="upper_camera">-->
-    <!--    <inertial>-->
-    <!--          <mass value="0.17671"/>-->
-    <!--          <origin xyz="0.022 0.0 0.0"/>-->
-    <!--          <inertia ixx="2.129e-5" ixy="7.329e-8" ixz="-1.11e-7" iyy="2.198e-4" iyz="-8.04e-7" izz="2.197e-4"/>-->
-    <!--        </inertial>-->
-    <!--        <visual>-->
-    <!--          <origin xyz=" 0 0 0 " rpy="0 -1.57 0"/>-->
-    <!--          <geometry>-->
-    <!--            <mesh filename="package://rm_description/meshes/common/camera.stl" scale="0.001 0.001 0.001"/>-->
-    <!--          </geometry>-->
-    <!--          <material name="Black"/>-->
-    <!--        </visual>-->
-    <!--        <collision>-->
-    <!--          <origin xyz="0 0 0" rpy="0 -1.57 0"/>-->
-    <!--          <geometry>-->
-    <!--            <mesh filename="package://rm_description/meshes/common/camera.stl" scale="0.001 0.001 0.001"/>-->
-    <!--          </geometry>-->
-    <!--        </collision>-->
-    <!--      </link>-->
-    <!--      <joint name="camera_joint" type="fixed">-->
-    <!--        <parent link="pitch"/>-->
-    <!--        <child link="camera"/>-->
-    <!--        <origin xyz="0.086  0.0 -0.040" rpy="-1.57 0 -1.57"/>-->
-    <!--        <axis xyz="0 0 1"/>-->
-    <!--      </joint>-->
+    <link name="upper_camera">
+      <inertial>
+        <mass value="0.111"/>
+        <origin xyz="24.786e-3 0.019e-3 14.471e-3"/>
+        <inertia ixx="15645.374e-9" ixy="94.19e-9" ixz="-143.444e-9" iyy="80877.924e-9"
+                 iyz="-45.908e-9" izz="80823.702e-9"/>
+      </inertial>
+      <visual>
+        <origin xyz=" 0 0 0 " rpy="0 0 0"/>
+        <geometry>
+          <mesh filename="package://rm_description/meshes/sentry/upper_camera.stl" scale="0.001 0.001 0.001"/>
+        </geometry>
+      </visual>
+      <collision>
+        <origin xyz="0 0 0" rpy="0 0 0"/>
+        <geometry>
+          <mesh filename="package://rm_description/meshes/sentry/upper_camera.stl" scale="0.001 0.001 0.001"/>
+        </geometry>
+      </collision>
+    </link>
+    <joint name="upper_camera_joint" type="fixed">
+       <parent link="upper_pitch"/>
+       <child link="upper_camera"/>
+       <origin xyz="29.642e-3 0 54.20e-3" rpy="0 0 0"/>
+       <axis xyz="0 0 1"/>
+    </joint>
 </robot>

File: urdf/sentry/upper_shooter.urdf.xacro (robot description, xacro)
@@ -1,19 +1,61 @@
 <robot xmlns:xacro="http://www.ros.org/wiki/xacro">
-    <xacro:include filename="$(find rm_description)/urdf/common/friction.urdf.xacro"/>
-    <xacro:property name="wheel_offset_x" value="0.009"/>
-    <xacro:property name="wheel_offset_y" value="0.0365"/>
-    <xacro:property name="wheel_offset_z" value="0.00576"/>
-    <xacro:friction_wheel prefixs="upper_left" connected_to="upper_pitch"
-                          wheel_x_offset="${wheel_offset_x}" wheel_y_offset="${-wheel_offset_y}"
-                          wheel_z_offset="${wheel_offset_z}"/>
-    <xacro:friction_wheel prefixs="upper_right" connected_to="upper_pitch"
-                          wheel_x_offset="${wheel_offset_x}" wheel_y_offset="${wheel_offset_y}"
-                          wheel_z_offset="${wheel_offset_z}"/>
+    <link name="upper_left_friction">
+        <inertial>
+             <mass value="0.15269"/>
+             <origin xyz="0 0 -0.004"/>
+             <inertia ixx="4.776e-5" ixy="2.192e-7" ixz="-1.28e-7" iyy="4.759e-5"
+                      iyz="-1.683e-7" izz="6.148e-5"/>
+        </inertial>
+        <visual>
+            <origin xyz="0 0 0" rpy="0 0 0"/>
+            <geometry>
+                <mesh filename="package://rm_description/meshes/sentry/upper_friction.stl" scale="0.001 0.001 0.001"/>
+            </geometry>
+        </visual>
+        <collision>
+            <origin xyz="0 0 0" rpy="0 0 0"/>
+            <geometry>
+                <mesh filename="package://rm_description/meshes/sentry/upper_friction.stl" scale="0.001 0.001 0.001"/>
+            </geometry>
+        </collision>
+    </link>
+    <joint name="upper_left_friction_wheel_joint" type="continuous">
+        <origin xyz="47e-3 36.50e-3 -0.4e-3" rpy="0 0 0"/>
+        <parent link="upper_pitch"/>
+        <child link="upper_left_friction"/>
+        <axis xyz="0 0 1 "/>
+    </joint>
+    <link name="upper_right_friction">
+        <inertial>
+             <mass value="0.15269"/>
+             <origin xyz="0 0 -0.004"/>
+             <inertia ixx="4.776e-5" ixy="2.192e-7" ixz="-1.28e-7" iyy="4.759e-5"
+                      iyz="-1.683e-7" izz="6.148e-5"/>
+        </inertial>
+        <visual>
+            <origin xyz="0 0 0" rpy="0 0 0"/>
+            <geometry>
+                <mesh filename="package://rm_description/meshes/sentry/upper_friction_wheel.stl" scale="0.001 0.001 0.001"/>
+            </geometry>
+        </visual>
+        <collision>
+            <origin xyz="0 0 0" rpy="0 0 0"/>
+            <geometry>
+                <mesh filename="package://rm_description/meshes/sentry/upper_friction_wheel.stl" scale="0.001 0.001 0.001"/>
+            </geometry>
+        </collision>
+    </link>
+    <joint name="upper_right_friction_wheel_joint" type="continuous">
+        <origin xyz="47e-3 -36.50e-3 -0.4e-3" rpy="0 0 0"/>
+        <parent link="upper_pitch"/>
+        <child link="upper_right_friction"/>
+        <axis xyz="0 0 1 "/>
+    </joint>
     <link name="upper_trigger">
         <inertial>
-            <mass value="0.328"/>
-            <origin xyz="1.854e-3 -4.952e-3 20.252e-3"/>
-            <inertia ixx="5.284e-4" ixy="26474.311e-9" ixz="-5533.967e-9" iyy="3.633e-4"
-                     iyz="3258.006e-9" izz="4.750e-4"/>
+            <mass value="344.827e-3"/>
+            <origin xyz="-26.584e-3 0.526e-3 14.311e-3"/>
+            <inertia ixx="2.365e-4" ixy="-100.189e-9" ixz="1.146e-4" iyy="6.707e-4"
+                     iyz="81.455e-9" izz="6.916e-4"/>
         </inertial>
         <visual>
@@ -31,8 +73,7 @@
     </link>
     <joint name="upper_trigger_joint" type="continuous">
-        <origin xyz="-64.86e-3 0 -19e-3" rpy="0 0 0"/>
+        <origin xyz="-0.142e-3 -23.51e-3 85.467e-3" rpy="0 0 0"/>
         <dynamics damping="0.0" friction="0.01"/>
-        <limit effort="1.0" velocity="43.54" lower="-1e16" upper="1e16"/>
-        <parent link="upper_pitch"/>
+        <parent link="base_link"/>
         <child link="upper_trigger"/>
         <axis xyz="0 0 1 "/>
