Commit message: Updated new verision sentry's urdf.

File: urdf/sentry/chassis.urdf.xacro (robot description, xacro)
@@ -7,6 +7,6 @@
                 <mass value="6392.711e-3"/>
                 <origin xyz="17.924e-3 -11.095e-3 51.909e-3"/>
-                <inertia ixx="1.795e-1" ixy="4.102e-3" ixz="-8.862e-3" iyy="1.461e-1"
-                         iyz="1.34e-2" izz="1.896e-1"/>
+                <inertia ixx="1.795e-1" ixy="-4.102e-3" ixz="-8.862e-3" iyy="1.461e-1"
+                         iyz="1.340e-2" izz="1.896e-1"/>
             </inertial>
             <visual>
@@ -19,5 +19,5 @@
                 <origin xyz="0 0 0" rpy="0 0 0"/>
                 <geometry>
-                    <mesh filename="package://rm_description/meshes/sentry/base_link.stl" scale="0.001 0.001 0.001"/>
+                    <mesh filename="package://rm_description/meshes/sentry/base_link_collision.stl" scale="0.001 0.001 0.001"/>
                 </geometry>
             </collision>
@@ -37,7 +37,7 @@
             </visual>
             <collision>
-                <origin xyz="0 -0.004 0" rpy="0 0 0"/>
+                <origin xyz="0 0 0" rpy="0 0 0"/>
                 <geometry>
-                    <box size="0.127 0.02435 0.127"/>
+                    <mesh filename="package://rm_description/meshes/sentry/drive_wheel.stl" scale="0.001 0.001 0.001"/>
                 </geometry>
             </collision>
@@ -49,31 +49,4 @@
             <child link="drive_wheel_link"/>
             <origin xyz="0 51.65e-3 94.5e-3" rpy="0 0 0"/>
-        </joint>
-        <link name="slider_link">
-            <inertial>
-                <mass value="66.212e-3"/>
-                <origin xyz="-3.002e-3 -13.823e-3 14.751e-3"/>
-                <inertia ixx="20612.923e-9" ixy="-2537.219e-9" ixz="-2423.351e-9" iyy="78493.793e-9"
-                         iyz="-347.633e-9" izz="86435.358e-9"/>
-            </inertial>
-            <visual>
-                <origin xyz="0 0 0" rpy="0 0 0"/>
-                <geometry>
-                    <mesh filename="package://rm_description/meshes/sentry/slider.stl" scale="0.001 0.001 0.001"/>
-                </geometry>
-            </visual>
-            <collision>
-                <origin xyz="-0.01 -0.001 0.01" rpy="0 0 0"/>
-                <geometry>
-                    <box size="0.14 0.064 0.0353"/>
-                </geometry>
-            </collision>
-        </link>
-        <joint name="slider_joint" type="prismatic">
-            <axis xyz="1 0 0"/>
-            <limit effort="1.2" velocity="34" lower="-1e9" upper="1e9"/>
-            <parent link="base_link"/>
-            <child link="slider_link"/>
-            <origin xyz="12e-3 -87e-3 43.70e-3" rpy="0 0 0"/>
         </joint>
         <link name="catapult_link">
@@ -100,7 +73,7 @@
             <axis xyz="0 1 0"/>
             <limit effort="1.2" velocity="34" lower="-1e9" upper="1e9"/>
-            <parent link="slider_link"/>
+            <parent link="base_link"/>
             <child link="catapult_link"/>
-            <origin xyz="0 0 0" rpy="0 0 0"/>
+            <origin xyz="12e-3 -87e-3 43.70e-3" rpy="0 0 0"/>
         </joint>
         <xacro:if value="$(arg use_simulation)">

File: urdf/sentry/driven_wheel1.urdf.xacro (robot description, xacro)
@@ -12,14 +12,14 @@
             </visual>
             <inertial>
-                <mass value="2.388e-3"/>
+                <mass value="0.712e-3"/>
                 <origin xyz="0 0 0" rpy="0 0 0"/>
-                <inertia ixx="15.764e-9" ixy="0" ixz="0" iyy="19.664e-9"
-                         iyz="1.425e-18" izz="15.764e-9"/>
+                <inertia ixx="11.315e-9" ixy="0" ixz="0" iyy="19.664e-9"
+                         iyz="0" izz="11.315e-9"/>
             </inertial>
             <collision>
-                <origin xyz="0 0.00015 0" rpy="0 0 0"/>
                 <xacro:insert_block name="pose"/>
                 <geometry>
-                    <box size="0.014 0.006 0.014"/>
+                    <mesh filename="package://rm_description/meshes/sentry/driven_wheel1.stl"
+                                              scale="0.001 0.001 0.001"/>
                 </geometry>
             </collision>

File: urdf/sentry/driven_wheel2.urdf.xacro (robot description, xacro)
@@ -18,8 +18,8 @@
             </inertial>
             <collision>
-                <origin xyz="0 0 -0.005" rpy="0 0 0"/>
                 <xacro:insert_block name="pose"/>
                 <geometry>
-                    <box size="0.014 0.014 0.006"/>
+                    <mesh filename="package://rm_description/meshes/sentry/driven_wheel2.stl"
+                                              scale="0.001 0.001 0.001"/>
                 </geometry>
             </collision>

File: urdf/sentry/lower_gimbal.urdf.xacro (robot description, xacro)
@@ -8,4 +8,5 @@
   <link name="lower_yaw">
     <visual>
+      <origin xyz="0 0 0" rpy="0 0 0"/>
       <geometry>
         <mesh filename="package://rm_description/meshes/sentry/lower_yaw.stl"
@@ -14,19 +15,14 @@
     </visual>
     <inertial>
-      <mass value="599.396e-3"/>
-      <origin xyz="-67.151e-3 -7.823e-3 -37.636e-3" rpy="0 0 0"/>
-      <inertia ixx="3.787e-4" ixy="-46745.03e-9" ixz="5459.222e-9" iyy="8.443e-4"
-               iyz="1835.055e-9" izz="6.561e-4"/>
+      <mass value="99.15e-3"/>
+      <origin xyz="-10.311e-3 -2.902e-3 -40.101e-3" rpy="0 0 0"/>
+      <inertia ixx="1.456e-4" ixy="-7242.148e-9" ixz="-28572.972e-9" iyy="1.608e-4"
+               iyz="-13303.908e-9" izz="52950.519e-9"/>
     </inertial>
     <collision>
-      <origin xyz="-0.008 0 -0.0535" rpy="0 0 0"/>
+      <origin xyz="0 0 0" rpy="0 0 0"/>
       <geometry>
-        <box size="0.085 0.069 0.13"/>
-      </geometry>
-    </collision>
-    <collision>
-      <origin xyz="-0.0822 0.02 -0.06" rpy="0 0 0"/>
-      <geometry>
-        <box size="0.064 0.028 0.12"/>
+        <mesh filename="package://rm_description/meshes/sentry/lower_yaw_collision.stl"
+                      scale="0.001 0.001 0.001"/>
       </geometry>
     </collision>
@@ -45,8 +41,8 @@
   <link name="lower_pitch">
     <inertial>
-      <mass value="584.157e-3"/>
-      <origin xyz="31.362e-3 -0.689e-3 -36.945e-3"/>
-      <inertia ixx="1.030e-3" ixy="-18463.46e-9" ixz="-9.122e-4" iyy="4.507e-3"
-               iyz="8105.967e-9" izz="4.096e-3"/>
+      <mass value="809.574e-3"/>
+      <origin xyz="21.588e-3 -0.686e-3 -30.256e-3"/>
+      <inertia ixx="2.031e-3" ixy="-27414.264e-9" ixz="-55245.014e-9" iyy="6.195e-3"
+               iyz="31445.023e-9" izz="4.728e-3"/>
     </inertial>
     <visual>
@@ -57,19 +53,7 @@
     </visual>
     <collision>
-      <origin xyz="-0.005 0 -0.065" rpy="0 0 0"/>
+      <origin xyz="0 0 0" rpy="0 0 0"/>
       <geometry>
-        <box size="0.25 0.075 0.068"/>
-      </geometry>
-    </collision>
-    <collision>
-      <origin xyz="0.125 0 0" rpy="0 0 0"/>
-      <geometry>
-        <box size="0.12 0.045 0.045"/>
-      </geometry>
-    </collision>
-    <collision>
-      <origin xyz="0.045 0 -0.008" rpy="0 0 0"/>
-      <geometry>
-        <box size="0.065 0.14 0.05"/>
+        <mesh filename="package://rm_description/meshes/sentry/lower_pitch_collision.stl" scale="0.001 0.001 0.001"/>
       </geometry>
     </collision>
@@ -86,5 +70,5 @@
                        soft_upper_limit="${pitch_upper_limit-threshold}"/>
   </joint>
-  <link name="lower_camera">
+  <!-- <link name="lower_camera">
     <inertial>
       <mass value="0.111"/>
@@ -100,5 +84,5 @@
     </visual>
     <collision>
-      <origin xyz="0.021 0 -0.015" rpy="0 0 0"/>
+      <origin xyz="0 0 -0.015" rpy="0 0 0"/>
       <geometry>
         <box size="0.0892 0.04 0.04"/>
@@ -109,6 +93,6 @@
      <parent link="lower_pitch"/>
      <child link="lower_camera"/>
-     <origin xyz="29.642e-3 0 -54.20e-3" rpy="0 0 0"/>
+     <origin xyz="19.642e-3 0 -54.20e-3" rpy="0 0 0"/>
      <axis xyz="0 0 1"/>
-  </joint>
+  </joint>-->
 </robot>

File: urdf/sentry/lower_shooter.urdf.xacro (robot description, xacro)
@@ -24,7 +24,7 @@
     </visual>
     <collision>
-      <origin xyz="0.005 0 -0.02" rpy="0 0 0"/>
+      <origin xyz="0 0 0" rpy="0 0 0"/>
       <geometry>
-        <box size="0.106 0.1 0.0663"/>
+        <mesh filename="package://rm_description/meshes/sentry/lower_trigger_collision.stl" scale="0.001 0.001 0.001"/>
       </geometry>
     </collision>

File: urdf/sentry/sentry.urdf.xacro (robot description, xacro)
@@ -4,4 +4,8 @@
     <xacro:arg name="load_gimbal" default="true"/>
     <xacro:arg name="load_shooter" default="true"/>
+    <xacro:arg name="upper_camera_link" default="upper_camera_link"/>
+    <xacro:arg name="upper_camera_optical_frame" default="upper_camera_optical_frame"/>
+    <xacro:arg name="lower_camera_link" default="lower_camera_link"/>
+    <xacro:arg name="lower_camera_optical_frame" default="lower_camera_optical_frame"/>
     <xacro:arg name="use_simulation" default="true"/>
     <xacro:if value="$(arg load_chassis)">
@@ -13,6 +17,23 @@
         <xacro:include filename="$(find rm_description)/urdf/sentry/lower_gimbal.urdf.xacro"/>
         <xacro:include filename="$(find rm_description)/urdf/sentry/lower_gimbal.transmission.urdf.xacro"/>
+        <xacro:include filename="$(find rm_description)/urdf/common/camera.urdf.xacro"/>
+        <xacro:include filename="$(find rm_description)/urdf/common/imu.urdf.xacro"/>
+        <xacro:IMU connected_to="lower_pitch" imu_name="lower_gimbal_imu" xyz="-0.0348 0 -0.0772" rpy="0 0 -${pi/2}"/>
+        <xacro:camera_sensor xyz="0.015 0 -0.052" rpy="0 0 0" frame_id="$(arg lower_camera_link)" parent="lower_pitch"
+                             camera_sim="$(arg use_simulation)"/>
+        <xacro:camera_optical_frame xyz="0.153 0 -0.0615" rpy="${pi/2} 0 ${pi/2}"
+                                    frame_id="$(arg lower_camera_optical_frame)"
+                                    parent="lower_pitch" camera_sim="$(arg use_simulation)"/>
         <xacro:include filename="$(find rm_description)/urdf/sentry/upper_gimbal.urdf.xacro"/>
         <xacro:include filename="$(find rm_description)/urdf/sentry/upper_gimbal.transmission.urdf.xacro"/>
+        <xacro:include filename="$(find rm_description)/urdf/common/camera.urdf.xacro"/>
+        <xacro:include filename="$(find rm_description)/urdf/common/imu.urdf.xacro"/>
+        <xacro:IMU connected_to="upper_pitch" imu_name="upper_gimbal_imu" xyz="-0.0348 0 0.0772" rpy="0 0 -${pi/2}"/>
+        <xacro:include filename="$(find rm_description)/urdf/common/camera.urdf.xacro"/>
+        <xacro:camera_sensor xyz="11.642e-3 0 81.20e-3" rpy="0 0 0" frame_id="$(arg upper_camera_link)" parent="upper_pitch"
+                             camera_sim="$(arg use_simulation)"/>
+        <xacro:camera_optical_frame xyz="0.153 0 -0.0615" rpy="${-pi/2} 0 ${-pi/2}"
+                                    frame_id="$(arg upper_camera_optical_frame)"
+                                    parent="upper_pitch" camera_sim="$(arg use_simulation)"/>
     </xacro:if>
     <xacro:if value="$(arg load_shooter)">

File: urdf/sentry/upper_gimbal.urdf.xacro (robot description, xacro)
@@ -8,4 +8,5 @@
     <link name="upper_yaw">
         <visual>
+            <origin xyz="0 0 0" rpy="0 0 0"/>
             <geometry>
                 <mesh filename="package://rm_description/meshes/sentry/upper_yaw.stl"
@@ -14,20 +15,15 @@
         </visual>
         <inertial>
-            <mass value="599.396e-3"/>
-            <origin xyz="-67.151e-3 7.823e-3 37.636e-3" rpy="0 0 0"/>
-            <inertia ixx="3.787e-4" ixy="46745.03e-9" ixz="5459.222e-9" iyy="8.443e-4"
-                     iyz="1835.055e-9" izz="6.561e-4"/>
+            <mass value="173.01e-3"/>
+            <origin xyz="-20.009e-3 23.734e-3 62.295e-3" rpy="0 0 0"/>
+            <inertia ixx="8.0227e-4" ixy="1.063e-4" ixz="2.307e-4" iyy="7.448e-4"
+                     iyz="-2.615e-4" izz="3.223e-4"/>
         </inertial>
         <collision>
-            <origin xyz="-0.008 0 0.0535" rpy="0 0 0"/>
-            <geometry>
-                <box size="0.085 0.069 0.13"/>
-            </geometry>
-        </collision>
-        <collision>
-            <origin xyz="-0.0822 -0.02 0.06" rpy="0 0 0"/>
-            <geometry>
-                <box size="0.064 0.028 0.12"/>
-            </geometry>
+          <origin xyz="0 0 0" rpy="0 0 0"/>
+          <geometry>
+            <mesh filename="package://rm_description/meshes/sentry/upper_yaw_collision.stl"
+                                  scale="0.001 0.001 0.001"/>
+          </geometry>
         </collision>
     </link>
@@ -45,8 +41,8 @@
     <link name="upper_pitch">
       <inertial>
-        <mass value="584.157e-3"/>
-        <origin xyz="31.362e-3 0.689e-3 36.945e-3"/>
-        <inertia ixx="1.030e-3" ixy="18463.46e-9" ixz="9.122e-4" iyy="4.507e-3"
-                 iyz="8105.967e-9" izz="4.096e-3"/>
+        <mass value="809.574e-3"/>
+        <origin xyz="21.588e-3 0.686e-3 30.256e-3"/>
+        <inertia ixx="2.031e-3" ixy="27414.264e-9" ixz="55245.014e-9" iyy="6.195e-3"
+                 iyz="31445.023e-9" izz="4.728e-3"/>
       </inertial>
       <visual>
@@ -57,13 +53,7 @@
       </visual>
       <collision>
-        <origin xyz="-0.005 0 0.065" rpy="0 0 0"/>
+        <origin xyz="0 0 0" rpy="0 0 0"/>
         <geometry>
-          <box size="0.25 0.075 0.068"/>
-        </geometry>
-      </collision>
-      <collision>
-        <origin xyz="0.125 0 0" rpy="0 0 0"/>
-        <geometry>
-          <box size="0.12 0.045 0.045"/>
+          <mesh filename="package://rm_description/meshes/sentry/upper_pitch_collision.stl" scale="0.001 0.001 0.001"/>
         </geometry>
       </collision>
@@ -80,5 +70,5 @@
                          soft_upper_limit="${pitch_upper_limit-threshold}"/>
     </joint>
-    <link name="upper_camera">
+    <!-- <link name="upper_camera">
       <inertial>
         <mass value="0.111"/>
@@ -94,5 +84,5 @@
       </visual>
       <collision>
-        <origin xyz="0.021 0 0.015" rpy="0 0 0"/>
+        <origin xyz="0 0 0.015" rpy="0 0 0"/>
         <geometry>
           <box size="0.0892 0.04 0.04"/>
@@ -103,6 +93,6 @@
        <parent link="upper_pitch"/>
        <child link="upper_camera"/>
-       <origin xyz="29.642e-3 0 54.20e-3" rpy="0 0 0"/>
+       <origin xyz="19.642e-3 0 54.20e-3" rpy="0 0 0"/>
        <axis xyz="0 0 1"/>
-    </joint>
+    </joint>-->
 </robot>

File: urdf/sentry/upper_shooter.urdf.xacro (robot description, xacro)
@@ -14,7 +14,7 @@
         </visual>
         <collision>
-            <origin xyz="0 -0.00125 0.012" rpy="0 0 0"/>
+            <origin xyz="0 0 0" rpy="0 0 0"/>
             <geometry>
-                <box size="0.072 0.07 0.055"/>
+                <mesh filename="package://rm_description/meshes/sentry/upper_friction_wheel.stl" scale="0.001 0.001 0.001"/>
             </geometry>
         </collision>
@@ -22,4 +22,6 @@
     <joint name="upper_left_friction_wheel_joint" type="continuous">
         <origin xyz="47e-3 36.50e-3 -0.4e-3" rpy="0 0 0"/>
+        <dynamics damping="0.0" friction="0.01"/>
+        <limit upper="1e16" lower="-1e16" effort="0.156" velocity="942.66"/>
         <parent link="upper_pitch"/>
         <child link="upper_left_friction"/>
@@ -40,7 +42,7 @@
         </visual>
         <collision>
-            <origin xyz="0 0.00125 0.012" rpy="0 0 0"/>
+            <origin xyz="0 0 0" rpy="0 0 0"/>
             <geometry>
-                <box size="0.072 0.07 0.055"/>
+                <mesh filename="package://rm_description/meshes/sentry/upper_friction_wheel.stl" scale="0.001 0.001 0.001"/>
             </geometry>
         </collision>
@@ -48,4 +50,6 @@
     <joint name="upper_right_friction_wheel_joint" type="continuous">
         <origin xyz="47e-3 -36.50e-3 -0.4e-3" rpy="0 0 0"/>
+        <dynamics damping="0.0" friction="0.01"/>
+        <limit upper="1e16" lower="-1e16" effort="0.156" velocity="942.66"/>
         <parent link="upper_pitch"/>
         <child link="upper_right_friction"/>
@@ -66,7 +70,7 @@
         </visual>
         <collision>
-            <origin xyz="0 0 0.006" rpy="0 0 0"/>
+            <origin xyz="0 0 0" rpy="0 0 0"/>
             <geometry>
-                <box size="0.105 0.104 0.045"/>
+                <mesh filename="package://rm_description/meshes/sentry/upper_trigger_collision.stl" scale="0.001 0.001 0.001"/>
             </geometry>
         </collision>
