Commit message: Updated new version sentry's urdf.

File: urdf/sentry/chassis.transmission.urdf.xacro (robot description, xacro)
@@ -4,5 +4,5 @@
         <type>transmission_interface/SimpleTransmission</type>
         <actuator name="drive_joint_motor">
-            <mechanicalReduction>19.2032</mechanicalReduction>
+            <mechanicalReduction>-13</mechanicalReduction>
         </actuator>
         <joint name="drive_wheel_joint">
@@ -10,3 +10,12 @@
         </joint>
     </transmission>
+    <transmission name="trans_catapult_joint">
+        <type>transmission_interface/SimpleTransmission</type>
+        <actuator name="catapult_motor">
+            <mechanicalReduction>-1</mechanicalReduction>
+        </actuator>
+        <joint name="catapult_joint">
+            <hardwareInterface>hardware_interface/EffortJointInterface</hardwareInterface>
+        </joint>
+    </transmission>
 </robot>

File: urdf/sentry/chassis.urdf.xacro (robot description, xacro)
@@ -2,12 +2,11 @@
     <xacro:include filename="driven_wheel1.urdf.xacro"/>
     <xacro:include filename="driven_wheel2.urdf.xacro"/>
-    <xacro:include filename="driven_wheel3.urdf.xacro"/>
     <xacro:macro name="chassis" params="use_simulation">
         <link name="base_link">
             <inertial>
-                <mass value="6982.046e-3"/>
-                <origin xyz="2.335e-3 21.529e-3 -63.905e-3"/>
-                <inertia ixx="1.984e-1" ixy="1.366e-3" ixz="2.748e-3" iyy="1.284e-1"
-                         iyz="3.820e-3" izz="1.524e-1"/>
+                <mass value="6392.711e-3"/>
+                <origin xyz="17.924e-3 -11.095e-3 51.909e-3"/>
+                <inertia ixx="1.795e-1" ixy="4.102e-3" ixz="-8.862e-3" iyy="1.461e-1"
+                         iyz="1.34e-2" izz="1.896e-1"/>
             </inertial>
             <visual>
@@ -26,8 +25,8 @@
         <link name="drive_wheel_link">
             <inertial>
-                <mass value="65.448e-3"/>
-                <origin xyz="0.027e-3 29.066e-3 0.001e-3"/>
-                <inertia ixx="74809.989e-9" ixy="-10.328e-9" ixz="-0.001e-9" iyy="32620.511e-9"
-                         iyz="-2.066e-9" izz="74795.135e-9"/>
+                <mass value="132.98e-3"/>
+                <origin xyz="-8.446e-13 -5.201e-3 -1.155e-12"/>
+                <inertia ixx="1.885e-4" ixy="1.005e-15" ixz="0.002e-9" iyy="3.687e-4"
+                         iyz="2.311e-15" izz="1.885e-4"/>
             </inertial>
             <visual>
@@ -38,7 +37,7 @@
             </visual>
             <collision>
-                <origin xyz="0 0 0" rpy="0 0 0"/>
+                <origin xyz="0 -0.004 0" rpy="0 0 0"/>
                 <geometry>
-                    <mesh filename="package://rm_description/meshes/sentry/drive_wheel.stl" scale="0.001 0.001 0.001"/>
+                    <box size="0.127 0.02435 0.127"/>
                 </geometry>
             </collision>
@@ -49,37 +48,121 @@
             <parent link="base_link"/>
             <child link="drive_wheel_link"/>
-            <origin xyz="0 -63.36e-3 5e-3" rpy="0 0 0"/>
+            <origin xyz="0 51.65e-3 94.5e-3" rpy="0 0 0"/>
+        </joint>
+        <link name="slider_link">
+            <inertial>
+                <mass value="66.212e-3"/>
+                <origin xyz="-3.002e-3 -13.823e-3 14.751e-3"/>
+                <inertia ixx="20612.923e-9" ixy="-2537.219e-9" ixz="-2423.351e-9" iyy="78493.793e-9"
+                         iyz="-347.633e-9" izz="86435.358e-9"/>
+            </inertial>
+            <visual>
+                <origin xyz="0 0 0" rpy="0 0 0"/>
+                <geometry>
+                    <mesh filename="package://rm_description/meshes/sentry/slider.stl" scale="0.001 0.001 0.001"/>
+                </geometry>
+            </visual>
+            <collision>
+                <origin xyz="-0.01 -0.001 0.01" rpy="0 0 0"/>
+                <geometry>
+                    <box size="0.14 0.064 0.0353"/>
+                </geometry>
+            </collision>
+        </link>
+        <joint name="slider_joint" type="prismatic">
+            <axis xyz="1 0 0"/>
+            <limit effort="1.2" velocity="34" lower="-1e9" upper="1e9"/>
+            <parent link="base_link"/>
+            <child link="slider_link"/>
+            <origin xyz="12e-3 -87e-3 43.70e-3" rpy="0 0 0"/>
+        </joint>
+        <link name="catapult_link">
+            <inertial>
+                <mass value="166.084e-3"/>
+                <origin xyz="-27.478e-3 -1.971e-3 -14.369e-3"/>
+                <inertia ixx="3.3471e-4" ixy="-5535.584e-9" ixz="2.741e-4" iyy="6.09e-4"
+                         iyz="23411.215e-9" izz="3.63e-4"/>
+            </inertial>
+            <visual>
+                <origin xyz="0 0 0" rpy="0 0 0"/>
+                <geometry>
+                    <mesh filename="package://rm_description/meshes/sentry/catapult.stl" scale="0.001 0.001 0.001"/>
+                </geometry>
+            </visual>
+            <collision>
+                <origin xyz="0 0 0" rpy="0 0 0"/>
+                <geometry>
+                    <mesh filename="package://rm_description/meshes/sentry/catapult.stl" scale="0.001 0.001 0.001"/>
+                </geometry>
+            </collision>
+        </link>
+        <joint name="catapult_joint" type="revolute">
+            <axis xyz="0 1 0"/>
+            <limit effort="1.2" velocity="34" lower="-1e9" upper="1e9"/>
+            <parent link="slider_link"/>
+            <child link="catapult_link"/>
+            <origin xyz="0 0 0" rpy="0 0 0"/>
         </joint>
         <xacro:if value="$(arg use_simulation)">
             <xacro:driven_wheel1 num="1">
-                <origin rpy="${-pi/2} 0 0"/>
+                <origin xyz="0 -2.5e-3 -8.008e-13" rpy="0 0 0"/>
                 <axis xyz="0 1 0"/>
-                <origin xyz="-0.0977 0.0839 -0.013" rpy="0 0 0"/>
+                <origin xyz="257.5e-3 -72.5e-3 37e-3" rpy="0 0 0"/>
             </xacro:driven_wheel1>
             <xacro:driven_wheel1 num="2">
-                <origin rpy="${-pi/2} 0 0"/>
+                <origin xyz="0 -2.5e-3 -8.008e-13" rpy="0 0 0"/>
                 <axis xyz="0 1 0"/>
-                <origin xyz="0.0977 0.0839 -0.013" rpy="0 0 0"/>
+                <origin xyz="-257.5e-3 -72.5e-3 37e-3" rpy="0 0 0"/>
             </xacro:driven_wheel1>
-            <xacro:driven_wheel2 num="3">
-                <origin rpy="0 0 0"/>
+            <xacro:driven_wheel1 num="3">
+                <origin xyz="0 -2.5e-3 -8.008e-13" rpy="0 0 0"/>
+                <axis xyz="0 1 0"/>
+                <origin xyz="-125e-3 65.2e-3 37e-3" rpy="0 0 0"/>
+            </xacro:driven_wheel1>
+            <xacro:driven_wheel1 num="4">
+                <origin xyz="0 -2.5e-3 -8.008e-13" rpy="0 0 0"/>
+                <axis xyz="0 1 0"/>
+                <origin xyz="125e-3 65.2e-3 37e-3" rpy="0 0 0"/>
+            </xacro:driven_wheel1>
+            <xacro:driven_wheel1 num="5">
+                <origin xyz="0 -2.5e-3 -8.008e-13" rpy="0 0 0"/>
+                <axis xyz="0 1 0"/>
+                <origin xyz="105e-3 -33.5e-3 -40e-3" rpy="0 0 0"/>
+            </xacro:driven_wheel1>
+            <xacro:driven_wheel1 num="6">
+                <origin xyz="0 -2.5e-3 -8.008e-13" rpy="0 0 0"/>
+                <axis xyz="0 1 0"/>
+                <origin xyz="-105e-3 -33.5e-3 -40e-3" rpy="0 0 0"/>
+            </xacro:driven_wheel1>
+            <xacro:driven_wheel1 num="7">
+                <origin xyz="0 -2.5e-3 -8.008e-13" rpy="0 0 0"/>
+                <axis xyz="0 1 0"/>
+                <origin xyz="-85e-3 44.5e-3 -40e-3" rpy="0 0 0"/>
+            </xacro:driven_wheel1>
+            <xacro:driven_wheel1 num="8">
+                <origin xyz="0 -2.5e-3 -8.008e-13" rpy="0 0 0"/>
+                <axis xyz="0 1 0"/>
+                <origin xyz="85e-3 44.5e-3 -40e-3" rpy="0 0 0"/>
+            </xacro:driven_wheel1>
+            <xacro:driven_wheel2 num="9">
+                <origin xyz="0 8.008e-13 -2.5e-3" rpy="0 0 0"/>
                 <axis xyz="0 0 1"/>
-                <origin xyz="0.11 0.098 -0.05486" rpy="0 0 0"/>
+                <origin xyz="192e-3 -97e-3 -5e-4" rpy="0 0 0"/>
             </xacro:driven_wheel2>
-            <xacro:driven_wheel2 num="4">
-                <origin rpy="0 0 0"/>
+            <xacro:driven_wheel2 num="10">
+                <origin xyz="0 8.008e-13 -2.5e-3" rpy="0 0 0"/>
                 <axis xyz="0 0 1"/>
-                <origin xyz="-0.11 0.098 -0.05486" rpy="0 0 0"/>
+                <origin xyz="-139.95e-3 -97e-3 4e-3" rpy="0 0 0"/>
             </xacro:driven_wheel2>
-            <xacro:driven_wheel3 num="5">
-                <origin rpy="0 0 0"/>
+            <xacro:driven_wheel2 num="11">
+                <origin xyz="0 8.008e-13 -2.5e-3" rpy="0 0 0"/>
                 <axis xyz="0 0 1"/>
-                <origin xyz="-0.07 -0.1 -0.05527" rpy="0 0 0"/>
-            </xacro:driven_wheel3>
-            <xacro:driven_wheel3 num="6">
-                <origin rpy="0 0 0"/>
+                <origin xyz="149e-3 97e-3 4e-3" rpy="0 0 0"/>
+            </xacro:driven_wheel2>
+            <xacro:driven_wheel2 num="12">
+               <origin xyz="0 8.008e-13 -2.5e-3" rpy="0 0 0"/>
                 <axis xyz="0 0 1"/>
-                <origin xyz="0.07 -0.1 0.05527" rpy="0 0 0"/>
-            </xacro:driven_wheel3>
+                <origin xyz="-149e-3 97e-3 4e-3" rpy="0 0 0"/>
+            </xacro:driven_wheel2>
         </xacro:if>
     </xacro:macro>

File: urdf/sentry/driven_wheel1.urdf.xacro (robot description, xacro)
@@ -1,37 +1,36 @@
 <robot xmlns:xacro="http://www.ros.org/wiki/xacro">
-  <xacro:property name="wheel_joint_effort" value="5"/>
-  <xacro:property name="wheel_joint_velocity" value="50"/>
-  <xacro:macro name="driven_wheel1" params="num *pose *axis *origin ">
-      <link name="link_driven_wheel${num}">
-          <visual>
-              <xacro:insert_block name="pose"/>
-              <geometry>
-                  <mesh filename="package://rm_description/meshes/sentry/driven_wheel1.stl"
-                        scale="0.001 0.001 0.001"/>
-              </geometry>
-          </visual>
-          <inertial>
-              <mass value="11.136e-3"/>
-              <origin xyz="0 0 0" rpy="0 0 0"/>
-              <inertia ixx="2319.294e-9" ixy="-0.016e-9" ixz="-2.80e-9" iyy="2720.243e-9"
-                       iyz="-7.716e-9" izz="1014.719e-9"/>
-          </inertial>
-          <collision>
-              <!--        <origin xyz="0 0 0" rpy="0 0 0"/>-->
-              <xacro:insert_block name="pose"/>
-              <geometry>
-                  <mesh filename="package://rm_description/meshes/sentry/driven_wheel1.stl"
-                        scale="0.001 0.001 0.001"/>
-              </geometry>
-          </collision>
-      </link>
-    <joint name="joint_wheel${num}" type="continuous">
-      <parent link="base_link"/>
-      <child link="link_driven_wheel${num}"/>
-      <xacro:insert_block name="axis"/>
-      <xacro:insert_block name="origin"/>
-      <limit effort="${wheel_joint_effort}" velocity="${wheel_joint_velocity}" lower="-1e16" upper="1e16"/>
-      <dynamics damping="0.0" friction="0.05"/>
-    </joint>
-  </xacro:macro>
+    <xacro:property name="wheel_joint_effort" value="5"/>
+    <xacro:property name="wheel_joint_velocity" value="50"/>
+    <xacro:macro name="driven_wheel1" params="num *pose *axis *origin ">
+        <link name="link_driven_wheel${num}">
+            <visual>
+                <xacro:insert_block name="pose"/>
+                <geometry>
+                    <mesh filename="package://rm_description/meshes/sentry/driven_wheel1.stl"
+                          scale="0.001 0.001 0.001"/>
+                </geometry>
+            </visual>
+            <inertial>
+                <mass value="2.388e-3"/>
+                <origin xyz="0 0 0" rpy="0 0 0"/>
+                <inertia ixx="15.764e-9" ixy="0" ixz="0" iyy="19.664e-9"
+                         iyz="1.425e-18" izz="15.764e-9"/>
+            </inertial>
+            <collision>
+                <origin xyz="0 0.00015 0" rpy="0 0 0"/>
+                <xacro:insert_block name="pose"/>
+                <geometry>
+                    <box size="0.014 0.006 0.014"/>
+                </geometry>
+            </collision>
+        </link>
+        <joint name="joint_wheel${num}" type="continuous">
+            <parent link="base_link"/>
+            <child link="link_driven_wheel${num}"/>
+            <xacro:insert_block name="axis"/>
+            <xacro:insert_block name="origin"/>
+            <limit effort="${wheel_joint_effort}" velocity="${wheel_joint_velocity}" lower="-1e16" upper="1e16"/>
+            <dynamics damping="0.0" friction="0.05"/>
+        </joint>
+    </xacro:macro>
 </robot>

File: urdf/sentry/driven_wheel2.urdf.xacro (robot description, xacro)
@@ -12,19 +12,18 @@
             </visual>
             <inertial>
-                <mass value="1.527e-3"/>
+                <mass value="0.712e-3"/>
                 <origin xyz="0 0 0" rpy="0 0 0"/>
-                <inertia ixx="29.25e-9" ixy="-3.862e-14" ixz="-0.001e-9" iyy="29.251e-9"
-                         iyz="-0.001e-9" izz="52.083e-9"/>
+                <inertia ixx="11.315e-9" ixy="0" ixz="0" iyy="11.315e-9"
+                         iyz="0" izz="19.664e-9"/>
             </inertial>
             <collision>
-                <!--        <origin xyz="0 0 0" rpy="0 0 0"/>-->
+                <origin xyz="0 0 -0.005" rpy="0 0 0"/>
                 <xacro:insert_block name="pose"/>
                 <geometry>
-                    <mesh filename="package://rm_description/meshes/sentry/driven_wheel2.stl"
-                          scale="0.001 0.001 0.001"/>
+                    <box size="0.014 0.014 0.006"/>
                 </geometry>
             </collision>
         </link>
-        <joint name="joint_wheel${num}" type="continuous">
+        <joint name="joint_wheel${num}" type="revolute">
             <parent link="base_link"/>
             <child link="link_driven_wheel${num}"/>

File: urdf/sentry/lower_gimbal.urdf.xacro (robot description, xacro)
@@ -14,14 +14,19 @@
     </visual>
     <inertial>
-      <mass value="1.84153"/>
-      <origin xyz="-48.613e-3 -7.311e-3 -40.711e-3" rpy="0 0 0"/>
-      <inertia ixx="9.308e-3" ixy="1.131e-3" ixz="-2.237e-3" iyy="2.582e-2"
-               iyz="-5.566e-4" izz="2.598e-2"/>
+      <mass value="599.396e-3"/>
+      <origin xyz="-67.151e-3 -7.823e-3 -37.636e-3" rpy="0 0 0"/>
+      <inertia ixx="3.787e-4" ixy="-46745.03e-9" ixz="5459.222e-9" iyy="8.443e-4"
+               iyz="1835.055e-9" izz="6.561e-4"/>
     </inertial>
     <collision>
-      <origin xyz="0 0 0" rpy="0 0 0"/>
+      <origin xyz="-0.008 0 -0.0535" rpy="0 0 0"/>
       <geometry>
-        <mesh filename="package://rm_description/meshes/sentry/lower_yaw.stl"
-              scale="0.001 0.001 0.001"/>
+        <box size="0.085 0.069 0.13"/>
+      </geometry>
+    </collision>
+    <collision>
+      <origin xyz="-0.0822 0.02 -0.06" rpy="0 0 0"/>
+      <geometry>
+        <box size="0.064 0.028 0.12"/>
       </geometry>
     </collision>
@@ -31,5 +36,5 @@
     <child link="lower_yaw"/>
     <axis xyz="0 0 1"/>
-    <origin xyz="2.261e-3 31.206e-3 -235.253e-3"/>
+    <origin xyz="0 0 -129e-3"/>
     <dynamics damping="0" friction="0.1"/>
     <limit effort="1.2" velocity="34" lower="${yaw_lower_limit}" upper="${yaw_upper_limit}"/>
@@ -40,8 +45,8 @@
   <link name="lower_pitch">
     <inertial>
-      <mass value="725.237e-3"/>
-      <origin xyz="4.587e-3 2.933e-3 17.233e-3"/>
-      <inertia ixx="2.408e-3" ixy="7.760e-5" ixz="-8.109e-5" iyy="1.183e-3"
-               iyz="-1.337e-4" izz="2.824e-3"/>
+      <mass value="584.157e-3"/>
+      <origin xyz="31.362e-3 -0.689e-3 -36.945e-3"/>
+      <inertia ixx="1.030e-3" ixy="-18463.46e-9" ixz="-9.122e-4" iyy="4.507e-3"
+               iyz="8105.967e-9" izz="4.096e-3"/>
     </inertial>
     <visual>
@@ -52,7 +57,19 @@
     </visual>
     <collision>
-      <origin xyz="0 0 0" rpy="0 0 0"/>
+      <origin xyz="-0.005 0 -0.065" rpy="0 0 0"/>
       <geometry>
-        <mesh filename="package://rm_description/meshes/sentry/lower_pitch.stl" scale="0.001 0.001 0.001"/>
+        <box size="0.25 0.075 0.068"/>
+      </geometry>
+    </collision>
+    <collision>
+      <origin xyz="0.125 0 0" rpy="0 0 0"/>
+      <geometry>
+        <box size="0.12 0.045 0.045"/>
+      </geometry>
+    </collision>
+    <collision>
+      <origin xyz="0.045 0 -0.008" rpy="0 0 0"/>
+      <geometry>
+        <box size="0.065 0.14 0.05"/>
       </geometry>
     </collision>
@@ -62,5 +79,5 @@
     <child link="lower_pitch"/>
     <axis xyz="0 1 0"/>
-    <origin xyz="0 0 -0.1"/>
+    <origin xyz="0 0 -87.993e-3"/>
     <dynamics damping="0" friction="0.1"/>
     <limit effort="1.2" velocity="13.82" lower="${pitch_lower_limit}" upper="${pitch_upper_limit}"/>
@@ -69,29 +86,29 @@
                        soft_upper_limit="${pitch_upper_limit-threshold}"/>
   </joint>
-  <!--  <link name="upper_camera">-->
-  <!--    <inertial>-->
-  <!--          <mass value="0.17671"/>-->
-  <!--          <origin xyz="0.022 0.0 0.0"/>-->
-  <!--          <inertia ixx="2.129e-5" ixy="7.329e-8" ixz="-1.11e-7" iyy="2.198e-4" iyz="-8.04e-7" izz="2.197e-4"/>-->
-  <!--        </inertial>-->
-  <!--        <visual>-->
-  <!--          <origin xyz=" 0 0 0 " rpy="0 -1.57 0"/>-->
-  <!--          <geometry>-->
-  <!--            <mesh filename="package://rm_description/meshes/common/camera.stl" scale="0.001 0.001 0.001"/>-->
-  <!--          </geometry>-->
-  <!--          <material name="Black"/>-->
-  <!--        </visual>-->
-  <!--        <collision>-->
-  <!--          <origin xyz="0 0 0" rpy="0 -1.57 0"/>-->
-  <!--          <geometry>-->
-  <!--            <mesh filename="package://rm_description/meshes/common/camera.stl" scale="0.001 0.001 0.001"/>-->
-  <!--          </geometry>-->
-  <!--        </collision>-->
-  <!--      </link>-->
-  <!--      <joint name="camera_joint" type="fixed">-->
-  <!--        <parent link="pitch"/>-->
-  <!--        <child link="camera"/>-->
-  <!--        <origin xyz="0.086  0.0 -0.040" rpy="-1.57 0 -1.57"/>-->
-  <!--        <axis xyz="0 0 1"/>-->
-  <!--      </joint>-->
+  <link name="lower_camera">
+    <inertial>
+      <mass value="0.111"/>
+      <origin xyz="24.789e-3 -0.019e-3 -14.471e-3"/>
+      <inertia ixx="15645.374e-9" ixy="-94.19e-9" ixz="143.444e-9" iyy="80877.924e-9"
+               iyz="-45.908e-9" izz="80823.702e-9"/>
+    </inertial>
+    <visual>
+      <origin xyz=" 0 0 0 " rpy="0 0 0"/>
+      <geometry>
+        <mesh filename="package://rm_description/meshes/sentry/lower_camera.stl" scale="0.001 0.001 0.001"/>
+      </geometry>
+    </visual>
+    <collision>
+      <origin xyz="0.021 0 -0.015" rpy="0 0 0"/>
+      <geometry>
+        <box size="0.0892 0.04 0.04"/>
+      </geometry>
+    </collision>
+  </link>
+  <joint name="lower_camera_joint" type="fixed">
+     <parent link="lower_pitch"/>
+     <child link="lower_camera"/>
+     <origin xyz="29.642e-3 0 -54.20e-3" rpy="0 0 0"/>
+     <axis xyz="0 0 1"/>
+  </joint>
 </robot>

File: urdf/sentry/lower_shooter.urdf.xacro (robot description, xacro)
@@ -1,7 +1,7 @@
 <robot xmlns:xacro="http://www.ros.org/wiki/xacro">
   <xacro:include filename="$(find rm_description)/urdf/common/friction.urdf.xacro"/>
-  <xacro:property name="wheel_offset_x" value="0.0504"/>
-  <xacro:property name="wheel_offset_y" value="0.0365"/>
-  <xacro:property name="wheel_offset_z" value="0.01072"/>
+  <xacro:property name="wheel_offset_x" value="0.047"/>
+  <xacro:property name="wheel_offset_y" value="-0.0365"/>
+  <xacro:property name="wheel_offset_z" value="-0.4e-3"/>
   <xacro:friction_wheel prefixs="lower_left" connected_to="lower_pitch"
                         wheel_x_offset="${wheel_offset_x}" wheel_y_offset="${-wheel_offset_y}"
@@ -12,8 +12,8 @@
   <link name="lower_trigger">
     <inertial>
-      <mass value="0.25496"/>
-      <origin xyz="0.282e-3 0.011e-3 18.873e-3"/>
-      <inertia ixx="2.844e-4" ixy="-432.025e-9" ixz="-882.662e-9" iyy="2.858e-4"
-               iyz="-19.177e-9" izz="2.347e-4"/>
+      <mass value="304.224e-3"/>
+      <origin xyz="-1.589e-3 0.036e-3 -24.868e-3"/>
+      <inertia ixx="3.630e-4" ixy="282.096e-9" ixz="-1745.045e-9" iyy="2.304e-4"
+               iyz="463.877e-9" izz="4.276e-4"/>
     </inertial>
     <visual>
@@ -24,15 +24,14 @@
     </visual>
     <collision>
-      <origin xyz="0 0 0" rpy="0 0 0"/>
+      <origin xyz="0.005 0 -0.02" rpy="0 0 0"/>
       <geometry>
-        <mesh filename="package://rm_description/meshes/sentry/lower_trigger.stl" scale="0.001 0.001 0.001"/>
+        <box size="0.106 0.1 0.0663"/>
       </geometry>
     </collision>
   </link>
   <joint name="lower_trigger_joint" type="continuous">
-    <origin xyz="0 0.15 -0.136" rpy="0 0 0"/>
+    <origin xyz="0 148.02e-3 -29.5e-3" rpy="0 0 0"/>
     <dynamics damping="0.0" friction="0.01"/>
-    <limit effort="1.0" velocity="43.54" lower="-1e16" upper="1e16"/>
-    <parent link="lower_pitch"/>
+    <parent link="base_link"/>
     <child link="lower_trigger"/>
     <axis xyz="0 0 1 "/>
