Commit message: Update sentry urdf

File: urdf/sentry/chassis.transmission.urdf.xacro (robot description, xacro)
@@ -4,5 +4,5 @@
         <type>transmission_interface/SimpleTransmission</type>
         <actuator name="drive_joint_motor">
-            <mechanicalReduction>19.2032</mechanicalReduction>
+            <mechanicalReduction>-13</mechanicalReduction>
         </actuator>
         <joint name="drive_wheel_joint">
@@ -10,3 +10,13 @@
         </joint>
     </transmission>
+    <transmission name="trans_catapult_joint">
+        <type>transmission_interface/SimpleTransmission</type>
+        <actuator name="catapult_motor">
+            <mechanicalReduction>-1</mechanicalReduction>
+        </actuator>
+        <joint name="catapult_joint">
+            <offset>0.28</offset>
+            <hardwareInterface>hardware_interface/EffortJointInterface</hardwareInterface>
+        </joint>
+    </transmission>
 </robot>

File: urdf/sentry/chassis.urdf.xacro (robot description, xacro)
@@ -2,12 +2,11 @@
     <xacro:include filename="driven_wheel1.urdf.xacro"/>
     <xacro:include filename="driven_wheel2.urdf.xacro"/>
-    <xacro:include filename="driven_wheel3.urdf.xacro"/>
     <xacro:macro name="chassis" params="use_simulation">
         <link name="base_link">
             <inertial>
-                <mass value="6982.046e-3"/>
-                <origin xyz="2.335e-3 21.529e-3 -63.905e-3"/>
-                <inertia ixx="1.984e-1" ixy="1.366e-3" ixz="2.748e-3" iyy="1.284e-1"
-                         iyz="3.820e-3" izz="1.524e-1"/>
+                <mass value="6392.711e-3"/>
+                <origin xyz="17.924e-3 -11.095e-3 51.909e-3"/>
+                <inertia ixx="1.795e-1" ixy="4.102e-3" ixz="-8.862e-3" iyy="1.461e-1"
+                         iyz="1.34e-2" izz="1.896e-1"/>
             </inertial>
             <visual>
@@ -26,8 +25,8 @@
         <link name="drive_wheel_link">
             <inertial>
-                <mass value="65.448e-3"/>
-                <origin xyz="0.027e-3 29.066e-3 0.001e-3"/>
-                <inertia ixx="74809.989e-9" ixy="-10.328e-9" ixz="-0.001e-9" iyy="32620.511e-9"
-                         iyz="-2.066e-9" izz="74795.135e-9"/>
+                <mass value="132.98e-3"/>
+                <origin xyz="-8.446e-13 -5.201e-3 -1.155e-12"/>
+                <inertia ixx="1.885e-4" ixy="1.005e-15" ixz="0.002e-9" iyy="3.687e-4"
+                         iyz="2.311e-15" izz="1.885e-4"/>
             </inertial>
             <visual>
@@ -38,7 +37,7 @@
             </visual>
             <collision>
-                <origin xyz="0 0 0" rpy="0 0 0"/>
+                <origin xyz="0 -0.004 0" rpy="0 0 0"/>
                 <geometry>
-                    <mesh filename="package://rm_description/meshes/sentry/drive_wheel.stl" scale="0.001 0.001 0.001"/>
+                    <box size="0.127 0.02435 0.127"/>
                 </geometry>
             </collision>
@@ -46,40 +45,97 @@
         <joint name="drive_wheel_joint" type="revolute">
             <axis xyz="0 1 0"/>
+            <limit effort="3.4" velocity="71.78" lower="-1e9" upper="1e9"/>
+            <parent link="base_link"/>
+            <child link="drive_wheel_link"/>
+            <origin xyz="0 51.65e-3 94.5e-3" rpy="0 0 0"/>
+        </joint>
+        <link name="catapult_link">
+            <inertial>
+                <mass value="166.084e-3"/>
+                <origin xyz="-27.478e-3 -1.971e-3 -14.369e-3"/>
+                <inertia ixx="3.3471e-4" ixy="-5535.584e-9" ixz="2.741e-4" iyy="6.09e-4"
+                         iyz="23411.215e-9" izz="3.63e-4"/>
+            </inertial>
+            <visual>
+                <origin xyz="0 0 0" rpy="0 0 0"/>
+                <geometry>
+                    <mesh filename="package://rm_description/meshes/sentry/catapult.stl" scale="0.001 0.001 0.001"/>
+                </geometry>
+            </visual>
+            <collision>
+                <origin xyz="0 0 0" rpy="0 0 0"/>
+                <geometry>
+                    <mesh filename="package://rm_description/meshes/sentry/catapult.stl" scale="0.001 0.001 0.001"/>
+                </geometry>
+            </collision>
+        </link>
+        <joint name="catapult_joint" type="revolute">
+            <axis xyz="0 1 0"/>
             <limit effort="1.2" velocity="34" lower="-1e9" upper="1e9"/>
             <parent link="base_link"/>
-            <child link="drive_wheel_link"/>
-            <origin xyz="0 -63.36e-3 5e-3" rpy="0 0 0"/>
+            <child link="catapult_link"/>
+            <origin xyz="0 -30e-3 0" rpy="0 0 0"/>
         </joint>
         <xacro:if value="$(arg use_simulation)">
             <xacro:driven_wheel1 num="1">
-                <origin rpy="${-pi/2} 0 0"/>
+                <origin xyz="0 -2.5e-3 -8.008e-13" rpy="0 0 0"/>
                 <axis xyz="0 1 0"/>
-                <origin xyz="-0.0977 0.0839 -0.013" rpy="0 0 0"/>
+                <origin xyz="257.5e-3 -72.5e-3 37e-3" rpy="0 0 0"/>
             </xacro:driven_wheel1>
             <xacro:driven_wheel1 num="2">
-                <origin rpy="${-pi/2} 0 0"/>
+                <origin xyz="0 -2.5e-3 -8.008e-13" rpy="0 0 0"/>
                 <axis xyz="0 1 0"/>
-                <origin xyz="0.0977 0.0839 -0.013" rpy="0 0 0"/>
+                <origin xyz="-257.5e-3 -72.5e-3 37e-3" rpy="0 0 0"/>
             </xacro:driven_wheel1>
-            <xacro:driven_wheel2 num="3">
-                <origin rpy="0 0 0"/>
+            <xacro:driven_wheel1 num="3">
+                <origin xyz="0 -2.5e-3 -8.008e-13" rpy="0 0 0"/>
+                <axis xyz="0 1 0"/>
+                <origin xyz="-125e-3 65.2e-3 37e-3" rpy="0 0 0"/>
+            </xacro:driven_wheel1>
+            <xacro:driven_wheel1 num="4">
+                <origin xyz="0 -2.5e-3 -8.008e-13" rpy="0 0 0"/>
+                <axis xyz="0 1 0"/>
+                <origin xyz="125e-3 65.2e-3 37e-3" rpy="0 0 0"/>
+            </xacro:driven_wheel1>
+            <xacro:driven_wheel1 num="5">
+                <origin xyz="0 -2.5e-3 -8.008e-13" rpy="0 0 0"/>
+                <axis xyz="0 1 0"/>
+                <origin xyz="105e-3 -33.5e-3 -40e-3" rpy="0 0 0"/>
+            </xacro:driven_wheel1>
+            <xacro:driven_wheel1 num="6">
+                <origin xyz="0 -2.5e-3 -8.008e-13" rpy="0 0 0"/>
+                <axis xyz="0 1 0"/>
+                <origin xyz="-105e-3 -33.5e-3 -40e-3" rpy="0 0 0"/>
+            </xacro:driven_wheel1>
+            <xacro:driven_wheel1 num="7">
+                <origin xyz="0 -2.5e-3 -8.008e-13" rpy="0 0 0"/>
+                <axis xyz="0 1 0"/>
+                <origin xyz="-85e-3 44.5e-3 -40e-3" rpy="0 0 0"/>
+            </xacro:driven_wheel1>
+            <xacro:driven_wheel1 num="8">
+                <origin xyz="0 -2.5e-3 -8.008e-13" rpy="0 0 0"/>
+                <axis xyz="0 1 0"/>
+                <origin xyz="85e-3 44.5e-3 -40e-3" rpy="0 0 0"/>
+            </xacro:driven_wheel1>
+            <xacro:driven_wheel2 num="9">
+                <origin xyz="0 8.008e-13 -2.5e-3" rpy="0 0 0"/>
                 <axis xyz="0 0 1"/>
-                <origin xyz="0.11 0.098 -0.05486" rpy="0 0 0"/>
+                <origin xyz="192e-3 -97e-3 -5e-4" rpy="0 0 0"/>
             </xacro:driven_wheel2>
-            <xacro:driven_wheel2 num="4">
-                <origin rpy="0 0 0"/>
+            <xacro:driven_wheel2 num="10">
+                <origin xyz="0 8.008e-13 -2.5e-3" rpy="0 0 0"/>
                 <axis xyz="0 0 1"/>
-                <origin xyz="-0.11 0.098 -0.05486" rpy="0 0 0"/>
+                <origin xyz="-139.95e-3 -97e-3 4e-3" rpy="0 0 0"/>
             </xacro:driven_wheel2>
-            <xacro:driven_wheel3 num="5">
-                <origin rpy="0 0 0"/>
+            <xacro:driven_wheel2 num="11">
+                <origin xyz="0 8.008e-13 -2.5e-3" rpy="0 0 0"/>
                 <axis xyz="0 0 1"/>
-                <origin xyz="-0.07 -0.1 -0.05527" rpy="0 0 0"/>
-            </xacro:driven_wheel3>
-            <xacro:driven_wheel3 num="6">
-                <origin rpy="0 0 0"/>
+                <origin xyz="149e-3 97e-3 4e-3" rpy="0 0 0"/>
+            </xacro:driven_wheel2>
+            <xacro:driven_wheel2 num="12">
+                <origin xyz="0 8.008e-13 -2.5e-3" rpy="0 0 0"/>
                 <axis xyz="0 0 1"/>
-                <origin xyz="0.07 -0.1 0.05527" rpy="0 0 0"/>
-            </xacro:driven_wheel3>
+                <origin xyz="-149e-3 97e-3 4e-3" rpy="0 0 0"/>
+            </xacro:driven_wheel2>
         </xacro:if>
     </xacro:macro>

File: urdf/sentry/lower_gimbal.transmission.urdf.xacro (robot description, xacro)
@@ -7,5 +7,5 @@
         </actuator>
         <joint name="lower_yaw_joint">
-            <offset>2.011</offset>
+            <offset>1.583</offset>
             <hardwareInterface>hardware_interface/EffortJointInterface</hardwareInterface>
         </joint>
@@ -14,8 +14,8 @@
         <type>transmission_interface/SimpleTransmission</type>
         <actuator name="lower_pitch_joint_motor">
-            <mechanicalReduction>1</mechanicalReduction>
+            <mechanicalReduction>11</mechanicalReduction>
         </actuator>
         <joint name="lower_pitch_joint">
-            <offset>1.151</offset>
+            <offset>0.84</offset>
             <hardwareInterface>hardware_interface/EffortJointInterface</hardwareInterface>
         </joint>

File: urdf/sentry/lower_gimbal.urdf.xacro (robot description, xacro)
@@ -1,97 +1,108 @@
 <?xml version="1.0" encoding="utf-8"?>
 <robot xmlns:xacro="http://www.ros.org/wiki/xacro">
-  <xacro:property name="threshold" value="0.03"/>
-  <xacro:property name="yaw_lower_limit" value="-2.461"/>
-  <xacro:property name="yaw_upper_limit" value="1.998"/>
-  <xacro:property name="pitch_lower_limit" value="0.129"/>
-  <xacro:property name="pitch_upper_limit" value="1.175"/>
-  <link name="lower_yaw">
-    <visual>
-      <geometry>
-        <mesh filename="package://rm_description/meshes/sentry/lower_yaw.stl"
-              scale="0.001 0.001 0.001"/>
-      </geometry>
-    </visual>
-    <inertial>
-      <mass value="1.84153"/>
-      <origin xyz="-48.613e-3 -7.311e-3 -40.711e-3" rpy="0 0 0"/>
-      <inertia ixx="9.308e-3" ixy="1.131e-3" ixz="-2.237e-3" iyy="2.582e-2"
-               iyz="-5.566e-4" izz="2.598e-2"/>
-    </inertial>
-    <collision>
-      <origin xyz="0 0 0" rpy="0 0 0"/>
-      <geometry>
-        <mesh filename="package://rm_description/meshes/sentry/lower_yaw.stl"
-              scale="0.001 0.001 0.001"/>
-      </geometry>
-    </collision>
-  </link>
-  <joint name="lower_yaw_joint" type="revolute">
-    <parent link="base_link"/>
-    <child link="lower_yaw"/>
-    <axis xyz="0 0 1"/>
-    <origin xyz="2.261e-3 31.206e-3 -235.253e-3"/>
-    <dynamics damping="0" friction="0.1"/>
-    <limit effort="1.2" velocity="34" lower="${yaw_lower_limit}" upper="${yaw_upper_limit}"/>
-    <safety_controller k_position="100" k_velocity="0.1"
-                       soft_lower_limit="${yaw_lower_limit+threshold}"
-                       soft_upper_limit="${yaw_upper_limit-threshold}"/>
-  </joint>
-  <link name="lower_pitch">
-    <inertial>
-      <mass value="725.237e-3"/>
-      <origin xyz="4.587e-3 2.933e-3 17.233e-3"/>
-      <inertia ixx="2.408e-3" ixy="7.760e-5" ixz="-8.109e-5" iyy="1.183e-3"
-               iyz="-1.337e-4" izz="2.824e-3"/>
-    </inertial>
-    <visual>
-      <origin xyz="0 0 0" rpy="0 0 0"/>
-      <geometry>
-        <mesh filename="package://rm_description/meshes/sentry/lower_pitch.stl" scale="0.001 0.001 0.001"/>
-      </geometry>
-    </visual>
-    <collision>
-      <origin xyz="0 0 0" rpy="0 0 0"/>
-      <geometry>
-        <mesh filename="package://rm_description/meshes/sentry/lower_pitch.stl" scale="0.001 0.001 0.001"/>
-      </geometry>
-    </collision>
-  </link>
-  <joint name="lower_pitch_joint" type="revolute">
-    <parent link="lower_yaw"/>
-    <child link="lower_pitch"/>
-    <axis xyz="0 1 0"/>
-    <origin xyz="0 0 -0.1"/>
-    <dynamics damping="0" friction="0.1"/>
-    <limit effort="1.2" velocity="13.82" lower="${pitch_lower_limit}" upper="${pitch_upper_limit}"/>
-    <safety_controller k_position="100" k_velocity="0.1"
-                       soft_lower_limit="${pitch_lower_limit+threshold}"
-                       soft_upper_limit="${pitch_upper_limit-threshold}"/>
-  </joint>
-  <!--  <link name="upper_camera">-->
-  <!--    <inertial>-->
-  <!--          <mass value="0.17671"/>-->
-  <!--          <origin xyz="0.022 0.0 0.0"/>-->
-  <!--          <inertia ixx="2.129e-5" ixy="7.329e-8" ixz="-1.11e-7" iyy="2.198e-4" iyz="-8.04e-7" izz="2.197e-4"/>-->
-  <!--        </inertial>-->
-  <!--        <visual>-->
-  <!--          <origin xyz=" 0 0 0 " rpy="0 -1.57 0"/>-->
-  <!--          <geometry>-->
-  <!--            <mesh filename="package://rm_description/meshes/common/camera.stl" scale="0.001 0.001 0.001"/>-->
-  <!--          </geometry>-->
-  <!--          <material name="Black"/>-->
-  <!--        </visual>-->
-  <!--        <collision>-->
-  <!--          <origin xyz="0 0 0" rpy="0 -1.57 0"/>-->
-  <!--          <geometry>-->
-  <!--            <mesh filename="package://rm_description/meshes/common/camera.stl" scale="0.001 0.001 0.001"/>-->
-  <!--          </geometry>-->
-  <!--        </collision>-->
-  <!--      </link>-->
-  <!--      <joint name="camera_joint" type="fixed">-->
-  <!--        <parent link="pitch"/>-->
-  <!--        <child link="camera"/>-->
-  <!--        <origin xyz="0.086  0.0 -0.040" rpy="-1.57 0 -1.57"/>-->
-  <!--        <axis xyz="0 0 1"/>-->
-  <!--      </joint>-->
+    <xacro:property name="threshold" value="0.01"/>
+    <xacro:property name="yaw_lower_limit" value="-3.6"/>
+    <xacro:property name="yaw_upper_limit" value="1.57"/>
+    <xacro:property name="pitch_lower_limit" value="-0.34"/>
+    <xacro:property name="pitch_upper_limit" value="0.93"/>
+    <link name="lower_yaw">
+        <visual>
+            <geometry>
+                <mesh filename="package://rm_description/meshes/sentry/lower_yaw.stl"
+                      scale="0.001 0.001 0.001"/>
+            </geometry>
+        </visual>
+        <inertial>
+            <mass value="99.15e-3"/>
+            <origin xyz="-10.311e-3 -2.902e-3 -40.101e-3" rpy="0 0 0"/>
+            <inertia ixx="1.456e-4" ixy="-7242.148e-9" ixz="-28572.972e-9" iyy="1.608e-4"
+                     iyz="-13303.908e-9" izz="52950.519e-9"/>
+        </inertial>
+        <collision>
+            <origin xyz="-0.166e-3 0 -49.546e-3" rpy="0 0 0"/>
+            <geometry>
+                <box size="0.094 0.032 0.0971"/>
+            </geometry>
+        </collision>
+    </link>
+    <joint name="lower_yaw_joint" type="revolute">
+        <parent link="base_link"/>
+        <child link="lower_yaw"/>
+        <axis xyz="0 0 1"/>
+        <origin xyz="0 0 -129e-3"/>
+        <dynamics damping="0" friction="0.1"/>
+        <limit effort="1.2" velocity="34" lower="${yaw_lower_limit}" upper="${yaw_upper_limit}"/>
+        <safety_controller k_position="100" k_velocity="0.1"
+                           soft_lower_limit="${yaw_lower_limit+threshold}"
+                           soft_upper_limit="${yaw_upper_limit-threshold}"/>
+    </joint>
+    <link name="lower_pitch">
+        <inertial>
+            <mass value="809.574e-3"/>
+            <origin xyz="21.588e-3 -0.686e-3 -30.256e-3"/>
+            <inertia ixx="2.031e-3" ixy="-27414.264e-9" ixz="-55245.014e-9" iyy="6.195e-3"
+                     iyz="31445.023e-9" izz="4.728e-3"/>
+        </inertial>
+        <visual>
+            <origin xyz="0 0 0" rpy="0 0 0"/>
+            <geometry>
+                <mesh filename="package://rm_description/meshes/sentry/lower_pitch.stl" scale="0.001 0.001 0.001"/>
+            </geometry>
+        </visual>
+        <collision>
+            <origin xyz="-0.014 0 -0.066" rpy="0 0 0"/>
+            <geometry>
+                <box size="0.25 0.075 0.064"/>
+            </geometry>
+        </collision>
+        <collision>
+            <origin xyz="77.07e-3 -1.201e-3 0" rpy="0 0 0"/>
+            <geometry>
+                <box size="0.21488 0.134 0.064"/>
+            </geometry>
+        </collision>
+        <collision>
+            <origin xyz="-58e-3 -13e-3 64e-3" rpy="0 0 0"/>
+            <geometry>
+                <box size="0.042 0.059 0.042"/>
+            </geometry>
+        </collision>
+    </link>
+    <joint name="lower_pitch_joint" type="revolute">
+        <parent link="lower_yaw"/>
+        <child link="lower_pitch"/>
+        <axis xyz="0 1 0"/>
+        <origin xyz="0 0 -87.993e-3"/>
+        <dynamics damping="0" friction="0.1"/>
+        <limit effort="3." velocity="86" lower="${pitch_lower_limit}" upper="${pitch_upper_limit}"/>
+        <safety_controller k_position="100" k_velocity="0.1"
+                           soft_lower_limit="${pitch_lower_limit+threshold}"
+                           soft_upper_limit="${pitch_upper_limit-threshold}"/>
+    </joint>
+    <link name="lower_camera">
+        <inertial>
+            <mass value="0.111"/>
+            <origin xyz="24.789e-3 -0.019e-3 -14.471e-3"/>
+            <inertia ixx="15645.374e-9" ixy="-94.19e-9" ixz="143.444e-9" iyy="80877.924e-9"
+                     iyz="-45.908e-9" izz="80823.702e-9"/>
+        </inertial>
+        <visual>
+            <origin xyz=" 0 0 0 " rpy="0 0 0"/>
+            <geometry>
+                <mesh filename="package://rm_description/meshes/sentry/lower_camera.stl" scale="0.001 0.001 0.001"/>
+            </geometry>
+        </visual>
+        <!--<collision>
+          <origin xyz="0 0 -0.015" rpy="0 0 0"/>
+          <geometry>
+            <box size="0.0892 0.04 0.04"/>
+          </geometry>
+        </collision>-->
+    </link>
+    <joint name="lower_camera_joint" type="fixed">
+        <parent link="lower_pitch"/>
+        <child link="lower_camera"/>
+        <origin xyz="19.642e-3 0 -54.20e-3" rpy="0 0 0"/>
+        <axis xyz="0 0 1"/>
+    </joint>
 </robot>

File: urdf/sentry/lower_shooter.transmission.urdf.xacro (robot description, xacro)
@@ -13,5 +13,5 @@
         <type>transmission_interface/SimpleTransmission</type>
         <actuator name="lower_left_friction_wheel_joint_motor">
-            <mechanicalReduction>-1</mechanicalReduction>
+            <mechanicalReduction>1</mechanicalReduction>
         </actuator>
         <joint name="lower_left_friction_wheel_joint">
@@ -22,5 +22,5 @@
         <type>transmission_interface/SimpleTransmission</type>
         <actuator name="lower_right_friction_wheel_joint_motor">
-            <mechanicalReduction>-1</mechanicalReduction>
+            <mechanicalReduction>1</mechanicalReduction>
         </actuator>
         <joint name="lower_right_friction_wheel_joint">

File: urdf/sentry/sentry.urdf.xacro (robot description, xacro)
@@ -4,8 +4,4 @@
     <xacro:arg name="load_gimbal" default="true"/>
     <xacro:arg name="load_shooter" default="true"/>
-    <xacro:arg name="upper_camera_link" default="upper_camera_link"/>
-    <xacro:arg name="upper_camera_optical_frame" default="upper_camera_optical_frame"/>
-    <xacro:arg name="lower_camera_link" default="lower_camera_link"/>
-    <xacro:arg name="lower_camera_optical_frame" default="lower_camera_optical_frame"/>
     <xacro:arg name="use_simulation" default="true"/>
     <xacro:if value="$(arg load_chassis)">
@@ -15,20 +11,11 @@
     </xacro:if>
     <xacro:if value="$(arg load_gimbal)">
+        <xacro:include filename="$(find rm_description)/urdf/common/imu.urdf.xacro"/>
         <xacro:include filename="$(find rm_description)/urdf/sentry/lower_gimbal.urdf.xacro"/>
         <xacro:include filename="$(find rm_description)/urdf/sentry/lower_gimbal.transmission.urdf.xacro"/>
-        <xacro:include filename="$(find rm_description)/urdf/common/camera.urdf.xacro"/>
-        <xacro:camera_sensor xyz="0.127 0 -0.047" rpy="0 0 0" frame_id="$(arg lower_camera_link)" parent="lower_pitch"
-                             camera_sim="$(arg use_simulation)"/>
-        <xacro:camera_optical_frame xyz="0.153 0 -0.0615" rpy="${pi/2} 0 ${pi/2}"
-                                    frame_id="$(arg lower_camera_optical_frame)"
-                                    parent="lower_pitch" camera_sim="$(arg use_simulation)"/>
+        <xacro:IMU connected_to="lower_pitch" imu_name="lower_gimbal_imu" xyz="0.08 0. 0.08" rpy="${pi} 0 ${pi/2}"/>
         <xacro:include filename="$(find rm_description)/urdf/sentry/upper_gimbal.urdf.xacro"/>
         <xacro:include filename="$(find rm_description)/urdf/sentry/upper_gimbal.transmission.urdf.xacro"/>
-        <xacro:include filename="$(find rm_description)/urdf/common/camera.urdf.xacro"/>
-        <xacro:camera_sensor xyz="0.127 0 -0.047" rpy="0 0 0" frame_id="$(arg upper_camera_link)" parent="upper_pitch"
-                             camera_sim="$(arg use_simulation)"/>
-        <xacro:camera_optical_frame xyz="0.153 0 -0.0615" rpy="${-pi/2} 0 ${-pi/2}"
-                                    frame_id="$(arg upper_camera_optical_frame)"
-                                    parent="upper_pitch" camera_sim="$(arg use_simulation)"/>
+        <xacro:IMU connected_to="upper_pitch" imu_name="upper_gimbal_imu" xyz="0.08 0. 0.08" rpy="0 0 -${pi/2}"/>
     </xacro:if>
     <xacro:if value="$(arg load_shooter)">

File: urdf/sentry/upper_gimbal.transmission.urdf.xacro (robot description, xacro)
@@ -7,5 +7,5 @@
         </actuator>
         <joint name="upper_yaw_joint">
-            <offset>3.021</offset>
+            <offset>2.6</offset>
             <hardwareInterface>hardware_interface/EffortJointInterface</hardwareInterface>
         </joint>
@@ -14,8 +14,8 @@
         <type>transmission_interface/SimpleTransmission</type>
         <actuator name="upper_pitch_joint_motor">
-            <mechanicalReduction>1</mechanicalReduction>
+            <mechanicalReduction>-11</mechanicalReduction>
         </actuator>
         <joint name="upper_pitch_joint">
-            <offset>0.498</offset>
+            <offset>0.47</offset>
             <hardwareInterface>hardware_interface/EffortJointInterface</hardwareInterface>
         </joint>
