Commit message: Update sentry urdf

File: urdf/sentry/upper_gimbal.urdf.xacro (robot description, xacro)
@@ -1,9 +1,9 @@
 <?xml version="1.0" encoding="utf-8"?>
 <robot xmlns:xacro="http://www.ros.org/wiki/xacro">
-    <xacro:property name="threshold" value="0.03"/>
-    <xacro:property name="yaw_lower_limit" value="-2.90"/>
-    <xacro:property name="yaw_upper_limit" value="2.97"/>
-    <xacro:property name="pitch_lower_limit" value="-0.843"/>
-    <xacro:property name="pitch_upper_limit" value="0.472"/>
+    <xacro:property name="threshold" value="0.05"/>
+    <xacro:property name="yaw_lower_limit" value="-2.63"/>
+    <xacro:property name="yaw_upper_limit" value="2.56"/>
+    <xacro:property name="pitch_lower_limit" value="-999"/>
+    <xacro:property name="pitch_upper_limit" value="999"/>
     <link name="upper_yaw">
         <visual>
@@ -14,14 +14,19 @@
         </visual>
         <inertial>
-            <mass value="934.339e-3"/>
-            <origin xyz="-0.08e-3 -61.185e-3 90.777e-3" rpy="0 0 0"/>
-            <inertia ixx="1.880e-2" ixy="-6662.219e-9" ixz="7064.827e-9" iyy="1.083e-2"
-                     iyz="7.150e-3" izz="9.057e-3"/>
+            <mass value="173.01e-3"/>
+            <origin xyz="-20.009e-3 23.734e-3 62.295e-3" rpy="0 0 0"/>
+            <inertia ixx="8.0227e-4" ixy="1.063e-4" ixz="2.307e-4" iyy="7.448e-4"
+                     iyz="-2.615e-4" izz="3.223e-4"/>
         </inertial>
         <collision>
-            <origin xyz="0 0 0" rpy="0 0 0"/>
+            <origin xyz="-0.074 0.0925 0.107" rpy="0 0 0"/>
             <geometry>
-                <mesh filename="package://rm_description/meshes/sentry/upper_yaw.stl"
-                      scale="0.001 0.001 0.001"/>
+                <box size="0.045 0.045 0.035"/>
+            </geometry>
+        </collision>
+        <collision>
+            <origin xyz="-0.166e-3 0 49.546e-3" rpy="0 0 0"/>
+            <geometry>
+                <box size="0.094 0.032 0.0971"/>
             </geometry>
         </collision>
@@ -31,5 +36,5 @@
         <child link="upper_yaw"/>
         <axis xyz="0 0 1"/>
-        <origin xyz="0 0 83.4e-3"/>
+        <origin xyz="0 -24.464e-3 228.5e-3"/>
         <dynamics damping="0" friction="0.1"/>
         <limit effort="1.2" velocity="13.82" lower="${yaw_lower_limit}" upper="${yaw_upper_limit}"/>
@@ -40,8 +45,8 @@
     <link name="upper_pitch">
         <inertial>
-            <mass value="1227.797e-3"/>
-            <origin xyz="15.667e-3 -0.268e-3 27.267e-3"/>
-            <inertia ixx="4.484e-3" ixy="813.964e-9" ixz="2.786e-4" iyy="6.599e-3"
-                     iyz="-6822.846e-9" izz="5.343E-3"/>
+            <mass value="809.574e-3"/>
+            <origin xyz="21.588e-3 0.686e-3 30.256e-3"/>
+            <inertia ixx="2.031e-3" ixy="27414.264e-9" ixz="55245.014e-9" iyy="6.195e-3"
+                     iyz="31445.023e-9" izz="4.728e-3"/>
         </inertial>
         <visual>
@@ -52,7 +57,19 @@
         </visual>
         <collision>
-            <origin xyz="0 0 0" rpy="0 0 0"/>
+            <origin xyz="-0.014 0 0.066" rpy="0 0 0"/>
             <geometry>
-                <mesh filename="package://rm_description/meshes/sentry/upper_pitch.stl" scale="0.001 0.001 0.001"/>
+                <box size="0.25 0.075 0.064"/>
+            </geometry>
+        </collision>
+        <collision>
+            <origin xyz="77.07e-3 -1.201e-3 0" rpy="0 0 0"/>
+            <geometry>
+                <box size="0.21488 0.134 0.064"/>
+            </geometry>
+        </collision>
+        <collision>
+            <origin xyz="-58e-3 13e-3 -64e-3" rpy="0 0 0"/>
+            <geometry>
+                <box size="0.042 0.059 0.042"/>
             </geometry>
         </collision>
@@ -62,36 +79,36 @@
         <child link="upper_pitch"/>
         <axis xyz="0 1 0"/>
-        <origin xyz="0 0 0.125"/>
+        <origin xyz="0 0 87.993e-3"/>
         <dynamics damping="0" friction="0.1"/>
-        <limit effort="1.2" velocity="13.82" lower="${pitch_lower_limit}" upper="${pitch_upper_limit}"/>
+        <limit effort="3." velocity="86" lower="${pitch_lower_limit}" upper="${pitch_upper_limit}"/>
         <safety_controller k_position="100" k_velocity="0.1"
                            soft_lower_limit="${pitch_lower_limit+threshold}"
                            soft_upper_limit="${pitch_upper_limit-threshold}"/>
     </joint>
-    <!--  <link name="upper_camera">-->
-    <!--    <inertial>-->
-    <!--          <mass value="0.17671"/>-->
-    <!--          <origin xyz="0.022 0.0 0.0"/>-->
-    <!--          <inertia ixx="2.129e-5" ixy="7.329e-8" ixz="-1.11e-7" iyy="2.198e-4" iyz="-8.04e-7" izz="2.197e-4"/>-->
-    <!--        </inertial>-->
-    <!--        <visual>-->
-    <!--          <origin xyz=" 0 0 0 " rpy="0 -1.57 0"/>-->
-    <!--          <geometry>-->
-    <!--            <mesh filename="package://rm_description/meshes/common/camera.stl" scale="0.001 0.001 0.001"/>-->
-    <!--          </geometry>-->
-    <!--          <material name="Black"/>-->
-    <!--        </visual>-->
-    <!--        <collision>-->
-    <!--          <origin xyz="0 0 0" rpy="0 -1.57 0"/>-->
-    <!--          <geometry>-->
-    <!--            <mesh filename="package://rm_description/meshes/common/camera.stl" scale="0.001 0.001 0.001"/>-->
-    <!--          </geometry>-->
-    <!--        </collision>-->
-    <!--      </link>-->
-    <!--      <joint name="camera_joint" type="fixed">-->
-    <!--        <parent link="pitch"/>-->
-    <!--        <child link="camera"/>-->
-    <!--        <origin xyz="0.086  0.0 -0.040" rpy="-1.57 0 -1.57"/>-->
-    <!--        <axis xyz="0 0 1"/>-->
-    <!--      </joint>-->
+    <link name="upper_camera">
+        <inertial>
+            <mass value="0.111"/>
+            <origin xyz="24.786e-3 0.019e-3 14.471e-3"/>
+            <inertia ixx="15645.374e-9" ixy="94.19e-9" ixz="-143.444e-9" iyy="80877.924e-9"
+                     iyz="-45.908e-9" izz="80823.702e-9"/>
+        </inertial>
+        <visual>
+            <origin xyz=" 0 0 0 " rpy="0 0 0"/>
+            <geometry>
+                <mesh filename="package://rm_description/meshes/sentry/upper_camera.stl" scale="0.001 0.001 0.001"/>
+            </geometry>
+        </visual>
+        <!-- <collision>
+          <origin xyz="0 0 0.015" rpy="0 0 0"/>
+          <geometry>
+            <box size="0.0892 0.04 0.04"/>
+          </geometry>
+        </collision>-->
+    </link>
+    <joint name="upper_camera_joint" type="fixed">
+        <parent link="upper_pitch"/>
+        <child link="upper_camera"/>
+        <origin xyz="19.642e-3 0 54.20e-3" rpy="0 0 0"/>
+        <axis xyz="0 0 1"/>
+    </joint>
 </robot>

File: urdf/sentry/upper_shooter.transmission.urdf.xacro (robot description, xacro)
@@ -4,5 +4,5 @@
         <type>transmission_interface/SimpleTransmission</type>
         <actuator name="upper_trigger_joint_motor">
-            <mechanicalReduction>1</mechanicalReduction>
+            <mechanicalReduction>-2.5</mechanicalReduction>
         </actuator>
         <joint name="upper_trigger_joint">
@@ -13,5 +13,5 @@
         <type>transmission_interface/SimpleTransmission</type>
         <actuator name="upper_left_friction_wheel_joint_motor">
-            <mechanicalReduction>-1</mechanicalReduction>
+            <mechanicalReduction>1</mechanicalReduction>
         </actuator>
         <joint name="upper_left_friction_wheel_joint">
@@ -22,5 +22,5 @@
         <type>transmission_interface/SimpleTransmission</type>
         <actuator name="upper_right_friction_wheel_joint_motor">
-            <mechanicalReduction>-1</mechanicalReduction>
+            <mechanicalReduction>1</mechanicalReduction>
         </actuator>
         <joint name="upper_right_friction_wheel_joint">

File: urdf/sentry/upper_shooter.urdf.xacro (robot description, xacro)
@@ -1,19 +1,61 @@
 <robot xmlns:xacro="http://www.ros.org/wiki/xacro">
-    <xacro:include filename="$(find rm_description)/urdf/common/friction.urdf.xacro"/>
-    <xacro:property name="wheel_offset_x" value="0.009"/>
-    <xacro:property name="wheel_offset_y" value="0.0365"/>
-    <xacro:property name="wheel_offset_z" value="0.00576"/>
-    <xacro:friction_wheel prefixs="upper_left" connected_to="upper_pitch"
-                          wheel_x_offset="${wheel_offset_x}" wheel_y_offset="${-wheel_offset_y}"
-                          wheel_z_offset="${wheel_offset_z}"/>
-    <xacro:friction_wheel prefixs="upper_right" connected_to="upper_pitch"
-                          wheel_x_offset="${wheel_offset_x}" wheel_y_offset="${wheel_offset_y}"
-                          wheel_z_offset="${wheel_offset_z}"/>
+    <link name="upper_left_friction">
+        <inertial>
+             <mass value="0.15269"/>
+             <origin xyz="0 0 -0.004"/>
+             <inertia ixx="4.776e-5" ixy="2.192e-7" ixz="-1.28e-7" iyy="4.759e-5"
+                      iyz="-1.683e-7" izz="6.148e-5"/>
+        </inertial>
+        <visual>
+            <origin xyz="0 0 0" rpy="0 0 0"/>
+            <geometry>
+                <mesh filename="package://rm_description/meshes/sentry/upper_friction_wheel.stl" scale="0.001 0.001 0.001"/>
+            </geometry>
+        </visual>
+        <!--<collision>
+            <origin xyz="0 -0.00125 0.012" rpy="0 0 0"/>
+            <geometry>
+                <box size="0.072 0.07 0.055"/>
+            </geometry>
+        </collision>-->
+    </link>
+    <joint name="upper_left_friction_wheel_joint" type="continuous">
+        <origin xyz="47e-3 36.50e-3 -0.4e-3" rpy="0 0 0"/>
+        <parent link="upper_pitch"/>
+        <child link="upper_left_friction"/>
+        <axis xyz="0 0 1 "/>
+    </joint>
+    <link name="upper_right_friction">
+        <inertial>
+             <mass value="0.15269"/>
+             <origin xyz="0 0 -0.004"/>
+             <inertia ixx="4.776e-5" ixy="2.192e-7" ixz="-1.28e-7" iyy="4.759e-5"
+                      iyz="-1.683e-7" izz="6.148e-5"/>
+        </inertial>
+        <visual>
+            <origin xyz="0 0 0" rpy="0 0 0"/>
+            <geometry>
+                <mesh filename="package://rm_description/meshes/sentry/upper_friction_wheel.stl" scale="0.001 0.001 0.001"/>
+            </geometry>
+        </visual>
+        <!--<collision>
+            <origin xyz="0 0.00125 0.012" rpy="0 0 0"/>
+            <geometry>
+                <box size="0.072 0.07 0.055"/>
+            </geometry>
+        </collision>-->
+    </link>
+    <joint name="upper_right_friction_wheel_joint" type="continuous">
+        <origin xyz="47e-3 -36.50e-3 -0.4e-3" rpy="0 0 0"/>
+        <parent link="upper_pitch"/>
+        <child link="upper_right_friction"/>
+        <axis xyz="0 0 1 "/>
+    </joint>
     <link name="upper_trigger">
         <inertial>
-            <mass value="0.328"/>
-            <origin xyz="1.854e-3 -4.952e-3 20.252e-3"/>
-            <inertia ixx="5.284e-4" ixy="26474.311e-9" ixz="-5533.967e-9" iyy="3.633e-4"
-                     iyz="3258.006e-9" izz="4.750e-4"/>
+            <mass value="344.827e-3"/>
+            <origin xyz="-26.584e-3 0.526e-3 14.311e-3"/>
+            <inertia ixx="2.365e-4" ixy="-100.189e-9" ixz="1.146e-4" iyy="6.707e-4"
+                     iyz="81.455e-9" izz="6.916e-4"/>
         </inertial>
         <visual>
@@ -24,15 +66,14 @@
         </visual>
         <collision>
-            <origin xyz="0 0 0" rpy="0 0 0"/>
+            <origin xyz="0 0 0.006" rpy="0 0 0"/>
             <geometry>
-                <mesh filename="package://rm_description/meshes/sentry/upper_trigger.stl" scale="0.001 0.001 0.001"/>
+                <box size="0.105 0.104 0.045"/>
             </geometry>
         </collision>
     </link>
     <joint name="upper_trigger_joint" type="continuous">
-        <origin xyz="-64.86e-3 0 -19e-3" rpy="0 0 0"/>
+        <origin xyz="-0.142e-3 -23.51e-3 85.467e-3" rpy="0 0 0"/>
         <dynamics damping="0.0" friction="0.01"/>
-        <limit effort="1.0" velocity="43.54" lower="-1e16" upper="1e16"/>
-        <parent link="upper_pitch"/>
+        <parent link="base_link"/>
         <child link="upper_trigger"/>
         <axis xyz="0 0 1 "/>
