Commit message: Update gimbal.transmission.urdf.xacro and gimbal.urdf.xacro of drone.

File: urdf/drone/gimbal.transmission.urdf.xacro (robot description, xacro)
@@ -7,5 +7,5 @@
         </actuator>
         <joint name="yaw_joint">
-            <offset>2.01749</offset>
+            <offset>5.20927</offset>
             <hardwareInterface>hardware_interface/EffortJointInterface</hardwareInterface>
         </joint>
@@ -14,8 +14,8 @@
         <type>transmission_interface/SimpleTransmission</type>
         <actuator name="pitch_joint_motor">
-            <mechanicalReduction>-1</mechanicalReduction>
+            <mechanicalReduction>11</mechanicalReduction>
         </actuator>
         <joint name="pitch_joint">
-            <offset>5.03</offset>
+            <offset>0.887</offset>
             <hardwareInterface>hardware_interface/EffortJointInterface</hardwareInterface>
         </joint>

File: urdf/drone/gimbal.urdf.xacro (robot description, xacro)
@@ -2,6 +2,6 @@
 <robot xmlns:xacro="http://www.ros.org/wiki/xacro">
     <xacro:property name="threshold" value="0.1"/>
-    <xacro:property name="pitch_lower_limit" value="-0.457"/>
-    <xacro:property name="pitch_upper_limit" value="0.430"/>
+    <xacro:property name="pitch_lower_limit" value="-0.6"/>
+    <xacro:property name="pitch_upper_limit" value="0.457"/>
     <xacro:property name="yaw_lower_limit" value="-0.627"/>
     <xacro:property name="yaw_upper_limit" value="0.627"/>
@@ -61,5 +61,5 @@
         <origin xyz="0 0 -0.09" rpy="0 0 0"/>
         <dynamics damping="0.0" friction="0.1"/>
-        <limit effort="1.2" velocity="13.82" lower="${pitch_lower_limit}" upper="${pitch_upper_limit}"/>
+        <limit effort="3.0" velocity="86" lower="${pitch_lower_limit}" upper="${pitch_upper_limit}"/>
         <safety_controller k_position="100" k_velocity="0.1"
                            soft_lower_limit="${pitch_lower_limit+threshold}"
